File: projects/Attiny/Attiny85SMD3/_autosave-mask.kicad_pcb (KiCad board)
At the start: 2 copper layers, 27 x 27 mm, 25 parts, among them CON1 AVR-ISP-6, IC1 ATTINY85-S, P0 CONN_01X01, P1 CONN_01X01, P2 CONN_01X01, P3 CONN_01X01, P4 CONN_01X01

Commit message: OSH Park Badge
Parts:
- removed BT1: Battery, myFootPrints:BATT_CR2032_SMD
- removed CON1: AVR-ISP-6, myFootPrints:AVR-ISP-6
- removed P0, P1, P2, P3, P4, PG0, PG1, PG2, PG3, PG4: CONN_01X01, myFootPrints:testPad
- removed P1: CONN_01X01, Pin_Headers:Pin_Header_Straight_1x01
Changed lines of the file:
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@@
 (kicad_pcb (version 4) (host pcbnew 4.0.4-stable)
   (general
-    (links 36)
+    (links 17)
     (no_connects 0)
     (area 194.094714 77.977999 223.012001 106.807001)
@@
     (tracks 115)
     (zones 0)
-    (modules 25)
+    (modules 12)
     (nets 14)
   )
@@
     (visible_elements 7FFEFFFF)
     (pcbplotparams
-      (layerselection 0x010f0_80000001)
+      (layerselection 0x00080_00000000)
       (usegerberextensions true)
       (excludeedgelayer true)
@@
       (drillshape 0)
       (scaleselection 1)
-      (outputdirectory ""))
+      (outputdirectory gerbers/))
   )
   (net 0 "")
@@
     )
   )
-  (module myFootPrints:testPad (layer F.Cu)
-    (at 211.582 95.885)
-    (descr "module 1 pin (ou trou mecanique de percage)")
-    (tags DEV)
-    (fp_text reference P1 (at 0 0) (layer F.SilkS) hide
-      (effects (font (size 0.508 0.508) (thickness 0.127)))
-    )
-    (fp_text value CONN_01X01 (at 0 0) (layer F.Fab)
-      (effects (font (size 0.127 0.127) (thickness 0.03175)))
-    )
-    (pad 1 smd circle (at 0 0) (size 1.016 1.016) (layers F.Cu F.Paste F.Mask)
-      (net 3 "Net-(CON1-Pad1)"))
-  )
-  (module myFootPrints:BATT_CR2032_SMD (layer B.Cu)
-    (at 207.645 93.345 180)
-    (tags battery)
-    (fp_text reference BT1 (at 0 -5.08 180) (layer B.SilkS) hide
-      (effects (font (size 1.72974 1.08712) (thickness 0.27178)) (justify mirror))
-    )
-    (fp_text value Battery (at 0 2.54 180) (layer B.SilkS) hide
-      (effects (font (size 1.524 1.016) (thickness 0.254)) (justify mirror))
-    )
-    (fp_line (start -7.1755 -6.5405) (end -10.541 -4.572) (layer B.SilkS) (width 0.15))
-    (fp_line (start 7.1755 -6.6675) (end 10.541 -4.572) (layer B.SilkS) (width 0.15))
-    (fp_arc (start -5.4229 -4.6355) (end -3.5179 -6.4135) (angle -90) (layer B.SilkS) (width 0.15))
-    (fp_arc (start 5.4102 -4.7625) (end 7.1882 -6.6675) (angle -90) (layer B.SilkS) (width 0.15))
-    (fp_arc (start -0.0635 -10.033) (end -3.556 -6.4135) (angle -90) (layer B.SilkS) (width 0.15))
-    (fp_line (start 7.62 7.874) (end 10.541 4.5085) (layer B.SilkS) (width 0.15))
-    (fp_line (start -10.541 4.572) (end -7.5565 7.9375) (layer B.SilkS) (width 0.15))
-    (fp_line (start -7.62 7.874) (end 7.62 7.874) (layer B.SilkS) (width 0.15))
-    (fp_line (start -10.541 -4.572) (end -10.541 4.572) (layer B.SilkS) (width 0.15))
-    (fp_line (start 10.541 -4.572) (end 10.541 4.572) (layer B.SilkS) (width 0.15))
-    (fp_circle (center 0 0) (end -10.16 0) (layer Dwgs.User) (width 0.15))
-    (pad 2 smd circle (at 0 0 180) (size 17.78 17.78) (layers B.Cu B.Paste B.Mask)
-      (net 1 GND))
-    (pad 1 smd rect (at -11.43 0 180) (size 2.54 5.08) (layers B.Cu B.Paste B.Mask)
-      (net 2 +BATT))
-    (pad 1 smd rect (at 11.43 0 180) (size 2.54 5.08) (layers B.Cu B.Paste B.Mask)
-      (net 2 +BATT))
-  )
   (module LEDs:LED-0603 (layer F.Cu)
     (at 208.28 101.6)
@@
     )
   )
-  (module Pin_Headers:Pin_Header_Straight_1x01 (layer F.Cu)
-    (at 207.645 81.28)
-    (descr "Through hole pin header")
-    (tags "pin header")
-    (fp_text reference P1 (at -0.6 -0.5) (layer F.SilkS) hide
-      (effects (font (size 0.127 0.127) (thickness 0.03175)))
-    )
-    (fp_text value CONN_01X01 (at 0 0.9) (layer F.Fab)
-      (effects (font (size 0.127 0.127) (thickness 0.03175)))
-    )
-    (pad P5 thru_hole circle (at 0 0) (size 3 3) (drill 2) (layers *.Cu *.Mask))
-  )
-  (module myFootPrints:AVR-ISP-6 (layer F.Cu)
-    (at 214.757 83.82 270)
-    (descr "6-lead dip package, row spacing 7.62 mm (300 mils)")
-    (tags "dil dip 2.54 300")
-    (fp_text reference CON1 (at 0 -2.54 270) (layer F.SilkS) hide
-      (effects (font (size 1 1) (thickness 0.15)))
-    )
-    (fp_text value AVR-ISP-6 (at 0 -3.72 270) (layer F.Fab) hide
-      (effects (font (size 1 1) (thickness 0.15)))
-    )
-    (pad 1 smd oval (at 0 0 270) (size 1.6 1.6) (layers F.Cu F.Paste F.Mask)
-      (net 3 "Net-(CON1-Pad1)"))
-    (pad 2 smd rect (at 2.54 0 270) (size 1.6 1.6) (layers F.Cu F.Paste F.Mask)
-      (net 2 +BATT))
-    (pad 3 smd oval (at 0 2.54 270) (size 1.6 1.6) (layers F.Cu F.Paste F.Mask)
-      (net 4 "Net-(CON1-Pad3)"))
-    (pad 4 smd oval (at 2.54 2.54 270) (size 1.6 1.6) (layers F.Cu F.Paste F.Mask)
-      (net 5 "Net-(CON1-Pad4)"))
-    (pad 5 smd oval (at 0 5.08 270) (size 1.6 1.6) (layers F.Cu F.Paste F.Mask)
-      (net 6 "Net-(CON1-Pad5)"))
-    (pad 6 smd oval (at 2.54 5.08 270) (size 1.6 1.6) (layers F.Cu F.Paste F.Mask)
-      (net 1 GND))
-  )
   (module Resistors_SMD:R_0201 (layer F.Cu)
     (at 205.74 103.505 180)
@@
     )
   )
-  (module myFootPrints:testPad (layer F.Cu)
-    (at 212.09 92.075)
-    (descr "module 1 pin (ou trou mecanique de percage)")
-    (tags DEV)
-    (fp_text reference P0 (at 0 0) (layer F.SilkS) hide
-      (effects (font (size 0.508 0.508) (thickness 0.127)))
-    )
-    (fp_text value CONN_01X01 (at 0 0) (layer F.Fab)
-      (effects (font (size 0.127 0.127) (thickness 0.03175)))
-    )
-    (pad 1 smd circle (at 0 0) (size 1.143 1.143) (layers F.Cu F.Paste F.Mask)
-      (net 5 "Net-(CON1-Pad4)"))
-  )
-  (module myFootPrints:testPad (layer F.Cu)
-    (at 211.201 99.06)
-    (descr "module 1 pin (ou trou mecanique de percage)")
-    (tags DEV)
-    (fp_text reference P2 (at 0 0) (layer F.SilkS) hide
-      (effects (font (size 0.508 0.508) (thickness 0.127)))
-    )
-    (fp_text value CONN_01X01 (at 0 0) (layer F.Fab)
-      (effects (font (size 0.127 0.127) (thickness 0.03175)))
-    )
-    (pad 1 smd circle (at 0 0) (size 0.889 0.889) (layers F.Cu F.Paste F.Mask)
-      (net 4 "Net-(CON1-Pad3)"))
-  )
-  (module myFootPrints:testPad (layer F.Cu)
-    (at 210.82 101.6)
-    (descr "module 1 pin (ou trou mecanique de percage)")
-    (tags DEV)
-    (fp_text reference P3 (at 0 0) (layer F.SilkS) hide
-      (effects (font (size 0.508 0.508) (thickness 0.127)))
-    )
-    (fp_text value CONN_01X01 (at 0 0) (layer F.Fab)
-      (effects (font (size 0.127 0.127) (thickness 0.03175)))
-    )
-    (pad 1 smd circle (at 0 0) (size 0.762 0.762) (layers F.Cu F.Paste F.Mask)
-      (net 11 "Net-(D3-Pad2)"))
-  )
-  (module myFootPrints:testPad (layer F.Cu)
-    (at 210.566 103.505)
-    (descr "module 1 pin (ou trou mecanique de percage)")
-    (tags DEV)
-    (fp_text reference P4 (at 0 0) (layer F.SilkS) hide
-      (effects (font (size 0.508 0.508) (thickness 0.127)))
-    )
-    (fp_text value CONN_01X01 (at 0 0) (layer F.Fab)
-      (effects (font (size 0.127 0.127) (thickness 0.03175)))
-    )
-    (pad 1 smd circle (at 0 0) (size 0.635 0.635) (layers F.Cu F.Paste F.Mask)
-      (net 12 "Net-(D4-Pad2)"))
-  )
-  (module myFootPrints:testPad (layer F.Cu)
-    (at 198.247 92.075)
-    (descr "module 1 pin (ou trou mecanique de percage)")
-    (tags DEV)
-    (fp_text reference PG0 (at 0 0) (layer F.SilkS) hide
-      (effects (font (size 0.508 0.508) (thickness 0.127)))
-    )
-    (fp_text value CONN_01X01 (at 0 0) (layer F.Fab)
-      (effects (font (size 0.127 0.127) (thickness 0.03175)))
-    )
-    (pad 1 smd oval (at 0 0) (size 0.762 1.4) (layers F.Cu F.Paste F.Mask)
-      (net 1 GND))
-  )
-  (module myFootPrints:testPad (layer F.Cu)
-    (at 198.6915 95.885)
-    (descr "module 1 pin (ou trou mecanique de percage)")
-    (tags DEV)
-    (fp_text reference PG1 (at 0 0) (layer F.SilkS) hide
-      (effects (font (size 0.508 0.508) (thickness 0.127)))
-    )
-    (fp_text value CONN_01X01 (at 0 0) (layer F.Fab)
-      (effects (font (size 0.127 0.127) (thickness 0.03175)))
-    )
-    (pad 1 smd oval (at 0 0) (size 0.762 1.1) (layers F.Cu F.Paste F.Mask)
-      (net 1 GND))
-  )
-  (module myFootPrints:testPad (layer F.Cu)
-    (at 199.898 99.06)
-    (descr "module 1 pin (ou trou mecanique de percage)")
-    (tags DEV)
-    (fp_text reference PG2 (at 0 0) (layer F.SilkS) hide
-      (effects (font (size 0.508 0.508) (thickness 0.127)))
-    )
-    (fp_text value CONN_01X01 (at 0 0) (layer F.Fab)
-      (effects (font (size 0.127 0.127) (thickness 0.03175)))
-    )
-    (pad 1 smd oval (at 0 0) (size 0.635 0.889) (layers F.Cu F.Paste F.Mask)
-      (net 1 GND))
-  )
-  (module myFootPrints:testPad (layer F.Cu)
-    (at 201.7395 101.6)
-    (descr "module 1 pin (ou trou mecanique de percage)")
-    (tags DEV)
-    (fp_text reference PG3 (at 0 0) (layer F.SilkS) hide
-      (effects (font (size 0.508 0.508) (thickness 0.127)))
-    )
-    (fp_text value CONN_01X01 (at 0 0) (layer F.Fab)
-      (effects (font (size 0.127 0.127) (thickness 0.03175)))
-    )
-    (pad 1 smd oval (at 0 0) (size 0.508 0.762) (layers F.Cu F.Paste F.Mask)
-      (net 1 GND))
-  )
-  (module myFootPrints:testPad (layer F.Cu)
-    (at 204.1525 103.505)
-    (descr "module 1 pin (ou trou mecanique de percage)")
-    (tags DEV)
-    (fp_text reference PG4 (at -0.0635 0) (layer F.SilkS) hide
-      (effects (font (size 0.635 0.635) (thickness 0.127)))
-    )
-    (fp_text value CONN_01X01 (at 0 0) (layer F.Fab)
-      (effects (font (size 0.127 0.127) (thickness 0.03175)))
-    )
-    (pad 1 smd oval (at 0 0) (size 0.508 0.762) (layers F.Cu F.Paste F.Mask)
-      (net 1 GND))
-  )
   (gr_text www.MakersBox.us (at 207.645 83.439) (layer B.SilkS)
