File: projects/Trinket_Shield/design_files/base.kicad_pcb (KiCad board)
At the start: 2 copper layers, 25.4 x 58.4 mm, 22 parts, among them P1 TRINKET_LEFT, P11 A4 - A0, P2 TRINKET_RIGHT, P3 LEFT_STEPPER, P4 RIGHT_STEPPER, P5 BATT1, P6 BATT2, P7 SERVO, P8 A5 - A1, P9 CONN_01X01, SW1 SPST, U1 ULN2803

Commit message: Update
Parts:
- P5, P6: footprint Terminal_Blocks:TerminalBlock_Pheonix_MPT-2.54mm_2pol -> Terminal_Blocks:TerminalBlock_Pheonix_PT-3.5mm_2pol
- moved P4 10.9 mm to (124.5, 94.0), turned to 90 degrees
- moved C2 7.62 mm to (137.2, 77.5)
- moved C1 5.08 mm to (137.2, 71.1)
- moved P2 2.54 mm to (129.5, 110.5)
- moved P3 2.54 mm to (125.7, 99.1)
- moved P5 1.14 mm to (128.0, 68.1)
- moved P6 1.14 mm to (128.0, 75.4)
Connections:
- P2 pad 6: (no net) -> /D6
- P2 pad 7: (no net) -> /D5
- P3 pad 5: Net-(P3-Pad5) -> /VBAT
- P4 pad 5: Net-(P3-Pad5) -> /VBAT
- P5 pad 1: (no net) -> GND
- P7 pad 2: Net-(P3-Pad5) -> /VBAT
- U1 pad 5: (no net) -> /D6
- U1 pad 6: (no net) -> /D5
Routing:
- net Net-(P3-Pad5): track 54.4 -> 0.00 mm
- net /VBAT: track 62.7 -> 90.0 mm
- net Net-(P6-Pad2): track 43.4 -> 17.7 mm
- net GND: track 78.2 -> 100.7 mm
- net /D8: track 66.6 -> 49.6 mm
- net /D6: track 0.00 -> 13.9 mm
- net /D5: track 0.00 -> 13.8 mm
- net Net-(P4-Pad1): track 22.8 -> 11.7 mm
- net Net-(P4-Pad2): track 19.3 -> 11.7 mm
- net Net-(P4-Pad4): track 7.88 -> 11.7 mm
- net /D3: track 11.2 -> 13.9 mm
- net /D4: track 11.2 -> 13.9 mm
- net Net-(P3-Pad2): track 6.89 -> 9.43 mm
- net Net-(P3-Pad1): track 6.88 -> 9.42 mm
- net Net-(P3-Pad4): track 6.93 -> 9.47 mm
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Other:
- board text added: "- + - +"
- board text added: "Ver 0.1 Sep 2018"
- board text removed: "+ - + -"
- board text removed: "Ver 0.0 Sep 2018"
