File: projects/Trinket_Shield/design_files/base.sch (KiCad schematic (older format))
At the start: 16 parts, among them P1 TRINKET_LEFT, P11 A4 - A0, P2 TRINKET_RIGHT, P3 LEFT_STEPPER, P4 RIGHT_STEPPER, P5 BATT1, P6 BATT2, P7 SERVO, P8 A5 - A1, SW1 SPST, U1 ULN2803

Commit message: Update
Connections:
- wire segments 62 -> 64
Other:
- note added: "- +"
- note removed: "+ -"
Changed lines of the file:
@@
 	0    -1   -1   0
 $EndComp
-Text Notes 6400 1750 0    60   ~ 0
-+ -
+Text Notes 6600 1750 2    60   ~ 0
+- +
 Text Notes 6700 1750 0    60   ~ 0
-+ -
+- +
 Wire Wire Line
 	6550 2100 6750 2100
@@
 	1    0    0    -1
 $EndComp
-$Comp
-L +BATT #PWR06
-U 1 1 59BB7317
-P 6300 2100
-F 0 "#PWR06" H 6300 1950 50  0001 C CNN
-F 1 "+BATT" H 6300 2240 50  0000 C CNN
-F 2 "" H 6300 2100 60  0000 C CNN
-F 3 "" H 6300 2100 60  0000 C CNN
-	1    6300 2100
-	0    -1   -1   0
-$EndComp
 Wire Wire Line
 	6300 2100 6450 2100
@@
 Connection ~ 7850 2850
 $Comp
-L GND #PWR07
+L GND #PWR06
 U 1 1 59BB7D8A
 P 6050 2950
-F 0 "#PWR07" H 6050 2700 50  0001 C CNN
+F 0 "#PWR06" H 6050 2700 50  0001 C CNN
 F 1 "GND" H 6050 2800 50  0000 C CNN
 F 2 "" H 6050 2950 60  0000 C CNN
@@
 Connection ~ 8650 2850
 $Comp
-L GND #PWR08
+L GND #PWR07
 U 1 1 59BB84D9
 P 8900 2400
-F 0 "#PWR08" H 8900 2150 50  0001 C CNN
+F 0 "#PWR07" H 8900 2150 50  0001 C CNN
 F 1 "GND" H 8900 2250 50  0000 C CNN
 F 2 "" H 8900 2400 60  0000 C CNN
@@
 Connection ~ 6950 3150
 $Comp
-L GND #PWR09
+L GND #PWR08
 U 1 1 59BB875A
 P 6950 3150
-F 0 "#PWR09" H 6950 2900 50  0001 C CNN
+F 0 "#PWR08" H 6950 2900 50  0001 C CNN
 F 1 "GND" H 6950 3000 50  0000 C CNN
 F 2 "" H 6950 3150 60  0000 C CNN
@@
 $EndComp
 $Comp
-L GND #PWR010
+L GND #PWR09
 U 1 1 59BB9EFB
 P 6500 3550
-F 0 "#PWR010" H 6500 3300 50  0001 C CNN
+F 0 "#PWR09" H 6500 3300 50  0001 C CNN
 F 1 "GND" H 6500 3400 50  0000 C CNN
 F 2 "" H 6500 3550 60  0000 C CNN
@@
 	5600 4200 5600 4700
 $Comp
-L GND #PWR011
+L GND #PWR010
 U 1 1 59BB7370
 P 5250 4700
-F 0 "#PWR011" H 5250 4450 50  0001 C CNN
+F 0 "#PWR010" H 5250 4450 50  0001 C CNN
 F 1 "GND" H 5250 4550 50  0000 C CNN
 F 2 "" H 5250 4700 60  0000 C CNN
@@
 $EndComp
 $Comp
-L GND #PWR012
+L GND #PWR011
 U 1 1 59BB73AE
 P 5700 4700
-F 0 "#PWR012" H 5700 4450 50  0001 C CNN
+F 0 "#PWR011" H 5700 4450 50  0001 C CNN
 F 1 "GND" H 5700 4550 50  0000 C CNN
 F 2 "" H 5700 4700 60  0000 C CNN
@@
 Wire Wire Line
 	5350 4300 5350 4700
+Wire Wire Line
+	5650 3350 5700 3350
+Wire Wire Line
+	5650 3450 5700 3450
+$Comp
+L GND #PWR012
+U 1 1 59CB1B18
+P 6300 2100
+F 0 "#PWR012" H 6300 1850 50  0001 C CNN
+F 1 "GND" H 6300 1950 50  0000 C CNN
+F 2 "" H 6300 2100 60  0000 C CNN
+F 3 "" H 6300 2100 60  0000 C CNN
+	1    6300 2100
+	1    0    0    -1
+$EndComp
+Connection ~ 8800 2850
 $EndSCHEMATC
