File: projects/Attiny/Attiny84SpinnerTHD_R3/base.kicad_pcb (KiCad board)
At the start: 2 copper layers, 88.9 x 27.9 mm, 29 parts, among them CON1 AVR-ISP-6, IC1 ATTINY84-S, P1 CONN_01X01, P2 CONN_01X01, SW1 SW_PUSH, SW2 SPST, U1 MLX92231

Commit message: Update
Other:
- board text added: "Rev 1.1 Sep 2017"
- board text removed: "Rev 1.0 Aug 2017"
Changed lines of the file:
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@@
     (links 46)
     (no_connects 0)
-    (area 157.48 66.04 247.700001 98.425001)
+    (area 158.699999 68.529999 247.700001 96.570001)
     (thickness 1.6)
     (drawings 25)
@@
   (gr_line (start 172.72 96.52) (end 233.68 96.52) (angle 90) (layer Edge.Cuts) (width 0.1))
   (gr_line (start 233.68 80.01) (end 233.68 85.09) (angle 90) (layer Dwgs.User) (width 0.254))
-  (gr_text "Rev 1.0\nAug 2017" (at 229.235 92.075) (layer B.SilkS)
+  (gr_text "Rev 1.1\nSep 2017" (at 229.235 92.075) (layer B.SilkS)
     (effects (font (size 1.25 1.25) (thickness 0.15)) (justify mirror))
   )

Commit message: PiFet Instructable published
Parts:
- R0, R1, R2, R3, R4, R5, R6, R7: value 330 -> 100
Other:
- board text added: "Rev 1.2 Dec 2017"
- board text removed: "Rev 1.1 Sep 2017"
Changed lines of the file:
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@@
     (links 46)
     (no_connects 0)
-    (area 158.699999 68.529999 247.700001 96.570001)
+    (area 157.48 66.04 247.700001 98.425001)
     (thickness 1.6)
     (drawings 25)
@@
     (35 F.Paste user)
     (36 B.SilkS user)
-    (37 F.SilkS user)
+    (37 F.SilkS user hide)
     (38 B.Mask user)
     (39 F.Mask user)
@@
       (effects (font (size 1 1) (thickness 0.15)))
     )
-    (fp_text value 330 (at 0 0 270) (layer F.SilkS)
+    (fp_text value 100 (at 0 0 270) (layer F.SilkS)
       (effects (font (size 1 1) (thickness 0.15)))
     )
@@
       (effects (font (size 1 1) (thickness 0.15)))
     )
-    (fp_text value 330 (at 0 0 270) (layer F.SilkS)
+    (fp_text value 100 (at 0 0 270) (layer F.SilkS)
       (effects (font (size 1 1) (thickness 0.15)))
     )
@@
       (effects (font (size 1 1) (thickness 0.15)))
     )
-    (fp_text value 330 (at 0 0 270) (layer F.SilkS)
+    (fp_text value 100 (at 0 0 270) (layer F.SilkS)
       (effects (font (size 1 1) (thickness 0.15)))
     )
@@
       (effects (font (size 1 1) (thickness 0.15)))
     )
-    (fp_text value 330 (at 0 0 270) (layer F.SilkS)
+    (fp_text value 100 (at 0 0 270) (layer F.SilkS)
       (effects (font (size 1 1) (thickness 0.15)))
     )
@@
       (effects (font (size 1 1) (thickness 0.15)))
     )
-    (fp_text value 330 (at 0 0 270) (layer F.SilkS)
+    (fp_text value 100 (at 0 0 270) (layer F.SilkS)
       (effects (font (size 1 1) (thickness 0.15)))
     )
@@
       (effects (font (size 1 1) (thickness 0.15)))
     )
-    (fp_text value 330 (at 0 0 270) (layer F.SilkS)
+    (fp_text value 100 (at 0 0 270) (layer F.SilkS)
       (effects (font (size 1 1) (thickness 0.15)))
     )
@@
       (effects (font (size 1 1) (thickness 0.15)))
     )
-    (fp_text value 330 (at 0 0 270) (layer F.SilkS)
+    (fp_text value 100 (at 0 0 270) (layer F.SilkS)
       (effects (font (size 1 1) (thickness 0.15)))
     )
@@
       (effects (font (size 1 1) (thickness 0.15)))
     )
-    (fp_text value 330 (at 0 0 270) (layer F.SilkS)
+    (fp_text value 100 (at 0 0 270) (layer F.SilkS)
       (effects (font (size 1 1) (thickness 0.15)))
     )
@@
   (gr_line (start 172.72 96.52) (end 233.68 96.52) (angle 90) (layer Edge.Cuts) (width 0.1))
   (gr_line (start 233.68 80.01) (end 233.68 85.09) (angle 90) (layer Dwgs.User) (width 0.254))
-  (gr_text "Rev 1.1\nSep 2017" (at 229.235 92.075) (layer B.SilkS)
+  (gr_text "Rev 1.2\nDec 2017" (at 229.235 92.075) (layer B.SilkS)
     (effects (font (size 1.25 1.25) (thickness 0.15)) (justify mirror))
   )
