File: projects/ChickTech_Robot/design_files_R2.1/base.kicad_pcb (KiCad board)
At the start: 2 copper layers, 31.8 x 58.4 mm, 32 parts, among them P1 TRINKET_LEFT, P2 TRINKET_RIGHT, P3 RIGHT_STEPPER, P4 LEFT_STEPPER, P5 BATT1, P6 BATT2, P7 SERVO, P8 A5 - A1, P9 CONN_01X01, Q1 OPTO_NPN, Q2 OPTO_NPN, SW1 SPST, SW2 SW_PUSH, U1 ULN2803

Commit message: PiFet Instructable published
Parts:
- D3: value IR_LED -> LED
- D5: value LED -> IR LED
- R3: value 100 -> 300
- R5: value 330 -> 100
- moved R5 3.17 mm to (148.0, 80.0)
- moved R3 2.54 mm to (151.1, 80.0)
Routing:
- net /A4: track 4.60 -> 16.6 mm
- net Net-(D5-Pad2): track 21.7 -> 11.8 mm
- net /D1: track 25.4 -> 19.2 mm
- net Net-(D3-Pad2): track 8.04 -> 6.50 mm
Changed lines of the file:
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@@
     (thickness 1.6)
     (drawings 52)
-    (tracks 265)
+    (tracks 259)
     (zones 0)
     (modules 32)
@@
       (effects (font (size 1 1) (thickness 0.15)))
     )
-    (fp_text value IR_LED (at 1.3 -2.9 90) (layer F.Fab)
+    (fp_text value LED (at 1.3 -2.9 90) (layer F.Fab)
       (effects (font (size 1 1) (thickness 0.15)))
     )
@@
       (effects (font (size 1 1) (thickness 0.15)))
     )
-    (fp_text value LED (at 1.3 -2.9 90) (layer F.Fab)
+    (fp_text value "IR LED" (at 1.3 -2.9 90) (layer F.Fab)
       (effects (font (size 1 1) (thickness 0.15)))
     )
@@
   )
   (module myFootPrints:Resistor_Horz (layer F.Cu)
-    (at 148.59 80.01 90)
+    (at 151.13 80.01 90)
     (descr "Resistor, Axial,  RM 10mm, 1/3W,")
     (tags "Resistor, Axial, RM 10mm, 1/3W,")
@@
       (effects (font (size 1 1) (thickness 0.15)))
     )
-    (fp_text value 100 (at 0 0 90) (layer F.SilkS)
+    (fp_text value 300 (at 0 0 90) (layer F.SilkS)
       (effects (font (size 1 1) (thickness 0.15)))
     )
@@
   )
   (module myFootPrints:Resistor_Horz (layer F.Cu)
-    (at 151.13 80.01 90)
+    (at 147.955 80.01 90)
     (descr "Resistor, Axial,  RM 10mm, 1/3W,")
     (tags "Resistor, Axial, RM 10mm, 1/3W,")
@@
       (effects (font (size 1 1) (thickness 0.15)))
     )
-    (fp_text value 330 (at 0 0 90) (layer F.SilkS)
+    (fp_text value 100 (at 0 0 90) (layer F.SilkS)
       (effects (font (size 1 1) (thickness 0.15)))
     )
@@
   (segment (start 130.302 88.9) (end 132.08 90.678) (width 0.4064) (layer B.Cu) (net 19))
   (segment (start 134.112 90.678) (end 134.62 90.17) (width 0.4064) (layer B.Cu) (net 19))
-  (segment (start 144.78 85.09) (end 146.685 83.185) (width 0.3048) (layer F.Cu) (net 20))
-  (segment (start 146.685 83.185) (end 148.59 83.185) (width 0.3048) (layer F.Cu) (net 20))
+  (segment (start 144.78 85.09) (end 143.51 85.09) (width 0.3048) (layer F.Cu) (net 20))
+  (segment (start 151.13 81.28) (end 151.13 83.185) (width 0.3048) (layer F.Cu) (net 20))
+  (segment (start 149.86 80.01) (end 151.13 81.28) (width 0.3048) (layer F.Cu) (net 20))
+  (segment (start 144.145 80.01) (end 149.86 80.01) (width 0.3048) (layer F.Cu) (net 20))
+  (segment (start 142.875 81.28) (end 144.145 80.01) (width 0.3048) (layer F.Cu) (net 20))
+  (segment (start 142.875 84.455) (end 142.875 81.28) (width 0.3048) (layer F.Cu) (net 20))
+  (segment (start 143.51 85.09) (end 142.875 84.455) (width 0.3048) (layer F.Cu) (net 20))
   (segment (start 132.334 82.677) (end 132.334 82.804) (width 0.3048) (layer B.Cu) (net 21))
   (segment (start 132.334 82.804) (end 133.35 83.82) (width 0.3048) (layer B.Cu) (net 21))
@@
   (segment (start 147.32 107.95) (end 147.32 102.235) (width 0.3048) (layer F.Cu) (net 26))
   (segment (start 147.955 108.585) (end 147.32 107.95) (width 0.3048) (layer F.Cu) (net 26))
-  (segment (start 148.59 76.835) (end 147.32 75.565) (width 0.4064) (layer B.Cu) (net 27))
-  (segment (start 148.59 71.755) (end 149.86 71.755) (width 0.4064) (layer B.Cu) (net 27))
-  (segment (start 147.32 73.025) (end 148.59 71.755) (width 0.4064) (layer B.Cu) (net 27))
-  (segment (start 147.32 75.565) (end 147.32 73.025) (width 0.4064) (layer B.Cu) (net 27))
-  (segment (start 148.59 76.835) (end 148.59 76.2) (width 0.4064) (layer B.Cu) (net 27) (status 30))
+  (segment (start 149.86 71.755) (end 150.495 71.755) (width 0.4064) (layer B.Cu) (net 27))
+  (segment (start 150.495 71.755) (end 151.765 73.025) (width 0.4064) (layer B.Cu) (net 27))
+  (segment (start 151.765 73.025) (end 151.765 76.2) (width 0.4064) (layer B.Cu) (net 27))
+  (segment (start 151.765 76.2) (end 151.13 76.835) (width 0.4064) (layer B.Cu) (net 27))
   (segment (start 149.86 103.505) (end 149.86 103.251) (width 0.4064) (layer B.Cu) (net 28) (status 30))
   (segment (start 149.86 103.251) (end 151.13 101.346) (width 0.4064) (layer B.Cu) (net 28) (status 20))
   (segment (start 151.13 101.346) (end 151.13 100.965) (width 0.4064) (layer B.Cu) (net 28) (status 30))
-  (segment (start 151.13 76.835) (end 151.13 77.47) (width 0.4064) (layer B.Cu) (net 29))
-  (segment (start 151.13 77.47) (end 149.86 78.74) (width 0.4064) (layer B.Cu) (net 29))
-  (segment (start 148.59 66.675) (end 149.86 66.675) (width 0.4064) (layer B.Cu) (net 29))
-  (segment (start 146.05 69.215) (end 148.59 66.675) (width 0.4064) (layer B.Cu) (net 29))
-  (segment (start 146.05 76.835) (end 146.05 69.215) (width 0.4064) (layer B.Cu) (net 29))
-  (segment (start 147.955 78.74) (end 146.05 76.835) (width 0.4064) (layer B.Cu) (net 29))
-  (segment (start 149.86 78.74) (end 147.955 78.74) (width 0.4064) (layer B.Cu) (net 29))
-  (segment (start 151.13 76.835) (end 151.765 76.835) (width 0.4064) (layer B.Cu) (net 29) (status 30))
-  (segment (start 151.765 76.835) (end 151.13 77.47) (width 0.4064) (layer B.Cu) (net 29) (status 10))
-  (segment (start 149.86 67.31) (end 149.86 66.675) (width 0.4064) (layer B.Cu) (net 29) (status 20))
+  (segment (start 147.32 76.2) (end 147.955 76.835) (width 0.4064) (layer B.Cu) (net 29))
+  (segment (start 147.32 68.58) (end 147.32 76.2) (width 0.4064) (layer B.Cu) (net 29))
+  (segment (start 149.225 66.675) (end 147.32 68.58) (width 0.4064) (layer B.Cu) (net 29))
+  (segment (start 149.86 66.675) (end 149.225 66.675) (width 0.4064) (layer B.Cu) (net 29))
   (segment (start 144.78 110.49) (end 145.415 110.49) (width 0.3048) (layer F.Cu) (net 30))
   (segment (start 145.415 110.49) (end 146.685 109.22) (width 0.3048) (layer F.Cu) (net 30))
@@
   (segment (start 150.495 93.98) (end 151.13 94.615) (width 0.3048) (layer F.Cu) (net 34))
   (segment (start 129.54 87.63) (end 130.175 87.63) (width 0.3048) (layer F.Cu) (net 34))
+  (segment (start 146.05 83.82) (end 146.685 83.185) (width 0.3048) (layer B.Cu) (net 35))
+  (segment (start 140.97 85.09) (end 142.24 83.82) (width 0.3048) (layer B.Cu) (net 35))
+  (segment (start 142.24 83.82) (end 146.05 83.82) (width 0.3048) (layer B.Cu) (net 35))
   (segment (start 129.54 85.09) (end 140.97 85.09) (width 0.3048) (layer B.Cu) (net 35))
-  (segment (start 151.13 81.915) (end 151.13 83.185) (width 0.3048) (layer B.Cu) (net 35))
-  (segment (start 150.495 81.28) (end 151.13 81.915) (width 0.3048) (layer B.Cu) (net 35))
-  (segment (start 147.32 81.28) (end 150.495 81.28) (width 0.3048) (layer B.Cu) (net 35))
-  (segment (start 146.685 81.915) (end 147.32 81.28) (width 0.3048) (layer B.Cu) (net 35))
-  (segment (start 146.685 83.185) (end 146.685 81.915) (width 0.3048) (layer B.Cu) (net 35))
-  (segment (start 146.05 83.82) (end 146.685 83.185) (width 0.3048) (layer B.Cu) (net 35))
-  (segment (start 142.24 83.82) (end 146.05 83.82) (width 0.3048) (layer B.Cu) (net 35))
-  (segment (start 140.97 85.09) (end 142.24 83.82) (width 0.3048) (layer B.Cu) (net 35))
+  (segment (start 146.685 83.185) (end 147.955 83.185) (width 0.3048) (layer B.Cu) (net 35))
   (zone (net 1) (net_name GND) (layer F.Cu) (hatch edge 0.508)
     (connect_pads (clearance 1))
