File: projects/Attiny/Attiny85Challenge/design_files/base.sch (KiCad schematic (older format))
At the start: 25 parts, among them CON1 AVR-ISP-6, IC1 IC1, P0 CONN_01X01, P1 CONN_01X01, P2 CONN_01X01, P3 CONN_01X01, P4 CONN_01X01, P5 CONN_01X01

Commit message: Challenge second Chance card
Parts:
- D3: footprint footprints:LED-0603 -> footprints:LED_0402
- D4: footprint footprints:LED-0603 -> footprints:LED_0201
Changed lines of the file:
@@
 F 0 "D3" H 6400 5350 50  0000 C CNN
 F 1 "LED" H 6400 5150 50  0000 C CNN
-F 2 "footprints:LED-0603" H 6400 5250 50  0001 C CNN
+F 2 "footprints:LED_0402" H 6400 5250 50  0001 C CNN
 F 3 "" H 6400 5250 50  0000 C CNN
 	1    6400 5250
@@
 F 0 "D4" H 6450 5700 50  0000 C CNN
 F 1 "LED" H 6450 5500 50  0000 C CNN
-F 2 "footprints:LED-0603" H 6450 5600 50  0001 C CNN
+F 2 "footprints:LED_0201" H 6450 5600 50  0001 C CNN
 F 3 "" H 6450 5600 50  0000 C CNN
 	1    6450 5600
