File: projects/pizero/pizero-MOSFET3/pizero.kicad_pcb (KiCad board)
At the start: 2 copper layers, 56 x 30 mm, 24 parts, among them J1 BARREL_JACK, P1 I2C, P3 Raspberry_Pi_+_Conn, P4 CONN_01X02, Q1 IRLB8271, SW1 SPST, SW2 SPST, SW3 SPST, U1 R-78-E

Commit message: Challenge second Chance card
Parts:
- P4: footprint project_footprints:TerminalBlock_Pheonix_MPT-2.54mm_2pol -> Terminal_Blocks:TerminalBlock_Pheonix_PT-3.5mm_2pol
- VAL: moved to B.Cu
- moved VAL 40.7 mm to (45.6, 59.8)
- moved VAL 31.5 mm to (77.0, 61.2), turned to 180 degrees
- moved C1 1.65 mm to (60.0, 52.4)
Routing:
- net +12V: track 81.7 -> 80.0 mm
- net GND: track 192.1 -> 191.4 mm
Other:
- board text added: "Rev 0.31 Jan 18"
- board text removed: "Rev 0.3 Nov 17"
