File: projects/Attiny/Attiny85HeartSMD1/design_files/base.kicad_pcb (KiCad board)
At the start: 2 copper layers, 31.5 x 31.5 mm, 12 parts, among them CON1 AVR-ISP-6, P1 CONN_01X01, P2 CONN_01X01, P3 CONN_01X01, SW1 SPST, SW2 SW_PUSH

Commit message: update
Parts:
- removed CON1: AVR-ISP-6, myFootPrints:AVR-ISP-6
- ATTINY1: value ATTINY85-S -> ATTINY85
- moved G*** 14.2 mm to (203.8, 100.3)
- moved P1 10.8 mm to (209.8, 79.5)
- moved SW2 8.95 mm to (212.1, 90.2), turned to 90 degrees
- moved P3 2.54 mm to (216.4, 100.1)
- moved P2 2.54 mm to (215.5, 101.0)
- moved SW1 2.27 mm to (200.0, 92.7)
- moved BT1 1.66 mm to (207.6, 92.1), turned to 45 degrees
- moved ATTINY1 1.08 mm to (214.6, 97.5)
Routing:
- net GND: track 74.0 -> 45.2 mm
- net Net-(ATTINY1-Pad2): track 34.5 -> 11.8 mm
- net Net-(ATTINY1-Pad1): track 17.9 -> 0.00 mm
- net Net-(ATTINY1-Pad7): track 13.9 -> 0.00 mm
- net +BATT: track 39.4 -> 30.8 mm
- net Net-(ATTINY1-Pad6): track 24.5 -> 18.9 mm
- net Net-(BT1-Pad1): track 52.9 -> 47.5 mm
- net Net-(ATTINY1-Pad3): track 7.60 -> 3.69 mm
- net Net-(ATTINY1-Pad5): track 16.1 -> 16.7 mm
Other:
- board size 31.5 x 31.5 mm -> 27 x 27 mm
