File: projects/chirp/design_files/project.kicad_pcb (KiCad board)
At the start: 2 copper layers, 20.3 x 26.7 mm, 10 parts, among them CON1 ISP, IC1 ATTINY85, J1 JMP, Q1 LIGHT

Commit message: Update
Parts:
- C1: footprint footprints:C_1206_HandSoldering -> Capacitors_SMD:C_0805_HandSoldering
- CON1: footprint Pin_Headers:Pin_Header_Straight_2x03_Pitch2.54mm -> footprints:Pin_Header_Straight_2x03_Pitch2.54mm
- D1: footprint LEDs:LED_1206_HandSoldering -> LEDs:LED_0805_HandSoldering
- IC1: footprint footprints:SOIC-8_3.9x4.9mm_Pitch1.27mm -> footprints:SOIJ-8_5.3x5.3mm_Pitch1.27mm
- J1: footprint Resistors_SMD:R_1206_HandSoldering -> myFootPrints:SW_SMD_TOUCH
- Q1: footprint footprints:PHOTO_TRANS -> Opto-Devices:PhotoDiode_SMD-DIL2_4.5x4
- R1: footprint Resistors_SMD:R_1206_HandSoldering -> Resistors_SMD:R_0805_HandSoldering
- moved D1 8.92 mm to (224.9, 99.5)
- moved CON1 4.87 mm to (214.9, 89.0)
- moved R1 4.85 mm to (224.9, 105.5), turned to 90 degrees
- moved C1 2.90 mm to (221.9, 91.5), turned to 180 degrees
- moved J1 2.39 mm to (209.4, 98.5), turned to 180 degrees
- moved IC1 1.98 mm to (217.9, 99.6)
- moved SP1 1.80 mm to (216.9, 108.5)
- moved Q1 1.18 mm to (209.4, 106.0), turned to 270 degrees
Connections:
- D1 pad 2: Net-(CON1-Pad1) -> Net-(CON1-Pad3)
- J1 pad 2: Net-(IC1-Pad3) -> Net-(IC1-Pad2)
- Q1 pad 1: GND -> Net-(IC1-Pad3)
- Q1 pad 2: (no net) -> GND
Routing:
- net +BATT: track 24.1 -> 54.0 mm
- net GND: track 61.8 -> 79.8 mm, vias 2 -> 1
- net Net-(CON1-Pad3): track 9.07 -> 26.1 mm
- net Net-(IC1-Pad2): track 11.6 -> 4.58 mm
- net Net-(CON1-Pad4): track 14.9 -> 21.6 mm
- net Net-(D1-Pad1): track 8.50 -> 3.30 mm
- net Net-(IC1-Pad3): track 3.27 -> 7.78 mm
- net Net-(CON1-Pad1): track 18.4 -> 15.8 mm
- net Net-(CON1-Pad5): track 8.95 -> 10.5 mm
Other:
- board text added: "V0.2"
