File: projects/rroll/design_files/project.kicad_pcb (KiCad board)
At the start: 2 copper layers, 20.3 x 26.7 mm, 10 parts, among them CON1 ISP, IC1 ATTINY85, J1 JMP, Q1 LIGHT

Commit message: rroll to fab
Parts:
- moved Q1 16.0 mm to (225.0, 109.1), turned to 90 degrees
- moved R1 1.50 mm to (225.0, 104.0)
- moved D1 1.22 mm to (225.0, 98.3)
- moved G*** 0.31 mm to (216.8, 100.2)
Routing:
- net GND: track 79.8 -> 59.1 mm
- net Net-(IC1-Pad3): track 7.78 -> 20.3 mm
Other:
- board text added: "Press Me?"
- board text added: "V0.3"
- board text removed: "V0.2"
