File: projects/Attiny/Attiny85HeartSMD/design_files/base.sch (KiCad schematic (older format))
At the start: 9 parts, among them CON1 AVR-ISP-6, IC1 ATTINY85-S, P1 CONN_01X01, SW1 SW_PUSH, SW2 SPST

Commit message: Updates
Parts:
- removed SW1: SW_PUSH, myFootPrints:SW_SMD_PUSH, symbol SW_PUSH
- BT1: footprint myFootPrints:BATT_CR2032_SMD -> footprints:BATT_CR2032_SMD; symbol Battery -> Battery-RESCUE-base
- C1: footprint Capacitors_SMD:C_1206_HandSoldering -> footprints:C_1206_HandSoldering
- CON1: footprint myFootPrints:AVR-ISP-6 -> footprints:AVR-ISP-6
- D1: symbol LED -> LED-RESCUE-base
- P1: footprint Pin_Headers:Pin_Header_Angled_1x01 -> footprints:Pin_Header_Straight_1x01
- R1: footprint Resistors_Universal:Resistor_SMDuniversal_0805to1206_HandSoldering -> footprints:R_1206_HandSoldering
- SW1: renamed from SW2; footprint myFootPrints:SPST_SMD -> footprints:SPST_SMD
- U1: renamed from IC1; value ATTINY85-S -> ATTINY85; footprint Housings_SOIC:SOIJ-8_5.3x5.3mm_Pitch1.27mm -> footprints:SOIJ-8_5.3x5.3mm_Pitch1.27mm
Connections:
- net GND: no longer R1.2
- net D1: now reaches CON1.1, U1.6 (PB1(MISO/DO/AIN1/OC0B/OC1A/PCINT1))
- net D2: now reaches CON1.3, U1.7 (PB2(SCK/USCK/SCL/T0/INT0/ADC1/PCINT2))
- net D0: now reaches CON1.4, D1.2 (A), U1.5 (PB0(MOSI/DI/SDA/AIN0/OC0A/OC1A/AREF/PCINT0))
- net D3: now reaches U1.2 (PB3(XTAL1/CLKI/OC1B/ADC3/PCINT3))
- net D4: now reaches U1.3 (PB4(XTAL2/CLKO/OC1B/ADC2/PCINT4))
- net D4: now also R1.2
- no-connect marks 1 -> 2
Other:
- moved on the sheet: BT1, C1, CON1, D1, P1, R1, SW1, U1
