File: projects/Art/project.kicad_pcb (KiCad board)
At the start: 2 copper layers, 15.2 x 15.2 mm, 9 parts

Commit message: Updates
Parts:
- removed the FPasteNeg at (100.0, 100.0)
- added G***: F.PasteNormal, footprints:cube_paste_normal, F.Cu at (100.0, 100.0)
