File: projects/Attiny/Attiny85ChallengeBodge/design_files/project.kicad_pcb (KiCad board)
At the start: 2 copper layers, 48.3 x 25.4 mm, 39 parts, among them CON1 AVR-ISP-6, IC1 IC1, J1 Conn_01x01, J10 Conn_01x01, J11 Conn_01x01, J12 Conn_01x01, J13 Conn_01x01, J14 Conn_01x01, J15 Conn_01x01, J2 Conn_01x01, J3 Conn_01x01, J4 Conn_01x01, J5 Conn_01x01, J6 Conn_01x01, J7 Conn_01x01, J8 Conn_01x01, J9 Conn_01x01, P5 CONN_01X01, SW1 SW_Push_SPDT

Commit message: update
Parts:
- R0, R1, R2, R3, R4: value 330 -> 100
- moved J10 2.54 mm to (186.7, 106.7)
- moved J10 2.54 mm to (186.7, 104.1)
- moved VAL 0.64 mm to (165.1, 96.5), turned to 90 degrees
Connections:
- R0 pad 2: Net-(D0-Pad2) -> Net-(R0-Pad2)
Routing:
- net Net-(D0-Pad2): track 3.44 -> 4.19 mm
- added copper zone on F.Cu, net GND
Changed lines of the file:
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@@
 (kicad_pcb (version 4) (host pcbnew 4.0.7)
   (general
-    (links 48)
-    (no_connects 2)
+    (links 47)
+    (no_connects 1)
     (area 142.189999 92.659999 190.550001 118.160001)
     (thickness 1.6)
@@
     (zones 0)
     (modules 39)
-    (nets 16)
+    (nets 17)
   )
   (page USLetter)
@@
   )
   (setup
-    (last_trace_width 0.1524)
+    (last_trace_width 0.3048)
     (user_trace_width 0.254)
     (user_trace_width 0.3048)
@@
   (net 14 "Net-(IC1-Pad3)")
   (net 15 "Net-(SW1-Pad3)")
+  (net 16 "Net-(R0-Pad2)")
   (net_class Default "This is the default net class."
     (clearance 0.1524)
@@
     (add_net "Net-(IC1-Pad2)")
     (add_net "Net-(IC1-Pad3)")
+    (add_net "Net-(R0-Pad2)")
     (add_net "Net-(SW1-Pad3)")
   )
   (module footprints:testPad (layer F.Cu)
-    (at 186.69 104.14)
+    (at 186.69 106.68)
     (descr "module 1 pin (ou trou mecanique de percage)")
     (tags DEV)
@@
   )
   (module footprints:testPad (layer F.Cu)
-    (at 186.69 106.68)
+    (at 186.69 104.14)
     (descr "module 1 pin (ou trou mecanique de percage)")
     (tags DEV)
@@
   )
   (module myFootPrints:MadeInOregonRev25 (layer F.Cu)
-    (at 165.735 96.52 180)
-    (fp_text reference VAL (at 0 0 180) (layer F.SilkS) hide
+    (at 165.1 96.52 90)
+    (fp_text reference VAL (at 0 0 90) (layer F.SilkS) hide
       (effects (font (size 1.143 1.143) (thickness 0.1778)))
     )
-    (fp_text value MadeInOregonRev25 (at 0 0 180) (layer F.SilkS) hide
+    (fp_text value MadeInOregonRev25 (at 0 0 90) (layer F.SilkS) hide
       (effects (font (size 1.143 1.143) (thickness 0.1778)))
     )
@@
       (effects (font (size 1 1) (thickness 0.15)))
     )
-    (fp_text value 330 (at 0 1.9) (layer F.Fab)
+    (fp_text value 100 (at 0 1.9) (layer F.Fab)
       (effects (font (size 1 1) (thickness 0.15)))
     )
@@
       (effects (font (size 1 1) (thickness 0.15)))
     )
-    (fp_text value 330 (at 0 1.5) (layer F.Fab)
+    (fp_text value 100 (at 0 1.5) (layer F.Fab)
       (effects (font (size 1 1) (thickness 0.15)))
     )
@@
       (net 4 "Net-(CON1-Pad3)"))
     (pad 2 smd rect (at 0.75 0) (size 0.5 0.9) (layers F.Cu F.Paste F.Mask)
-      (net 10 "Net-(D0-Pad2)"))
+      (net 16 "Net-(R0-Pad2)"))
     (model ${KISYS3DMOD}/Resistors_SMD.3dshapes/R_0603.wrl
       (at (xyz 0 0 0))
@@
       (effects (font (size 1 1) (thickness 0.15)))
     )
-    (fp_text value 330 (at 0 1.5) (layer F.Fab)
+    (fp_text value 100 (at 0 1.5) (layer F.Fab)
       (effects (font (size 1 1) (thickness 0.15)))
     )
@@
       (effects (font (size 1 1) (thickness 0.15)))
     )
-    (fp_text value 330 (at 0 1.45) (layer F.Fab)
+    (fp_text value 100 (at 0 1.45) (layer F.Fab)
       (effects (font (size 1 1) (thickness 0.15)))
     )
@@
       (effects (font (size 1 1) (thickness 0.15)))
     )
-    (fp_text value 330 (at 0 1.5) (layer F.Fab)
+    (fp_text value 100 (at 0 1.5) (layer F.Fab)
       (effects (font (size 1 1) (thickness 0.15)))
     )
@@
   (segment (start 166.37 103.505) (end 165.1 102.235) (width 0.4064) (layer F.Cu) (net 1))
   (segment (start 181.61 104.14) (end 181.61 102.87) (width 0.4064) (layer F.Cu) (net 1))
-  (segment (start 152.781 103.124) (end 152.781 104.14) (width 0.4064) (layer F.Cu) (net 1))
-  (segment (start 153.67 102.235) (end 152.781 103.124) (width 0.4064) (layer F.Cu) (net 1))
+  (segment (start 152.781 104.394) (end 152.781 104.14) (width 0.4064) (layer F.Cu) (net 1) (status 10))
+  (segment (start 153.67 102.235) (end 152.781 104.394) (width 0.4064) (layer F.Cu) (net 1) (status 20))
   (segment (start 157.48 102.235) (end 153.67 102.235) (width 0.4064) (layer F.Cu) (net 1))
   (segment (start 165.1 102.235) (end 157.48 102.235) (width 0.4064) (layer F.Cu) (net 1))
@@
   (segment (start 175.26 105.41) (end 175.26 104.013) (width 0.4064) (layer B.Cu) (net 9))
   (segment (start 171.45 101.092) (end 175.26 105.41) (width 0.4064) (layer B.Cu) (net 9))
-  (segment (start 184.9 106.68) (end 186.69 106.68) (width 0.4064) (layer F.Cu) (net 10))
+  (segment (start 186.69 104.14) (end 186.69 106.68) (width 0.3048) (layer F.Cu) (net 10))
   (segment (start 186.69 104.14) (end 185.039 104.14) (width 0.4064) (layer F.Cu) (net 10))
   (segment (start 179.07 106.68) (end 179.07 106.045) (width 0.4064) (layer F.Cu) (net 11))
@@
   (segment (start 158.75 108.585) (end 158.115 109.22) (width 0.4064) (layer F.Cu) (net 13))
   (segment (start 160.84 106.68) (end 158.75 106.68) (width 0.4064) (layer F.Cu) (net 13))
-  (segment (start 151.13 106.68) (end 151.13 111.76) (width 0.4064) (layer F.Cu) (net 14))
+  (segment (start 151.13 106.68) (end 151.13 111.76) (width 0.4064) (layer F.Cu) (net 14) (status 10))
   (segment (start 151.765 112.395) (end 154.78 112.395) (width 0.4064) (layer B.Cu) (net 14))
   (via (at 151.765 112.395) (size 0.6858) (drill 0.3302) (layers F.Cu B.Cu) (net 14))
   (segment (start 151.13 111.76) (end 151.765 112.395) (width 0.4064) (layer F.Cu) (net 14))
-  (segment (start 151.13 106.68) (end 152.92 106.68) (width 0.4064) (layer F.Cu) (net 14))
+  (segment (start 151.13 106.68) (end 152.92 106.68) (width 0.4064) (layer F.Cu) (net 14) (status 10))
+  (zone (net 1) (net_name GND) (layer F.Cu) (hatch edge 0.508)
+    (connect_pads (clearance 0.35))
+    (min_thickness 0.2)
+    (fill yes (arc_segments 32) (thermal_gap 0.508) (thermal_bridge_width 0.508))
+    (polygon
+      (pts
+        (xy 195.58 120.65) (xy 139.7 120.65) (xy 139.7 90.17) (xy 195.58 90.17)
+      )
+    )
+  )
 )
