File: projects/translator/design_files/project.sch (KiCad schematic (older format))
At the start: 10 parts, among them CON1 AVR-ISP-6, CON2 AVR-ISP-6, U1 TXB0104D, U2 MIC5225-3.3

Commit message: updates
Parts:
- C1: renamed from C6; footprint Capacitors_SMD:C_0805 -> footprints:C_0805
- C2: renamed from C7; footprint Capacitors_SMD:C_0603 -> footprints:C_0603
- C3: renamed from C8; footprint Capacitors_SMD:C_0805 -> footprints:C_0805
- CON1, CON2: footprint Pin_Headers:Pin_Header_Straight_2x03_Pitch2.54mm -> footprints:Pin_Header_Straight_2x03_Pitch2.54mm
- R2: renamed from R9; footprint Resistors_SMD:R_0603 -> footprints:R_0603
- U1: footprint Housings_SOIC:SOIC-14_3.9x8.7mm_Pitch1.27mm -> footprints:SOIC-14_3.9x8.7mm_Pitch1.27mm
- U2: footprint TO_SOT_Packages_SMD:SOT-23-5 -> footprints:SOT-23-5
Connections:
- net labels removed: VBUS
Changed lines of the file:
@@
 encoding utf-8
 Sheet 1 1
-Title "32u4"
+Title "ISP Translator"
 Date ""
 Rev ""
@@
 $EndDescr
 $Comp
-L +3V3 #PWR01
-U 1 1 5B3FDCB5
-P 2000 850
-F 0 "#PWR01" H 2000 700 50  0001 C CNN
-F 1 "+3V3" H 2000 990 50  0000 C CNN
-F 2 "" H 2000 850 50  0001 C CNN
-F 3 "" H 2000 850 50  0001 C CNN
-	1    2000 850
-	-1   0    0    1
-$EndComp
-$Comp
-L GND #PWR02
+L GND #PWR01
 U 1 1 5B3FDCF5
-P 2450 850
-F 0 "#PWR02" H 2450 600 50  0001 C CNN
-F 1 "GND" H 2450 700 50  0000 C CNN
-F 2 "" H 2450 850 50  0001 C CNN
-F 3 "" H 2450 850 50  0001 C CNN
-	1    2450 850
-	1    0    0    -1
-$EndComp
-$Comp
-L PWR_FLAG #FLG03
+P 1600 850
+F 0 "#PWR01" H 1600 600 50  0001 C CNN
+F 1 "GND" H 1600 700 50  0000 C CNN
+F 2 "" H 1600 850 50  0001 C CNN
+F 3 "" H 1600 850 50  0001 C CNN
+	1    1600 850
+	1    0    0    -1
+$EndComp
+$Comp
+L PWR_FLAG #FLG02
 U 1 1 5B3FDD3A
 P 1200 850
-F 0 "#FLG03" H 1200 925 50  0001 C CNN
+F 0 "#FLG02" H 1200 925 50  0001 C CNN
 F 1 "PWR_FLAG" H 1200 1000 50  0000 C CNN
 F 2 "" H 1200 850 50  0001 C CNN
@@
 $EndComp
 $Comp
-L PWR_FLAG #FLG04
-U 1 1 5B3FDD50
-P 2000 850
-F 0 "#FLG04" H 2000 925 50  0001 C CNN
-F 1 "PWR_FLAG" H 2000 1000 50  0000 C CNN
-F 2 "" H 2000 850 50  0001 C CNN
-F 3 "" H 2000 850 50  0001 C CNN
-	1    2000 850
-	1    0    0    -1
-$EndComp
-$Comp
-L PWR_FLAG #FLG05
+L PWR_FLAG #FLG03
 U 1 1 5B3FDD67
-P 2450 850
-F 0 "#FLG05" H 2450 925 50  0001 C CNN
-F 1 "PWR_FLAG" H 2450 1000 50  0000 C CNN
-F 2 "" H 2450 850 50  0001 C CNN
-F 3 "" H 2450 850 50  0001 C CNN
-	1    2450 850
+P 1600 850
+F 0 "#FLG03" H 1600 925 50  0001 C CNN
+F 1 "PWR_FLAG" H 1600 1000 50  0000 C CNN
+F 2 "" H 1600 850 50  0001 C CNN
+F 3 "" H 1600 850 50  0001 C CNN
+	1    1600 850
 	1    0    0    -1
 $EndComp
@@
 F 0 "U2" H 1550 2025 50  0000 C CNN
 F 1 "MIC5225-3.3" H 1700 2025 50  0000 L CNN
-F 2 "TO_SOT_Packages_SMD:SOT-23-5" H 1700 2125 50  0001 C CNN
+F 2 "footprints:SOT-23-5" H 1700 2125 50  0001 C CNN
 F 3 "" H 1700 1800 50  0001 C CNN
 	1    1700 1800
@@
 $EndComp
 $Comp
-L GND #PWR06
+L GND #PWR04
 U 1 1 5B3FF1A9
 P 1700 2350
-F 0 "#PWR06" H 1700 2100 50  0001 C CNN
+F 0 "#PWR04" H 1700 2100 50  0001 C CNN
 F 1 "GND" H 1700 2200 50  0000 C CNN
 F 2 "" H 1700 2350 50  0001 C CNN
@@
 $EndComp
 $Comp
-L R R9
+L R R2
 U 1 1 5B3FF1C8
 P 1200 1800
-F 0 "R9" V 1280 1800 50  0000 C CNN
+F 0 "R2" V 1280 1800 50  0000 C CNN
 F 1 "100K" V 1200 1800 50  0000 C CNN
-F 2 "Resistors_SMD:R_0603" V 1130 1800 50  0001 C CNN
+F 2 "footprints:R_0603" V 1130 1800 50  0001 C CNN
 F 3 "" H 1200 1800 50  0001 C CNN
 	1    1200 1800
@@
 $EndComp
 $Comp
-L C C6
+L C C1
 U 1 1 5B3FF285
 P 950 2200
-F 0 "C6" H 975 2300 50  0000 L CNN
+F 0 "C1" H 975 2300 50  0000 L CNN
 F 1 "10uF" H 975 2100 50  0000 L CNN
-F 2 "Capacitors_SMD:C_0805" H 988 2050 50  0001 C CNN
+F 2 "footprints:C_0805" H 988 2050 50  0001 C CNN
 F 3 "" H 950 2200 50  0001 C CNN
 	1    950  2200
@@
 $EndComp
 $Comp
-L C C8
+L C C3
 U 1 1 5B3FF2D3
 P 2100 2200
-F 0 "C8" H 2125 2300 50  0000 L CNN
+F 0 "C3" H 2125 2300 50  0000 L CNN
 F 1 "10uF" H 2125 2100 50  0000 L CNN
-F 2 "Capacitors_SMD:C_0805" H 2138 2050 50  0001 C CNN
+F 2 "footprints:C_0805" H 2138 2050 50  0001 C CNN
 F 3 "" H 2100 2200 50  0001 C CNN
 	1    2100 2200
@@
 $EndComp
 $Comp
-L C C7
+L C C2
 U 1 1 5B3FF331
 P 2400 2200
-F 0 "C7" H 2425 2300 50  0000 L CNN
+F 0 "C2" H 2425 2300 50  0000 L CNN
 F 1 "1uF" H 2425 2100 50  0000 L CNN
-F 2 "Capacitors_SMD:C_0603" H 2438 2050 50  0001 C CNN
+F 2 "footprints:C_0603" H 2438 2050 50  0001 C CNN
 F 3 "" H 2400 2200 50  0001 C CNN
 	1    2400 2200
@@
 $EndComp
 $Comp
-L +3V3 #PWR07
+L +3V3 #PWR05
 U 1 1 5B3FF64D
 P 2400 1700
-F 0 "#PWR07" H 2400 1550 50  0001 C CNN
+F 0 "#PWR05" H 2400 1550 50  0001 C CNN
 F 1 "+3V3" H 2400 1840 50  0000 C CNN
 F 2 "" H 2400 1700 50  0001 C CNN
@@
 F 0 "CON1" H 6995 4140 50  0000 C CNN
 F 1 "AVR-ISP-6" H 6835 3670 50  0000 L BNN
-F 2 "Pin_Headers:Pin_Header_Straight_2x03_Pitch2.54mm" V 6580 3940 50  0001 C CNN
+F 2 "footprints:Pin_Header_Straight_2x03_Pitch2.54mm" V 6580 3940 50  0001 C CNN
 F 3 "" H 7075 3900 50  0001 C CNN
 	1    7100 3900
@@
 MOSI_5V
 $Comp
-L GND #PWR08
+L GND #PWR06
 U 1 1 5B5296C8
 P 7750 4000
-F 0 "#PWR08" H 7750 3750 50  0001 C CNN
+F 0 "#PWR06" H 7750 3750 50  0001 C CNN
 F 1 "GND" H 7750 3850 50  0000 C CNN
 F 2 "" H 7750 4000 50  0001 C CNN
@@
 F 0 "U1" H 4675 4555 50  0000 C CNN
 F 1 "TXB0104D" H 5300 4550 50  0000 C CNN
-F 2 "Housings_SOIC:SOIC-14_3.9x8.7mm_Pitch1.27mm" H 5000 3050 50  0001 C CNN
+F 2 "footprints:SOIC-14_3.9x8.7mm_Pitch1.27mm" H 5000 3050 50  0001 C CNN
 F 3 "" H 5060 3995 50  0001 C CNN
 	1    4950 3900
@@
 F 0 "CON2" H 2695 4040 50  0000 C CNN
 F 1 "AVR-ISP-6" H 2535 3570 50  0000 L BNN
-F 2 "Pin_Headers:Pin_Header_Straight_2x03_Pitch2.54mm" V 2280 3840 50  0001 C CNN
+F 2 "footprints:Pin_Header_Straight_2x03_Pitch2.54mm" V 2280 3840 50  0001 C CNN
 F 3 "" H 2775 3800 50  0001 C CNN
 	1    2800 3800
@@
 MOSI_3V
 $Comp
-L GND #PWR09
+L GND #PWR07
 U 1 1 5B565482
 P 3450 3900
-F 0 "#PWR09" H 3450 3650 50  0001 C CNN
+F 0 "#PWR07" H 3450 3650 50  0001 C CNN
 F 1 "GND" H 3450 3750 50  0000 C CNN
 F 2 "" H 3450 3900 50  0001 C CNN
@@
 	4150 4200 4550 4200
 $Comp
-L GND #PWR010
+L GND #PWR08
 U 1 1 5B565A1F
 P 4950 4600
-F 0 "#PWR010" H 4950 4350 50  0001 C CNN
+F 0 "#PWR08" H 4950 4350 50  0001 C CNN
 F 1 "GND" H 4950 4450 50  0000 C CNN
 F 2 "" H 4950 4600 50  0001 C CNN
@@
 $EndComp
 $Comp
-L +3V3 #PWR011
+L +3V3 #PWR09
 U 1 1 5B565A78
 P 4850 3200
-F 0 "#PWR011" H 4850 3050 50  0001 C CNN
+F 0 "#PWR09" H 4850 3050 50  0001 C CNN
 F 1 "+3V3" H 4850 3340 50  0000 C CNN
 F 2 "" H 4850 3200 50  0001 C CNN
@@
 $EndComp
 $Comp
-L VBUS #PWR012
-U 1 1 5B565AAC
-P 5050 3200
-F 0 "#PWR012" H 5050 3050 50  0001 C CNN
-F 1 "VBUS" H 5050 3350 50  0000 C CNN
-F 2 "" H 5050 3200 50  0001 C CNN
-F 3 "" H 5050 3200 50  0001 C CNN
-	1    5050 3200
-	1    0    0    -1
-$EndComp
-$Comp
-L +3V3 #PWR013
+L +3V3 #PWR010
 U 1 1 5B565AFD
 P 3450 3700
-F 0 "#PWR013" H 3450 3550 50  0001 C CNN
+F 0 "#PWR010" H 3450 3550 50  0001 C CNN
 F 1 "+3V3" H 3450 3840 50  0000 C CNN
 F 2 "" H 3450 3700 50  0001 C CNN
@@
 ~RESET_3V
 $Comp
-L +3V3 #PWR014
+L +3V3 #PWR011
 U 1 1 5B565F71
 P 4300 3200
-F 0 "#PWR014" H 4300 3050 50  0001 C CNN
+F 0 "#PWR011" H 4300 3050 50  0001 C CNN
 F 1 "+3V3" H 4300 3340 50  0000 C CNN
 F 2 "" H 4300 3200 50  0001 C CNN
@@
 	4300 3400 4550 3400
 $Comp
-L +5V #PWR015
+L +5V #PWR012
 U 1 1 5B5665EC
 P 1200 850
-F 0 "#PWR015" H 1200 700 50  0001 C CNN
+F 0 "#PWR012" H 1200 700 50  0001 C CNN
 F 1 "+5V" H 1200 990 50  0000 C CNN
 F 2 "" H 1200 850 50  0001 C CNN
@@
 $EndComp
 $Comp
-L +5V #PWR016
+L +5V #PWR013
 U 1 1 5B566662
 P 950 1800
-F 0 "#PWR016" H 950 1650 50  0001 C CNN
+F 0 "#PWR013" H 950 1650 50  0001 C CNN
 F 1 "+5V" H 950 1940 50  0000 C CNN
 F 2 "" H 950 1800 50  0001 C CNN
@@
 $EndComp
 $Comp
-L +5V #PWR017
+L +5V #PWR014
 U 1 1 5B5666CE
 P 7750 3800
-F 0 "#PWR017" H 7750 3650 50  0001 C CNN
+F 0 "#PWR014" H 7750 3650 50  0001 C CNN
 F 1 "+5V" H 7750 3940 50  0000 C CNN
 F 2 "" H 7750 3800 50  0001 C CNN
@@
 	2700 2350 2700 2300
 Connection ~ 2400 2350
+$Comp
+L +5V #PWR015
+U 1 1 5B567090
+P 5050 3200
+F 0 "#PWR015" H 5050 3050 50  0001 C CNN
+F 1 "+5V" H 5050 3340 50  0000 C CNN
+F 2 "" H 5050 3200 50  0001 C CNN
+F 3 "" H 5050 3200 50  0001 C CNN
+	1    5050 3200
+	1    0    0    -1
+$EndComp
 $EndSCHEMATC
