File: projects/Beetje/design_files_press/project.kicad_pcb (KiCad board)
At the start: 2 copper layers, 25.4 x 25.4 mm, 10 parts, among them J2 Conn_01x06, J4 Conn_01x08, U2 MPL3115A

Commit message: Updates
Parts:
- U2: footprint Housings_LGA:LGA-8_3x5mm_Pitch1.25mm -> footprints:MPL3115A
Changed lines of the file:
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@@
-(kicad_pcb (version 4) (host pcbnew 4.0.7)
+(kicad_pcb (version 4) (host pcbnew 4.0.6)
   (general
     (links 17)
     (no_connects 0)
-    (area 142.164999 86.284999 167.715001 111.835001)
+    (area 125.73 78.580001 182.145715 114.400001)
     (thickness 1.6)
     (drawings 21)
@@
   )
   (setup
-    (last_trace_width 0.3048)
+    (last_trace_width 0.25)
     (user_trace_width 0.3048)
     (user_trace_width 0.4064)
@@
     (pad 8 thru_hole oval (at 0 17.78 270) (size 1.7 1.7) (drill 1) (layers *.Cu *.Mask)
       (net 2 VBUS))
-  )
-  (module Housings_LGA:LGA-8_3x5mm_Pitch1.25mm (layer F.Cu)
-    (at 154.94 99.06)
-    (descr LGA-8)
-    (tags "lga land grid array")
-    (attr smd)
-    (fp_text reference U2 (at 0 -3.65) (layer F.SilkS) hide
-      (effects (font (size 1 1) (thickness 0.15)))
-    )
-    (fp_text value MPL3115A (at 0 3.65) (layer F.Fab)
-      (effects (font (size 1 1) (thickness 0.15)))
-    )
-    (fp_text user %R (at 0 0) (layer F.Fab)
-      (effects (font (size 0.5 0.5) (thickness 0.075)))
-    )
-    (fp_line (start 1.5 -2.5) (end 1.5 2.5) (layer F.Fab) (width 0.1))
-    (fp_line (start 1.5 2.5) (end -1.5 2.5) (layer F.Fab) (width 0.1))
-    (fp_line (start -1.5 2.5) (end -1.5 -1.75) (layer F.Fab) (width 0.1))
-    (fp_line (start -1.5 -1.75) (end -0.75 -2.5) (layer F.Fab) (width 0.1))
-    (fp_line (start -0.75 -2.5) (end 1.5 -2.5) (layer F.Fab) (width 0.1))
-    (fp_line (start 1.15 -2.6) (end 1.65 -2.6) (layer F.SilkS) (width 0.12))
-    (fp_line (start 1.65 -2.6) (end 1.65 -2.1) (layer F.SilkS) (width 0.12))
-    (fp_line (start 1.65 2.1) (end 1.65 2.6) (layer F.SilkS) (width 0.12))
-    (fp_line (start 1.65 2.6) (end 1.15 2.6) (layer F.SilkS) (width 0.12))
-    (fp_line (start -1.15 2.6) (end -1.65 2.6) (layer F.SilkS) (width 0.12))
-    (fp_line (start -1.65 2.6) (end -1.65 2.1) (layer F.SilkS) (width 0.12))
-    (fp_line (start -1.55 -2.6) (end -0.6 -2.6) (layer F.SilkS) (width 0.12))
-    (fp_line (start -1.8 -2.75) (end 1.8 -2.75) (layer F.CrtYd) (width 0.05))
-    (fp_line (start -1.8 -2.75) (end -1.8 2.75) (layer F.CrtYd) (width 0.05))
-    (fp_line (start 1.8 2.75) (end 1.8 -2.75) (layer F.CrtYd) (width 0.05))
-    (fp_line (start 1.8 2.75) (end -1.8 2.75) (layer F.CrtYd) (width 0.05))
-    (pad 4 smd rect (at -1.075 1.875) (size 0.95 0.55) (layers F.Cu F.Paste F.Mask)
-      (net 14 VCC))
-    (pad 1 smd rect (at -1.075 -1.875) (size 0.95 0.55) (layers F.Cu F.Paste F.Mask)
-      (net 14 VCC))
-    (pad 2 smd rect (at -1.075 -0.625) (size 0.95 0.55) (layers F.Cu F.Paste F.Mask)
-      (net 15 "Net-(C4-Pad1)"))
-    (pad 3 smd rect (at -1.075 0.625) (size 0.95 0.55) (layers F.Cu F.Paste F.Mask)
-      (net 1 GND))
-    (pad 8 smd rect (at 1.075 -1.875) (size 0.95 0.55) (layers F.Cu F.Paste F.Mask)
-      (net 6 /SCL))
-    (pad 7 smd rect (at 1.075 -0.625) (size 0.95 0.55) (layers F.Cu F.Paste F.Mask)
-      (net 7 /SDA))
-    (pad 6 smd rect (at 1.075 0.625) (size 0.95 0.55) (layers F.Cu F.Paste F.Mask)
-      (net 4 /D10))
-    (pad 5 smd rect (at 1.075 1.875) (size 0.95 0.55) (layers F.Cu F.Paste F.Mask)
-      (net 5 /D9))
-    (model ${KISYS3DMOD}/Housings_LGA.3dshapes/LGA-8_3x5mm_Pitch1.25mm.wrl
-      (at (xyz 0 0 0))
-      (scale (xyz 1 1 1))
-      (rotate (xyz 0 0 0))
-    )
   )
   (module Capacitors_SMD:C_0805 (layer F.Cu)
@@
       (xy -1.29032 -1.15062)) (layer B.SilkS) (width 0.00254))
   )
+  (module footprints:MPL3115A (layer F.Cu)
+    (at 154.94 99.06)
+    (descr LGA-8)
+    (tags "lga land grid array")
+    (attr smd)
+    (fp_text reference U2 (at 0 -3.65) (layer F.SilkS) hide
+      (effects (font (size 1 1) (thickness 0.15)))
+    )
+    (fp_text value MPL3115A (at 0 3.65) (layer F.Fab)
+      (effects (font (size 1 1) (thickness 0.15)))
+    )
+    (fp_circle (center 0 1.25) (end 0.25 1.5) (layer F.SilkS) (width 0.1))
+    (fp_line (start -0.5 -1.5) (end -0.5 -1.25) (layer F.SilkS) (width 0.1))
+    (fp_line (start -0.5 -1.25) (end -0.25 -1.5) (layer F.SilkS) (width 0.1))
+    (fp_line (start -0.25 -1.5) (end -0.5 -1.5) (layer F.SilkS) (width 0.1))
+    (fp_text user %R (at 0 0) (layer F.Fab)
+      (effects (font (size 0.5 0.5) (thickness 0.075)))
+    )
+    (fp_line (start 1.5 -2.5) (end 1.5 2.5) (layer F.Fab) (width 0.1))
+    (fp_line (start 1.5 2.5) (end -1.5 2.5) (layer F.Fab) (width 0.1))
+    (fp_line (start -1.5 2.5) (end -1.5 -1.75) (layer F.Fab) (width 0.1))
+    (fp_line (start -1.5 -1.75) (end -0.75 -2.5) (layer F.Fab) (width 0.1))
+    (fp_line (start -0.75 -2.5) (end 1.5 -2.5) (layer F.Fab) (width 0.1))
+    (fp_line (start 1.15 -2.6) (end 1.65 -2.6) (layer F.SilkS) (width 0.12))
+    (fp_line (start 1.65 -2.6) (end 1.65 -2.1) (layer F.SilkS) (width 0.12))
+    (fp_line (start 1.65 2.1) (end 1.65 2.6) (layer F.SilkS) (width 0.12))
+    (fp_line (start 1.65 2.6) (end 1.15 2.6) (layer F.SilkS) (width 0.12))
+    (fp_line (start -1.15 2.6) (end -1.65 2.6) (layer F.SilkS) (width 0.12))
+    (fp_line (start -1.65 2.6) (end -1.65 2.1) (layer F.SilkS) (width 0.12))
+    (fp_line (start -1.55 -2.6) (end -0.6 -2.6) (layer F.SilkS) (width 0.12))
+    (fp_line (start -1.8 -2.75) (end 1.8 -2.75) (layer F.CrtYd) (width 0.05))
+    (fp_line (start -1.8 -2.75) (end -1.8 2.75) (layer F.CrtYd) (width 0.05))
+    (fp_line (start 1.8 2.75) (end 1.8 -2.75) (layer F.CrtYd) (width 0.05))
+    (fp_line (start 1.8 2.75) (end -1.8 2.75) (layer F.CrtYd) (width 0.05))
+    (pad 4 smd rect (at -1.075 1.875) (size 0.95 0.55) (layers F.Cu F.Paste F.Mask)
+      (net 14 VCC))
+    (pad 1 smd rect (at -1.075 -1.875) (size 0.95 0.55) (layers F.Cu F.Paste F.Mask)
+      (net 14 VCC))
+    (pad 2 smd rect (at -1.075 -0.625) (size 0.95 0.55) (layers F.Cu F.Paste F.Mask)
+      (net 15 "Net-(C4-Pad1)"))
+    (pad 3 smd rect (at -1.075 0.625) (size 0.95 0.55) (layers F.Cu F.Paste F.Mask)
+      (net 1 GND))
+    (pad 8 smd rect (at 1.075 -1.875) (size 0.95 0.55) (layers F.Cu F.Paste F.Mask)
+      (net 6 /SCL))
+    (pad 7 smd rect (at 1.075 -0.625) (size 0.95 0.55) (layers F.Cu F.Paste F.Mask)
+      (net 7 /SDA))
+    (pad 6 smd rect (at 1.075 0.625) (size 0.95 0.55) (layers F.Cu F.Paste F.Mask)
+      (net 4 /D10))
+    (pad 5 smd rect (at 1.075 1.875) (size 0.95 0.55) (layers F.Cu F.Paste F.Mask)
+      (net 5 /D9))
+    (model ${KISYS3DMOD}/Housings_LGA.3dshapes/LGA-8_3x5mm_Pitch1.25mm.wrl
+      (at (xyz 0 0 0))
+      (scale (xyz 1 1 1))
+      (rotate (xyz 0 0 0))
+    )
+  )
   (gr_text "I2C: 0X60\nINT1: D10\nINT2: D9" (at 151.13 105.41) (layer F.SilkS)

Commit message: Updates
Parts:
- R1, R2: value 1K -> 4K7
Changed lines of the file:
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@@
     (links 17)
     (no_connects 0)
-    (area 125.73 78.580001 182.145715 114.400001)
+    (area 142.164999 86.284999 167.715001 111.835001)
     (thickness 1.6)
     (drawings 21)
@@
     (34 B.Paste user)
     (35 F.Paste user)
-    (36 B.SilkS user)
+    (36 B.SilkS user hide)
     (37 F.SilkS user)
     (38 B.Mask user)
@@
       (effects (font (size 1 1) (thickness 0.15)))
     )
-    (fp_text value 1K (at 0 1.5 180) (layer F.Fab)
+    (fp_text value 4K7 (at 0 1.5 180) (layer F.Fab)
       (effects (font (size 1 1) (thickness 0.15)))
     )
@@
       (effects (font (size 1 1) (thickness 0.15)))
     )
-    (fp_text value 1K (at 0 1.5 180) (layer F.Fab)
-      (effects (font (size 1 1) (thickness 0.15)))
-    )
+    (fp_text value 4K7 (at 0 1.5 180) (layer F.Fab)
+      (effects (font (size 1 1) (thickness 0.15)))
+    )
