File: projects/Beetje/design_files_press/project.sch (KiCad schematic (older format))
At the start: 8 parts, among them J2 Conn_01x06, J4 Conn_01x08, U2 MPL3115A

Commit message: Updates
Parts:
- U2: footprint Housings_LGA:LGA-8_3x5mm_Pitch1.25mm -> footprints:MPL3115A
Changed lines of the file:
@@
 F 0 "U2" H 6700 4450 50  0000 C CNN
 F 1 "MPL3115A" H 7600 3650 50  0000 C CNN
-F 2 "Housings_LGA:LGA-8_3x5mm_Pitch1.25mm" H 7200 4050 50  0001 C CIN
+F 2 "footprints:MPL3115A" H 7200 4050 50  0001 C CIN
 F 3 "" H 7200 4050 50  0001 C CNN
 	1    7200 4050

Commit message: Updates
Parts:
- R1, R2: value 1K -> 4K7
Changed lines of the file:
@@
 P 8200 3950
 F 0 "R2" V 8280 3950 50  0000 C CNN
-F 1 "1K" V 8200 3950 50  0000 C CNN
+F 1 "4K7" V 8200 3950 50  0000 C CNN
 F 2 "Resistors_SMD:R_0603" V 8130 3950 50  0001 C CNN
 F 3 "" H 8200 3950 50  0001 C CNN
@@
 P 8200 3800
 F 0 "R1" V 8280 3800 50  0000 C CNN
-F 1 "1K" V 8200 3800 50  0000 C CNN
+F 1 "4K7" V 8200 3800 50  0000 C CNN
 F 2 "Resistors_SMD:R_0603" V 8130 3800 50  0001 C CNN
 F 3 "" H 8200 3800 50  0001 C CNN
