File: projects/Beetje/design_files_LiPo/project V1.kicad_pcb (KiCad board)
At the start: 2 copper layers, 25.4 x 25.4 mm, 18 parts, among them J1 JSTSH, J2 Beetje_Bottom, J3 JSTPH, J4 Beetje_Top, SW1 SW_SPDT, U1 MCP73833

Commit message: Updates
Parts:
- removed D4: D, footprints:D_SOD-123F
- removed R4: 10K, footprints:R_0805_HandSoldering
- removed R5: 4K7, footprints:R_0805_HandSoldering
- C1, C2: footprint Capacitors_SMD:C_1206 -> footprints:C_0805
- D1: value PWR -> CHG
- D3: value CHG -> D_TVS; footprint footprints:LED_0805_HandSoldering -> Diodes_SMD:D_0805
- R3: value 1K -> 10K
- U1: value MCP73833 -> MCP73831; footprint Housings_SSOP:MSOP-10_3x3mm_Pitch0.5mm -> footprints:SOT-23-5_HandSoldering
- moved D1 27.1 mm to (146.1, 115.6), turned to 90 degrees
- moved R1 20.0 mm to (146.1, 110.5), turned to 90 degrees
- moved R3 18.5 mm to (131.4, 99.1)
- moved D3 18.1 mm to (132.1, 104.1), turned to 90 degrees
- moved C2 9.44 mm to (137.2, 97.2), turned to 180 degrees
- moved J1 4.20 mm to (126.4, 99.7), turned to 0 degrees
- moved C1 1.91 mm to (137.2, 106.0)
- moved U1 1.42 mm to (137.2, 101.6), turned to 0 degrees
- moved J3 0.90 mm to (135.9, 109.9)
- turned D2 to 90 degrees
- turned R2 to 90 degrees
Connections:
- D2 pad 1: Net-(D2-Pad1) -> GND
- D2 pad 2: VBUS -> Net-(D2-Pad2)
- D3 pad 1: Net-(D3-Pad1) -> Net-(C2-Pad1)
- D3 pad 2: VBUS -> GND
- J3 pad 1: Net-(C2-Pad1) -> GND
- J3 pad 2: GND -> Net-(C2-Pad1)
- R1 pad 1: Net-(R1-Pad1) -> Net-(D1-Pad1)
- R1 pad 2: Net-(D1-Pad1) -> Net-(R1-Pad2)
- R2 pad 1: Net-(R2-Pad1) -> Net-(D2-Pad2)
- R2 pad 2: Net-(D2-Pad1) -> Net-(R1-Pad2)
- R3 pad 2: Net-(D3-Pad1) -> GND
- SW1 pad 2: VCC -> Net-(C2-Pad1)
- SW1 pad 3: Net-(D4-Pad1) -> +BATT
- U1 pad 1: VBUS -> Net-(R1-Pad2)
- U1 pad 2: VBUS -> GND
- U1 pad 3: Net-(R2-Pad1) -> Net-(C2-Pad1)
- U1 pad 4: Net-(R3-Pad1) -> VBUS
- U1 pad 5: GND -> Net-(R3-Pad1)
Routing:
- net VCC: track 33.3 -> 0.00 mm, vias 1 -> 0
- net Net-(R1-Pad2): track 0.00 -> 27.8 mm, vias 0 -> 2
- net +BATT: track 0.00 -> 19.9 mm
- net VBUS: track 59.5 -> 46.2 mm, vias 0 -> 4
- net Net-(C2-Pad1): track 32.9 -> 44.4 mm
- net Net-(R2-Pad1): track 8.86 -> 0.00 mm
- net GND: track 55.0 -> 62.8 mm, vias 7 -> 5
- net Net-(R1-Pad1): track 7.08 -> 0.00 mm
- net Net-(R4-Pad1): track 5.13 -> 0.00 mm
- net Net-(D1-Pad1): track 2.38 -> 7.19 mm
- net Net-(R3-Pad1): track 14.9 -> 18.8 mm, vias 0 -> 2
- net Net-(R5-Pad1): track 2.71 -> 0.00 mm
- net Net-(D4-Pad1): track 2.49 -> 0.00 mm
- net Net-(D3-Pad1): track 2.38 -> 0.00 mm
- net Net-(D2-Pad2): track 0.00 -> 2.38 mm
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- added copper zone on B.Cu, net Net-(C2-Pad1)
- added copper zone on F.Cu, net Net-(C2-Pad1)
- added copper zone on B.Cu, net VBUS
- added copper zone on F.Cu, net VBUS
Other:
- board text added: "R3: 10K= 100 mA 5K = 200 mA 2K = 500 mA 1K = 1000 mA"
- board text added: "Rev 0.3 Sep 2018"
- board text removed: "R5: 10K= 100 mA 5K = 200 mA 2K = 500 mA 1K = 1000 mA"
- board text removed: "Rev 0.4 Apr 2020"
