File: projects/Beetje/design_files_LiPo/project.kicad_pcb (KiCad board)
At the start: 2 copper layers, 25.4 x 25.4 mm, 15 parts, among them J1 JSTSH, J2 Beetje_Bottom, J3 JSTPH, J4 Beetje_Top, SW1 SW_SPDT, U1 MCP73831

Commit message: Updates
Parts:
- D1, D2: footprint footprints:R_0805_HandSoldering -> footprints:LED_0805_HandSoldering
Other:
- board text added: "Rev 0.3 Sep 2018"
- board text removed: "Rev 0.2 Sep 2018"

Commit message: Updates
Parts:
- D3: value D -> D_TVS; footprint footprints:D_SOD-123F -> Diodes_SMD:D_0805
- moved D3 0.90 mm to (132.1, 104.1), turned to 90 degrees
Connections:
- D3 pad 2: Net-(D3-Pad2) -> GND
- J1 pad 2: Net-(D3-Pad2) -> Net-(C2-Pad1)
- J3 pad 2: Net-(D3-Pad2) -> Net-(C2-Pad1)
Routing:
- net Net-(D3-Pad2): track 21.8 -> 0.00 mm
- net Net-(C2-Pad1): track 26.4 -> 44.4 mm, vias 3 -> 0
- net GND: track 59.8 -> 62.8 mm

Commit message: Updates
Parts:
- added D4: D, footprints:D_SOD-123F, F.Cu at (141.6, 97.4)
- added R4: 10K, footprints:R_0805_HandSoldering, F.Cu at (131.1, 99.6)
- added R5: 4K7, footprints:R_0805_HandSoldering, F.Cu at (136.7, 99.6)
- C1, C2: footprint footprints:C_0805 -> Capacitors_SMD:C_1206
- D1: value CHG -> PWR
- D3: value D_TVS -> CHG; footprint Diodes_SMD:D_0805 -> footprints:LED_0805_HandSoldering
- J2: footprint footprints:Beetje_Bottom -> beetje_footprints:Beetje_Bottom
- J4: footprint footprints:Beetje_Top -> beetje_footprints:Beetje_Top
- R3: value 10K -> 1K
- U1: value MCP73831 -> MCP73833; footprint footprints:SOT-23-5_HandSoldering -> Housings_SSOP:MSOP-10_3x3mm_Pitch0.5mm
- moved D1 27.1 mm to (126.0, 97.3), turned to 180 degrees
- moved R1 20.0 mm to (131.1, 97.3), turned to 180 degrees
- moved R3 18.5 mm to (146.1, 110.5)
- moved D3 18.1 mm to (146.1, 115.6), turned to 270 degrees
- moved C2 9.44 mm to (134.0, 106.0), turned to 0 degrees
- moved J1 4.20 mm to (128.1, 103.5), turned to 270 degrees
- moved C1 1.91 mm to (139.1, 106.0)
- moved U1 1.42 mm to (136.5, 102.9), turned to 180 degrees
- moved J3 0.90 mm to (135.3, 110.5)
- turned D2 to 270 degrees
- turned R2 to 270 degrees
Connections:
- D2 pad 1: GND -> Net-(D2-Pad1)
- D2 pad 2: Net-(D2-Pad2) -> VBUS
- D3 pad 1: Net-(C2-Pad1) -> Net-(D3-Pad1)
- D3 pad 2: GND -> VBUS
- J3 pad 1: GND -> Net-(C2-Pad1)
- J3 pad 2: Net-(C2-Pad1) -> GND
- R1 pad 1: Net-(D1-Pad1) -> Net-(R1-Pad1)
- R1 pad 2: Net-(R1-Pad2) -> Net-(D1-Pad1)
- R2 pad 1: Net-(D2-Pad2) -> Net-(R2-Pad1)
- R2 pad 2: Net-(R1-Pad2) -> Net-(D2-Pad1)
- R3 pad 2: GND -> Net-(D3-Pad1)
- SW1 pad 2: Net-(C2-Pad1) -> VCC
- SW1 pad 3: +BATT -> Net-(D4-Pad1)
- U1 pad 1: Net-(R1-Pad2) -> VBUS
- U1 pad 2: GND -> VBUS
- U1 pad 3: Net-(C2-Pad1) -> Net-(R2-Pad1)
- U1 pad 4: VBUS -> Net-(R3-Pad1)
- U1 pad 5: Net-(R3-Pad1) -> GND
Routing:
- net VCC: track 0.00 -> 33.3 mm, vias 0 -> 1
- net Net-(R1-Pad2): track 27.8 -> 0.00 mm, vias 2 -> 0
- net +BATT: track 19.9 -> 0.00 mm
- net VBUS: track 46.2 -> 59.5 mm, vias 4 -> 0
- net Net-(C2-Pad1): track 44.4 -> 32.9 mm
- net Net-(R2-Pad1): track 0.00 -> 8.86 mm
- net GND: track 62.8 -> 55.0 mm, vias 5 -> 7
- net Net-(R1-Pad1): track 0.00 -> 7.08 mm
- net Net-(R4-Pad1): track 0.00 -> 5.13 mm
- net Net-(D1-Pad1): track 7.19 -> 2.38 mm
- net Net-(R3-Pad1): track 18.8 -> 14.9 mm, vias 2 -> 0
- net Net-(R5-Pad1): track 0.00 -> 2.71 mm
- net Net-(D4-Pad1): track 0.00 -> 2.49 mm
- net Net-(D3-Pad1): track 0.00 -> 2.38 mm
- net Net-(D2-Pad2): track 2.38 -> 0.00 mm
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- removed copper zone on B.Cu, net Net-(C2-Pad1)
- removed copper zone on F.Cu, net Net-(C2-Pad1)
- removed copper zone on B.Cu, net VBUS
- removed copper zone on F.Cu, net VBUS
Other:
- board text added: "R5: 10K= 100 mA 5K = 200 mA 2K = 500 mA 1K = 1000 mA"
- board text added: "Rev 0.5 Apr 2020"
- board text removed: "R3: 10K= 100 mA 5K = 200 mA 2K = 500 mA 1K = 1000 mA"
- board text removed: "Rev 0.3 Sep 2018"

Commit message: Updates
Parts:
- D2: value DONE -> CHG
- D3: value CHG -> DONE
Other:
- board text added: "Rev 0.6 Apr 2020"
- board text removed: "Rev 0.5 Apr 2020"
Changed lines of the file:
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@@
     (links 28)
     (no_connects 0)
-    (area 121.92 84.930001 163.095715 120.201)
+    (area 123.114999 92.634999 148.665001 118.185001)
     (thickness 1.6)
     (drawings 28)
@@
       (effects (font (size 1 1) (thickness 0.15)))
     )
-    (fp_text value 1K (at 0 1.524 270) (layer F.SilkS)
+    (fp_text value 1K (at -1.24 1.625 270) (layer F.SilkS)
       (effects (font (size 1 1) (thickness 0.15)))
     )
@@
       (effects (font (size 1 1) (thickness 0.15)))
     )
-    (fp_text value 1K (at 0 -1.651 270) (layer F.SilkS)
+    (fp_text value 1K (at -1.24 1.55 270) (layer F.SilkS)
       (effects (font (size 1 1) (thickness 0.15)))
     )
@@
       (effects (font (size 1 1) (thickness 0.15)))
     )
-    (fp_text value DONE (at 0 1.397 270) (layer F.SilkS)
+    (fp_text value CHG (at -0.57 1.375 270) (layer F.SilkS)
       (effects (font (size 1 1) (thickness 0.15)))
     )
@@
       (effects (font (size 1 1) (thickness 0.15)))
     )
-    (fp_text value CHG (at 0 -1.651 270) (layer F.SilkS)
+    (fp_text value DONE (at -1.07 -1.7 270) (layer F.SilkS)
       (effects (font (size 1 1) (thickness 0.15)))
     )
@@
     (effects (font (size 0.75 0.75) (thickness 0.15)) (justify left mirror))
   )
-  (gr_text "Rev 0.5\nApr 2020" (at 146.812 116.332) (layer B.SilkS)
+  (gr_text "Rev 0.6\nApr 2020" (at 146.812 116.332) (layer B.SilkS)
     (effects (font (size 0.75 0.75) (thickness 0.15)) (justify left mirror))
   )
