File: projects/Beetje/design_files_template/project.kicad_pcb (KiCad board)
At the start: 2 copper layers, 25.4 x 25.4 mm, 8 parts, among them J2 Beetje_Bottom, J4 Beetje_Top, SW1 SW_Push

Commit message: Updates
Parts:
- moved SW1 6.62 mm to (141.7, 123.4)
- moved D1 4.78 mm to (133.2, 125.0)
- moved C1 3.74 mm to (127.6, 123.3)
- moved R1 3.25 mm to (133.0, 121.7)
Changed lines of the file:
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@@
-(kicad_pcb (version 4) (host pcbnew 4.0.6)
+(kicad_pcb (version 4) (host pcbnew 4.0.7)
   (general
     (links 7)
     (no_connects 7)
-    (area 140.894999 85.014999 166.445001 110.565001)
+    (area 123.114999 92.634999 148.665001 118.185001)
     (thickness 1.6)
     (drawings 16)
@@
   )
   (module footprints:C_0603 (layer F.Cu)
-    (at 127 127 90)
+    (at 127.635 123.317 90)
     (descr "Capacitor SMD 0603, reflow soldering, AVX (see smccp.pdf)")
     (tags "capacitor 0603")
@@
   )
   (module footprints:LED_0603 (layer F.Cu)
-    (at 134.62 129.54)
+    (at 133.223 124.968)
     (descr "LED 0603 smd package")
     (tags "LED led 0603 SMD smd SMT smt smdled SMDLED smtled SMTLED")
@@
   )
   (module footprints:R_0603 (layer F.Cu)
-    (at 134.62 124.46)
+    (at 132.969 121.666)
     (descr "Resistor SMD 0603, reflow soldering, Vishay (see dcrcw.pdf)")
     (tags "resistor 0603")
@@
   )
   (module footprints:SW_SPST_KMR2 (layer F.Cu)
-    (at 147.32 127)
+    (at 141.732 123.444)
     (descr "CK components KMR2 tactile switch http://www.ckswitches.com/media/1479/kmr2.pdf")
     (tags "tactile switch kmr2")

Commit message: updates
Parts:
- moved VAL 1.52 mm to (127.0, 109.0)
- moved REF*** 1.40 mm to (139.2, 109.3)
Other:
- board text added: "D9 SDA SCL MI MO SCK"
- board text added: "RST D10 A0 A1 BAT BCC GND VBUS"
Changed lines of the file:
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@@
     (area 123.114999 92.634999 148.665001 118.185001)
     (thickness 1.6)
-    (drawings 16)
+    (drawings 18)
     (tracks 0)
     (zones 0)
@@
   )
   (module footprints:KiCad-Logo2_8mm_SilkScreen (layer B.Cu)
-    (at 139.192 110.744 180)
+    (at 139.192 109.347 180)
     (descr "KiCad Logo")
     (tags "Logo KiCad")
@@
   )
   (module footprints:MadeInOregonRev25 (layer F.Cu)
-    (at 127 107.442)
+    (at 127 108.966)
     (fp_text reference VAL (at 0 0) (layer F.SilkS) hide
       (effects (font (size 1.143 1.143) (thickness 0.1778)))
@@
     )
   )
+  (gr_text "D9 SDA SCL  MI  MO SCK" (at 140.716 115.189) (layer B.SilkS)
+    (effects (font (size 0.7 0.75) (thickness 0.175)) (justify left mirror))
+  )
+  (gr_text "RST D10  A0  A1  BAT BCC GND VBUS" (at 145.415 95.758) (layer B.SilkS)
+    (effects (font (size 0.7 0.675) (thickness 0.16875)) (justify left mirror))
+  )
   (gr_text "Beetje Blok" (at 125.73 97.79) (layer F.SilkS)
     (effects (font (size 1.75 1.75) (thickness 0.4) italic) (justify left))
   )
-  (gr_text "Rev 0.0\nAug 2018" (at 129.54 111.76) (layer B.SilkS)
+  (gr_text "Rev 0.0\nAug 2018" (at 146.685 115.951) (layer B.SilkS)
     (effects (font (size 0.75 0.75) (thickness 0.15)) (justify left mirror))
   )
@@
     (arrow2b (pts (xy 148.59 87.630001) (xy 147.463496 88.216422)))
   )
-  (gr_text www.MakersBox.us (at 147.701 114.554) (layer B.SilkS)
+  (gr_text www.MakersBox.us (at 147.574 113.284) (layer B.SilkS)
     (effects (font (size 1.75 1.75) (thickness 0.3) italic) (justify left mirror))
   )

Commit message: Updates
Parts:
- J2: footprint footprints:Pin_Header_Straight_1x06_Pitch2.54mm -> footprints:Beetje_Bottom
- J4: footprint footprints:Pin_Header_Straight_1x08_Pitch2.54mm -> footprints:Beetje_Top
Other:
- board text added: "Rev 0.0 Sep 2018"
- board text removed: "D9 SDA SCL MI MO SCK"
- board text removed: "RST D10 A0 A1 BAT BCC GND VBUS"
- board text removed: "Rev 0.0 Aug 2018"
- board text removed: "SCK MO MI SCL SDA D9"
- board text removed: "VBUS GND VCC BAT A1 A0 D10 RST"
