File: projects/Beetje/design_files_OLED/project.sch (KiCad schematic (older format))
At the start: 14 parts, among them J1 12FFCC, J2 Beetje_Bottom, J4 Beetje_Top

Commit message: Updates
Parts:
- C1, C2, C3: footprint footprints:C_0603 -> footprints:C_0805_HandSoldering
- J2: footprint footprints:Pin_Header_Straight_1x06_Pitch2.54mm -> footprints:Beetje_Bottom
- J4: footprint footprints:Pin_Header_Straight_1x08_Pitch2.54mm -> footprints:Beetje_Top
- R1, R2, R3, R4, R5, R6: footprint footprints:R_0603 -> footprints:R_0805_HandSoldering
Connections:
- net +BATT: now also J4.7 (Pin_7); no longer J4.5 (Pin_5)
- net A0: now also J2.1 (Pin_1); no longer J4.3 (Pin_3)
- net D10: now also J4.3 (Pin_3); no longer J4.2 (Pin_2)
- net D9: now also J4.2 (Pin_2), J4.6 (Pin_6); no longer J2.1 (Pin_1), J2.6 (Pin_6)
- net GND: now also J2.6 (Pin_6); no longer J4.7 (Pin_7)
- net VCC: now also J2.5 (Pin_5); no longer J4.6 (Pin_6)
- net A1 renamed MISO
- net MISO: now also J1.3 (Pin_3), J2.4 (Pin_4), JP1.1, R1.2
- net SCL renamed MOSI
- net MOSI: now also J4.5 (Pin_5); no longer J2.5 (Pin_5)
- removed net SDA: J1.3 (Pin_3), J2.2 (Pin_2), J2.4 (Pin_4), JP1.1, R1.2
- new net D6: J2.2 (Pin_2)
Other:
- note added: "Beetje Footprint"
- note removed: "SDA D2\nSCL D3\nMISO D15\nMOSI D14\nSCK D16"
