File: projects/Beetje/design_files_32U4/project.kicad_pcb (KiCad board)
At the start: 2 copper layers, 25.4 x 25.4 mm, 27 parts, among them CON1 AVR-ISP-6, J2 Conn_01x06, J4 Conn_01x08, SW1 RESET, U1 ATMEGA32U4-AU, U2 MIC5225-3.3, X3 USB_OTG, Y1 8 Mhz

Commit message: Updates
Parts:
- D1, D4, F1: moved to F.Cu
- SW1: value RESET -> RST
- moved D4 9.15 mm to (159.0, 90.7)
- moved D1 9.02 mm to (153.8, 90.7)
- moved C6 4.07 mm to (147.6, 96.8)
- moved C7 3.86 mm to (148.5, 100.2), turned to 270 degrees
- moved R5 3.05 mm to (148.8, 103.4)
- moved R4 2.92 mm to (148.8, 106.4)
- moved F1 2.90 mm to (147.3, 92.5), turned to 270 degrees
- moved JMP1 1.78 mm to (149.6, 95.4)
- moved C9 1.27 mm to (144.3, 98.0)
- moved R9 1.27 mm to (143.9, 91.6)
- moved U2 1.27 mm to (144.1, 94.6)
- moved X3 1.27 mm to (144.1, 104.1)
- moved C8 1.09 mm to (151.8, 106.9)
- moved CON1 0.76 mm to (159.4, 99.8)
- moved REF*** 0.76 mm to (158.6, 105.0)
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Routing:
- net /VHI: track 8.75 -> 21.5 mm, vias 1 -> 2
- net VBUS: track 21.2 -> 27.7 mm
- net +BATT: track 3.79 -> 9.92 mm, vias 0 -> 1
- net Net-(F1-Pad2): track 9.84 -> 13.1 mm, vias 1 -> 2
- net GND: track 123.5 -> 126.4 mm
- net /D-: track 5.75 -> 8.18 mm
- net /D+: track 8.37 -> 10.6 mm
- net /A1: track 5.39 -> 7.40 mm
- net Net-(R4-Pad2): track 3.06 -> 5.02 mm
- net /SCK: track 22.3 -> 20.5 mm
- net /MOSI: track 24.2 -> 22.6 mm
- net VCC: track 90.2 -> 88.9 mm, vias 4 -> 5
- net /~RESET: track 36.2 -> 37.3 mm
- net /A0: track 4.67 -> 5.60 mm
- net /MISO: track 19.4 -> 18.6 mm
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Other:
- board text added: "+ ISP -"
- board text added: "Rev 0.1 Aug 2018"
- board text removed: "- ISP +"
- board text removed: "Rev 0.0 Aug 2018"

Commit message: Updates
Parts:
- moved VAL 0.28 mm to (164.2, 97.9)
- moved REF*** 0.25 mm to (158.6, 105.3)
Other:
- board text added: "Beetje 32U4 Blok"
- board text added: "D9 SDA SCL MI MO SCK"
- board text added: "RST D10 A0 A0 BAT VCC GND VBUS"
- board text removed: "Beetje Blok 32U4"
Changed lines of the file:
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@@
-(kicad_pcb (version 4) (host pcbnew 4.0.6)
+(kicad_pcb (version 4) (host pcbnew 4.0.7)
   (general
     (links 77)
@@
     (area 142.164999 86.284999 167.715001 111.835001)
     (thickness 1.6)
-    (drawings 19)
+    (drawings 21)
     (tracks 416)
     (zones 0)
@@
     (34 B.Paste user)
     (35 F.Paste user)
-    (36 B.SilkS user hide)
+    (36 B.SilkS user)
     (37 F.SilkS user)
     (38 B.Mask user)
@@
     (44 Edge.Cuts user)
     (45 Margin user)
-    (46 B.CrtYd user)
+    (46 B.CrtYd user hide)
     (47 F.CrtYd user)
     (48 B.Fab user hide)
@@
   )
   (setup
-    (last_trace_width 0.3048)
+    (last_trace_width 0.25)
     (user_trace_width 0.3048)
     (user_trace_width 0.4064)
@@
     (pad 1 smd rect (at -1.8 -0.7 90) (size 1.4 1.05) (layers F.Cu F.Paste F.Mask)
       (net 1 GND))
-    (model ${KISYS3DMOD}/Buttons_Switches_SMD.3dshapes/SW_SPST_KMR2.wrl
-      (at (xyz 0 0 0))
-      (scale (xyz 1 1 1))
-      (rotate (xyz 0 0 0))
-    )
-    (model "C:/Users/Maker's Box/Downloads/3d_switch (1)/walter/switch/smd_push2.wrl"
-      (at (xyz 0 0 0))
-      (scale (xyz 1 1 1))
-      (rotate (xyz 0 0 0))
-    )
   )
   (module myFootPrints:MadeInOregonRev25 (layer F.Cu)
-    (at 164.084 98.171)
+    (at 164.211 97.917)
     (fp_text reference VAL (at 0 0) (layer F.SilkS) hide
       (effects (font (size 1.143 1.143) (thickness 0.1778)))
@@
   )
   (module footprints:KiCad-Logo2_8mm_SilkScreen (layer B.Cu)
-    (at 158.623 105.029 180)
+    (at 158.623 105.283 180)
     (descr "KiCad Logo")
     (tags "Logo KiCad")
@@
     )
   )
+  (gr_text "RST D10  A0  A0  BAT VCC GND VBUS" (at 164.719 89.535) (layer B.SilkS)
+    (effects (font (size 0.7 0.675) (thickness 0.16875)) (justify left mirror))
+  )
+  (gr_text "D9 SDA SCL  MI  MO SCK" (at 159.512 108.712) (layer B.SilkS)
+    (effects (font (size 0.7 0.75) (thickness 0.175)) (justify left mirror))
+  )
   (gr_text "Rev 0.1\nAug 2018" (at 148.463 104.013) (layer B.SilkS)
     (effects (font (size 0.75 0.75) (thickness 0.15)) (justify left mirror))
@@
     (arrow2b (pts (xy 167.64 81.280001) (xy 166.513496 81.866422)))
   )
-  (gr_text "+ ISP -" (at 156.845 94.234) (layer B.SilkS)
-    (effects (font (size 1.25 1.25) (thickness 0.3)) (justify mirror))
+  (gr_text "+ ISP -" (at 156.591 95.25) (layer B.SilkS)
+    (effects (font (size 1 1) (thickness 0.25)) (justify mirror))
   )
   (gr_circle (center 152.781 93.98) (end 152.781 93.726) (layer F.SilkS) (width 0.2))
-  (gr_text www.MakersBox.us (at 166.751 108.204) (layer B.SilkS)
+  (gr_text www.MakersBox.us (at 166.878 93.599) (layer B.SilkS)
     (effects (font (size 1.75 1.75) (thickness 0.3) italic) (justify left mirror))
   )
-  (gr_text "Beetje Blok\n32U4" (at 167.132 91.44) (layer B.SilkS)
+  (gr_text "Beetje 32U4 Blok\n" (at 167.132 91.44) (layer B.SilkS)
     (effects (font (size 1.75 1.75) (thickness 0.4) italic) (justify left mirror))
   )
@@
     (effects (font (size 0.7 0.75) (thickness 0.175)) (justify left))
   )
-  (segment (start 165.416 94.0655) (end 165.416 95.442) (width 0.3048) (layer F.Cu) (net 1) (status 400000))
+  (segment (start 165.416 94.0655) (end 165.416 95.442) (width 0.3048) (layer F.Cu) (net 1))
   (segment (start 164.973 95.885) (end 165.416 95.442) (width 0.3048) (layer F.Cu) (net 1))
   (segment (start 164.973 97.409) (end 164.973 95.885) (width 0.3048) (layer F.Cu) (net 1))
@@
   (segment (start 163.957 101.219) (end 163.957 98.425) (width 0.3048) (layer F.Cu) (net 1))
   (segment (start 163.957 101.219) (end 163.957 101.723802) (width 0.3048) (layer F.Cu) (net 1))
-  (segment (start 165.416 94.0655) (end 165.6065 93.875) (width 0.3048) (layer F.Cu) (net 1) (status C00000))
+  (segment (start 165.416 94.0655) (end 165.6065 93.875) (width 0.3048) (layer F.Cu) (net 1))
   (segment (start 163.997 91.694) (end 164.4015 91.694) (width 0.4064) (layer F.Cu) (net 1))
   (segment (start 160.045 92.05) (end 160.401 91.694) (width 0.4064) (layer F.Cu) (net 1))
   (segment (start 160.401 91.694) (end 163.997 91.694) (width 0.4064) (layer F.Cu) (net 1))
   (segment (start 160.045 92.852) (end 160.045 92.05) (width 0.4064) (layer F.Cu) (net 1))
-  (segment (start 165.6065 92.899) (end 165.6065 93.875) (width 0.4064) (layer F.Cu) (net 1) (status 800000))
+  (segment (start 165.6065 92.899) (end 165.6065 93.875) (width 0.4064) (layer F.Cu) (net 1))
   (segment (start 164.4015 91.694) (end 165.6065 92.899) (width 0.4064) (layer F.Cu) (net 1))
   (segment (start 163.957 101.981) (end 163.957 101.723802) (width 0.3048) (layer F.Cu) (net 1))

Commit message: Updates
Parts:
- added R3: 4K7, footprints:R_0603, F.Cu at (159.4, 107.3)
- added R6: 4K7, footprints:R_0603, F.Cu at (161.3, 107.3)
- added SW2: D4, footprints:EVQ-P7A, F.Cu at (166.4, 101.0)
- J2: value Conn_01x06 -> Beetje Bottom; footprint footprints:Pin_Header_Straight_1x06_Pitch2.54mm -> footprints:Beetje_Bottom
- J4: value Conn_01x08 -> Beetje Top; footprint footprints:Pin_Header_Straight_1x08_Pitch2.54mm -> footprints:Beetje_Top
- moved R7 9.57 mm to (167.0, 107.3)
- moved R1 6.87 mm to (163.2, 107.3)
- moved R2 2.62 mm to (165.1, 107.3)
- moved D13 0.51 mm to (165.1, 110.4)
- moved D3 0.51 mm to (161.3, 110.4)
- moved D5 0.51 mm to (163.2, 110.4)
- moved SW1 0.06 mm to (166.4, 92.1)
Connections:
- J2 pad 1: /D9 -> /A0
- J4 pad 2: /D10 -> /D6
- J4 pad 3: /A0 -> /D9
- J4 pad 4: /A1 -> /D10
- SW1 pad 1: GND -> /~RESET
- SW1 pad 2: /~RESET -> GND
Routing:
- net /A0: track 5.60 -> 27.5 mm, vias 0 -> 1
- net /D6: track 0.00 -> 15.9 mm, vias 0 -> 1
- net /D13: track 5.04 -> 14.5 mm
- net Net-(D13-Pad2): track 13.4 -> 4.30 mm
- net /D4: track 0.00 -> 8.20 mm
- net /A1: track 7.40 -> 0.00 mm
- net Net-(D3-Pad1): track 9.21 -> 2.53 mm
- net /D10: track 10.3 -> 16.9 mm
- net GND: track 126.4 -> 120.6 mm, vias 5 -> 3
- net VCC: track 88.9 -> 93.6 mm, vias 5 -> 2
- net /TXLED: track 7.93 -> 3.31 mm
- net /SDA: track 8.32 -> 12.3 mm, vias 0 -> 1
- net /RXLED: track 30.9 -> 27.1 mm
- net Net-(D5-Pad1): track 5.75 -> 2.53 mm
- net +BATT: track 9.92 -> 8.59 mm, vias 1 -> 0
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Other:
- board text added: ">"
- board text added: "Rev 0.2 Sep 2018"
- board text removed: "D9 SDA SCL MI MO SCK"
- board text removed: "RST D10 A0 A0 BAT VCC GND VBUS"
- board text removed: "Rev 0.1 Aug 2018"
- board text removed: "SCK MO MI SCL SDA D9"
- board text removed: "VBUS GND VCC BAT A1 A0 D10 RST"

Commit message: Updates
Parts:
- R1, R2, R7: value 180 -> 330
- moved JMP1 1.40 mm to (151.0, 95.2)
Connections:
- J2 pad 1: /A0 -> /~RESET
- J2 pad 2: /SDA -> /D6
- J2 pad 4: /MISO -> /SDA
- J2 pad 5: /MOSI -> VCC
- J2 pad 6: /SCK -> GND
- J4 pad 1: /~RESET -> /A0
- J4 pad 2: /D6 -> /D9
- J4 pad 3: /D9 -> /D10
- J4 pad 4: /D10 -> /MISO
- J4 pad 5: +BATT -> /MOSI
- J4 pad 6: VCC -> /SCK
- J4 pad 7: GND -> +BATT
Routing:
- net /A0: track 27.5 -> 8.53 mm
- net /~RESET: track 36.9 -> 50.7 mm, vias 1 -> 2
- net /SDA: track 12.3 -> 25.4 mm
- net /D6: track 15.9 -> 27.9 mm, vias 1 -> 3
- net VCC: track 93.6 -> 82.3 mm, vias 2 -> 1
- net /MISO: track 18.6 -> 26.5 mm
- net GND: track 120.6 -> 126.1 mm, vias 3 -> 4
- net +BATT: track 8.59 -> 13.9 mm
- net /SCK: track 20.5 -> 24.2 mm
- net Net-(R4-Pad2): track 5.02 -> 8.63 mm
- net VBUS: track 27.8 -> 24.5 mm
- net /RXLED: track 27.1 -> 23.9 mm
- net /VHI: track 22.5 -> 19.4 mm, vias 2 -> 0
- net /MOSI: track 22.6 -> 24.9 mm
- net /D-: track 8.18 -> 10.0 mm, vias 0 -> 2
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Other:
- board text added: "Rev 0.3 Sep 2018"
- board text removed: "Rev 0.2 Sep 2018"

Commit message: Updates
Connections:
- J2 pad 1: /~RESET -> /A0
- J4 pad 1: /A0 -> /~RESET
Routing:
- net /A0: track 8.53 -> 32.4 mm
- net /~RESET: track 50.7 -> 47.8 mm, vias 2 -> 3
- net VCC: track 82.3 -> 83.5 mm
- net /D13: track 14.7 -> 15.7 mm
- net GND: track 126.1 -> 125.4 mm
Other:
- board text added: "I2C"

Commit message: Updates
Changed lines of the file:
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@@
-(kicad_pcb (version 4) (host pcbnew 4.0.6)
+(kicad_pcb (version 4) (host pcbnew 4.0.7)
   (general
     (links 85)
     (no_connects 0)
-    (area 142.164999 86.284999 167.715001 111.835001)
+    (area 125.73 78.580001 182.145715 116.332001)
     (thickness 1.6)
     (drawings 28)
-    (tracks 421)
+    (tracks 422)
     (zones 0)
     (modules 30)
@@
   )
   (setup
-    (last_trace_width 0.3048)
+    (last_trace_width 0.4064)
     (user_trace_width 0.3048)
     (user_trace_width 0.4064)
@@
   (segment (start 164.338 104.013) (end 164.465 104.14) (width 0.3048) (layer B.Cu) (net 36))
   (segment (start 163.576 104.013) (end 164.338 104.013) (width 0.3048) (layer B.Cu) (net 36))
-  (segment (start 165.1 106.172) (end 165.1 106.565) (width 0.3048) (layer F.Cu) (net 36) (status 800000))
+  (segment (start 165.1 106.172) (end 165.1 106.565) (width 0.3048) (layer F.Cu) (net 36))
   (segment (start 164.465 105.537) (end 165.1 106.172) (width 0.3048) (layer F.Cu) (net 36))
   (segment (start 163.195 106.565) (end 162.953 106.565) (width 0.25) (layer F.Cu) (net 37))
@@
   (segment (start 165.443 111.163) (end 167.005 109.601) (width 0.3048) (layer F.Cu) (net 43))
   (segment (start 167.005 109.601) (end 167.005 108.065) (width 0.3048) (layer F.Cu) (net 43))
+  (segment (start 147.066 98.298) (end 147.066 92.964) (width 0.4064) (layer B.Cu) (net 44))
+  (segment (start 145.639 102.84) (end 145.288 102.489) (width 0.4064) (layer F.Cu) (net 44))
+  (segment (start 145.288 102.489) (end 145.288 100.838) (width 0.4064) (layer F.Cu) (net 44))
+  (segment (start 145.288 100.838) (end 145.796 100.33) (width 0.4064) (layer F.Cu) (net 44))
+  (via (at 145.796 100.33) (size 0.6) (drill 0.4) (layers F.Cu B.Cu) (net 44))
+  (segment (start 145.796 100.33) (end 147.066 99.06) (width 0.4064) (layer B.Cu) (net 44))
+  (segment (start 147.066 99.06) (end 147.066 98.298) (width 0.4064) (layer B.Cu) (net 44))
   (segment (start 146.495 102.84) (end 145.639 102.84) (width 0.4064) (layer F.Cu) (net 44))
-  (segment (start 147.066 99.06) (end 147.066 98.298) (width 0.4064) (layer B.Cu) (net 44))
-  (segment (start 145.796 100.33) (end 147.066 99.06) (width 0.4064) (layer B.Cu) (net 44))
-  (via (at 145.796 100.33) (size 0.6) (drill 0.4) (layers F.Cu B.Cu) (net 44))
-  (segment (start 145.288 100.838) (end 145.796 100.33) (width 0.4064) (layer F.Cu) (net 44))
-  (segment (start 145.288 102.489) (end 145.288 100.838) (width 0.4064) (layer F.Cu) (net 44))
-  (segment (start 145.639 102.84) (end 145.288 102.489) (width 0.4064) (layer F.Cu) (net 44))
-  (segment (start 147.32 93.091) (end 147.32 93.906) (width 0.3048) (layer F.Cu) (net 44))
-  (segment (start 147.066 92.837) (end 147.32 93.091) (width 0.3048) (layer F.Cu) (net 44))
-  (via (at 147.066 92.837) (size 0.6) (drill 0.4) (layers F.Cu B.Cu) (net 44))
-  (segment (start 147.066 98.298) (end 147.066 92.837) (width 0.3048) (layer B.Cu) (net 44))
+  (segment (start 147.32 93.218) (end 147.32 93.906) (width 0.4064) (layer F.Cu) (net 44) (status 800000))
+  (segment (start 146.812 92.71) (end 147.32 93.218) (width 0.4064) (layer F.Cu) (net 44))
+  (via (at 146.812 92.71) (size 0.6) (drill 0.4) (layers F.Cu B.Cu) (net 44))
+  (segment (start 147.066 92.964) (end 146.812 92.71) (width 0.4064) (layer B.Cu) (net 44))
   (segment (start 161.29 109.563) (end 161.455 109.563) (width 0.3048) (layer F.Cu) (net 45))
   (segment (start 161.455 109.563) (end 162.953 108.065) (width 0.3048) (layer F.Cu) (net 45))
