File: projects/Beetje/design_files_32U4/project.sch (KiCad schematic (older format))
At the start: 25 parts, among them CON1 AVR-ISP-6, J2 Beetje Bottom, J4 Beetje Top, SW1 RESET, U1 ATMEGA32U4-AU, U2 MIC5225-3.3, X3 USB_OTG, Y1 8 Mhz

Commit message: Updates
Connections:
- wire segments 98 -> 99
Changed lines of the file:
@@
 Text Notes 2250 5000 0    60   ~ 0
 Beetje Footprint
+Wire Wire Line
+	3950 4550 3950 4650
 $EndSCHEMATC

Commit message: Updates
Parts:
- added R3, R6: 4K7, footprints:R_0603, symbol R
- added SW2: D4, footprints:EVQ-P7A, symbol SW_Push
- J2: footprint footprints:Pin_Header_Straight_1x06_Pitch2.54mm -> footprints:Beetje_Bottom
- J4: footprint footprints:Pin_Header_Straight_1x08_Pitch2.54mm -> footprints:Beetje_Top
- R1, R2, R7: value 180 -> 330
- SW1: value RESET -> RST
Connections:
- wire segments 99 -> 107
- no-connect marks 18 -> 17
Other:
- moved on the sheet: D13, D3, D5, R1, R2, R7

Commit message: Updates
Other:
- note added: "SparkFun's Qwiic:\nBlack = GND\nRed = 3.3V\nBlue = SDA\nYellow = SCL"
Changed lines of the file:
@@
 L +BATT #PWR017
 U 1 1 5B402C38
-P 2600 5550
-F 0 "#PWR017" H 2600 5400 50  0001 C CNN
-F 1 "+BATT" V 2600 5800 50  0000 C CNN
-F 2 "" H 2600 5550 50  0001 C CNN
-F 3 "" H 2600 5550 50  0001 C CNN
-	1    2600 5550
+P 2600 5750
+F 0 "#PWR017" H 2600 5600 50  0001 C CNN
+F 1 "+BATT" V 2600 6000 50  0000 C CNN
+F 2 "" H 2600 5750 50  0001 C CNN
+F 3 "" H 2600 5750 50  0001 C CNN
+	1    2600 5750
 	0    -1   -1   0
 $EndComp
@@
 	0    -1   -1   0
 $EndComp
-Text Label 2600 5450 0    60   ~ 0
+Text Label 2600 5350 0    60   ~ 0
 D10
-Text Label 2600 5350 0    60   ~ 0
+Text Label 2600 5250 0    60   ~ 0
 D9
 Text Label 4000 5350 0    60   ~ 0
 SCL
-Text Label 4000 5250 0    60   ~ 0
+Text Label 4000 5450 0    60   ~ 0
 SDA
+Text Label 3900 5150 0    60   ~ 0
+~RESET
 Text Label 2600 5150 0    60   ~ 0
-~RESET
-Text Label 4050 5150 0    60   ~ 0
 A0
-Text Label 2600 5250 0    60   ~ 0
+Text Label 4050 5250 0    60   ~ 0
 D6
-Text Label 4000 5650 0    60   ~ 0
+Text Label 2600 5650 0    60   ~ 0
 SCK
-Text Label 3950 5550 0    60   ~ 0
+Text Label 2600 5550 0    60   ~ 0
 MOSI
-Text Label 3950 5450 0    60   ~ 0
+Text Label 2600 5450 0    60   ~ 0
 MISO
 $Comp
@@
 L GND #PWR020
 U 1 1 5B41D2F5
-P 2600 5750
-F 0 "#PWR020" H 2600 5500 50  0001 C CNN
-F 1 "GND" V 2600 5550 50  0000 C CNN
-F 2 "" H 2600 5750 50  0001 C CNN
-F 3 "" H 2600 5750 50  0001 C CNN
-	1    2600 5750
-	0    1    1    0
+P 3950 5650
+F 0 "#PWR020" H 3950 5400 50  0001 C CNN
+F 1 "GND" V 3950 5450 50  0000 C CNN
+F 2 "" H 3950 5650 50  0001 C CNN
+F 3 "" H 3950 5650 50  0001 C CNN
+	1    3950 5650
+	0    -1   -1   0
 $EndComp
 Text Label 7300 2800 0    60   ~ 0
@@
 L VCC #PWR026
 U 1 1 5B6E81BF
-P 2600 5650
-F 0 "#PWR026" H 2600 5500 50  0001 C CNN
-F 1 "VCC" V 2600 5850 50  0000 C CNN
-F 2 "" H 2600 5650 50  0001 C CNN
-F 3 "" H 2600 5650 50  0001 C CNN
-	1    2600 5650
-	0    -1   -1   0
+P 3950 5550
+F 0 "#PWR026" H 3950 5400 50  0001 C CNN
+F 1 "VCC" V 3950 5750 50  0000 C CNN
+F 2 "" H 3950 5550 50  0001 C CNN
+F 3 "" H 3950 5550 50  0001 C CNN
+	1    3950 5550
+	0    1    1    0
 $EndComp
 NoConn ~ 7550 3200
@@
 	3850 5450 4150 5450
 Wire Wire Line
-	3850 5550 4150 5550
-Wire Wire Line
-	3850 5650 4150 5650
+	3850 5550 3950 5550
+Wire Wire Line
+	3850 5650 3950 5650
 Wire Wire Line
 	2650 1950 2900 1950
@@
 	8300 3250 8300 3350
 Connection ~ 8200 3250
+Text Notes 2350 6850 0    60   ~ 0
+SparkFun's Qwiic:\nBlack = GND\nRed = 3.3V\nBlue = SDA\nYellow = SCL
 $EndSCHEMATC

Commit message: Updates
Connections:
- wire segments 107 -> 124
Other:
- note added: "Beetje Footprint Rev 0.3"
- note removed: "Beetje Footprint"
Changed lines of the file:
@@
 L +BATT #PWR017
 U 1 1 5B402C38
-P 2600 5750
-F 0 "#PWR017" H 2600 5600 50  0001 C CNN
-F 1 "+BATT" V 2600 6000 50  0000 C CNN
-F 2 "" H 2600 5750 50  0001 C CNN
-F 3 "" H 2600 5750 50  0001 C CNN
-	1    2600 5750
+P 2750 5750
+F 0 "#PWR017" H 2750 5600 50  0001 C CNN
+F 1 "+BATT" V 2750 6000 50  0000 C CNN
+F 2 "" H 2750 5750 50  0001 C CNN
+F 3 "" H 2750 5750 50  0001 C CNN
+	1    2750 5750
 	0    -1   -1   0
 $EndComp
@@
 L VBUS #PWR018
 U 1 1 5B402FA5
-P 2600 5850
-F 0 "#PWR018" H 2600 5700 50  0001 C CNN
-F 1 "VBUS" V 2600 6050 50  0000 C CNN
-F 2 "" H 2600 5850 50  0001 C CNN
-F 3 "" H 2600 5850 50  0001 C CNN
-	1    2600 5850
+P 2750 5850
+F 0 "#PWR018" H 2750 5700 50  0001 C CNN
+F 1 "VBUS" V 2750 6050 50  0000 C CNN
+F 2 "" H 2750 5850 50  0001 C CNN
+F 3 "" H 2750 5850 50  0001 C CNN
+	1    2750 5850
 	0    -1   -1   0
 $EndComp
@@
 Text Label 4000 5450 0    60   ~ 0
 SDA
-Text Label 3900 5150 0    60   ~ 0
+Text Label 2600 5150 0    60   ~ 0
 ~RESET
-Text Label 2600 5150 0    60   ~ 0
+Text Label 4050 5150 0    60   ~ 0
 A0
 Text Label 4050 5250 0    60   ~ 0
@@
 P 3000 5450
 F 0 "J4" H 3000 5850 50  0000 C CNN
-F 1 "Beetje Top" H 3000 4950 50  0000 C CNN
+F 1 "Beetje Top" H 2850 4950 50  0000 C CNN
 F 2 "footprints:Beetje_Top" H 3000 5450 50  0001 C CNN
 F 3 "" H 3000 5450 50  0001 C CNN
@@
 P 3650 5350
 F 0 "J2" H 3650 5650 50  0000 C CNN
-F 1 "Beetje Bottom" H 3650 4950 50  0000 C CNN
+F 1 "Beetje Bottom" H 3400 4950 50  0000 C CNN
 F 2 "footprints:Beetje_Bottom" H 3650 5350 50  0001 C CNN
 F 3 "" H 3650 5350 50  0001 C CNN
@@
 5V:\nU2 = MIC5225-5\nY1 = 16 Mhz\nJMP1 = Short
 Text Notes 2250 5000 0    60   ~ 0
-Beetje Footprint
+Beetje Footprint Rev 0.3
 $Comp
 L SW_Push SW2
@@
 	7250 5700 7550 5700
 Wire Wire Line
-	5750 5950 6300 5950
+	5750 5950 6000 5950
+Wire Wire Line
+	6000 5950 6050 5950
+Wire Wire Line
+	6050 5950 6100 5950
+Wire Wire Line
+	6100 5950 6200 5950
+Wire Wire Line
+	6200 5950 6300 5950
 Connection ~ 6200 5950
 Connection ~ 6100 5950
@@
 Connection ~ 6050 5950
 Wire Wire Line
-	5950 2550 6400 2550
+	5950 2550 6050 2550
+Wire Wire Line
+	6050 2550 6150 2550
+Wire Wire Line
+	6150 2550 6300 2550
+Wire Wire Line
+	6300 2550 6400 2550
 Connection ~ 6300 2550
 Connection ~ 6050 2550
@@
 	5000 4250 4700 4250
 Wire Wire Line
-	2300 2900 3750 2900
+	2300 2900 3050 2900
+Wire Wire Line
+	3050 2900 3450 2900
+Wire Wire Line
+	3450 2900 3750 2900
 Wire Wire Line
 	3050 2900 3050 2700
@@
 Connection ~ 3450 2900
 Wire Wire Line
-	3350 2300 3750 2300
+	3350 2300 3450 2300
+Wire Wire Line
+	3450 2300 3750 2300
 Wire Wire Line
 	3750 2300 3750 2600
 Wire Wire Line
-	3450 1950 3450 2600
+	3450 1950 3450 2300
+Wire Wire Line
+	3450 2300 3450 2600
 Connection ~ 3450 2300
 Connection ~ 3750 2300
@@
 	2750 2400 2700 2400
 Wire Wire Line
-	2050 2400 2400 2400
-Wire Wire Line
-	2300 2250 2300 2600
+	2050 2400 2300 2400
+Wire Wire Line
+	2300 2400 2400 2400
+Wire Wire Line
+	2300 2250 2300 2400
+Wire Wire Line
+	2300 2400 2300 2600
 Connection ~ 2300 2400
 Wire Wire Line
-	2400 2300 2750 2300
+	2400 2300 2650 2300
+Wire Wire Line
+	2650 2300 2750 2300
 Wire Wire Line
 	2400 2400 2400 2300
@@
 	2800 5650 2600 5650
 Wire Wire Line
-	2800 5750 2600 5750
-Wire Wire Line
-	2800 5850 2600 5850
+	2800 5750 2750 5750
+Wire Wire Line
+	2800 5850 2750 5850
 Wire Wire Line
 	8550 4900 8550 5000
 Wire Wire Line
-	8550 5300 8550 5450
+	8550 5300 8550 5350
+Wire Wire Line
+	8550 5350 8550 5450
 Wire Wire Line
 	5000 3400 4950 3400
@@
 	9150 5000 9150 4950
 Wire Wire Line
-	8850 4650 9150 4650
+	8850 4650 9000 4650
+Wire Wire Line
+	9000 4650 9150 4650
 Wire Wire Line
 	9000 4650 9000 4600
@@
 	8100 3350 8100 3250
 Wire Wire Line
-	8100 3250 8300 3250
+	8100 3250 8200 3250
+Wire Wire Line
+	8200 3250 8300 3250
 Wire Wire Line
 	8300 3250 8300 3350

Commit message: Updates
Parts:
- R1, R2: value 330 -> 1K
- R3: renamed from R7; value 330 -> 1K
- renumbered C6 to C1, C8 to C2, C9 to C3, C7 to C4, D3 to D1, D5 to D2, D13 to D3, D1 to D5, R3 to R4, R6 to R5, R4 to R6, R5 to R7, R9 to R8, X3 to X1
Connections:
- wire segments 124 -> 107
Changed lines of the file:
@@
 Sheet 1 1
 Title "Beetje 32U4 Board"
-Date "2018-08-10"
-Rev "0.0"
+Date "2018-09-28"
+Rev "0.4"
 Comp "www.MakersBox.us"
 Comment1 "648.ken@gmail.com"
@@
 NoConn ~ 5700 2550
 $Comp
-L C C9
+L C C3
 U 1 1 5B3FDF75
 P 4850 4650
-F 0 "C9" H 4875 4750 50  0000 L CNN
+F 0 "C3" H 4875 4750 50  0000 L CNN
 F 1 "10uF" H 4875 4550 50  0000 L CNN
 F 2 "footprints:C_0805" H 4888 4500 50  0001 C CNN
@@
 $EndComp
 $Comp
-L USB_OTG X3
+L USB_OTG X1
 U 1 1 5B3FE368
 P 3950 4150
-F 0 "X3" H 3750 4600 50  0000 L CNN
+F 0 "X1" H 3750 4600 50  0000 L CNN
 F 1 "USB_OTG" H 3750 4500 50  0000 L CNN
 F 2 "footprints:USB_Micro-B_Molex-105017-0001" H 4100 4100 50  0001 C CNN
@@
 $EndComp
 $Comp
-L R R4
+L R R6
 U 1 1 5B3FE405
 P 4550 4150
-F 0 "R4" V 4500 4000 50  0000 C CNN
+F 0 "R6" V 4500 4000 50  0000 C CNN
 F 1 "22" V 4550 4150 50  0000 C CNN
 F 2 "footprints:R_0603" V 4480 4150 50  0001 C CNN
@@
 $EndComp
 $Comp
-L R R5
+L R R7
 U 1 1 5B3FE482
 P 4550 4250
-F 0 "R5" V 4600 4100 50  0000 C CNN
+F 0 "R7" V 4600 4100 50  0000 C CNN
 F 1 "22" V 4550 4250 50  0000 C CNN
 F 2 "footprints:R_0603" V 4480 4250 50  0001 C CNN
@@
 $EndComp
 $Comp
-L R R9
+L R R8
 U 1 1 5B3FF1C8
 P 2550 2400
-F 0 "R9" V 2630 2400 50  0000 C CNN
+F 0 "R8" V 2630 2400 50  0000 C CNN
 F 1 "100K" V 2550 2400 50  0000 C CNN
 F 2 "footprints:R_0603" V 2480 2400 50  0001 C CNN
@@
 $EndComp
 $Comp
-L C C6
+L C C1
 U 1 1 5B3FF285
 P 2300 2750
-F 0 "C6" H 2325 2850 50  0000 L CNN
+F 0 "C1" H 2325 2850 50  0000 L CNN
 F 1 "10uF" H 2325 2650 50  0000 L CNN
 F 2 "footprints:C_0805" H 2338 2600 50  0001 C CNN
@@
 $EndComp
 $Comp
-L C C8
+L C C2
 U 1 1 5B3FF2D3
 P 3450 2750
-F 0 "C8" H 3475 2850 50  0000 L CNN
+F 0 "C2" H 3475 2850 50  0000 L CNN
 F 1 "10uF" H 3475 2650 50  0000 L CNN
 F 2 "footprints:C_0805" H 3488 2600 50  0001 C CNN
@@
 $EndComp
 $Comp
-L C C7
+L C C4
 U 1 1 5B3FF331
 P 3750 2750
-F 0 "C7" H 3775 2850 50  0000 L CNN
+F 0 "C4" H 3775 2850 50  0000 L CNN
 F 1 "1uF" H 3775 2650 50  0000 L CNN
 F 2 "footprints:C_0603" H 3788 2600 50  0001 C CNN
@@
 $EndComp
 $Comp
-L D_Schottky D1
+L D_Schottky D5
 U 1 1 5B3FF7CC
 P 2650 2100
-F 0 "D1" H 2650 2200 50  0000 C CNN
+F 0 "D5" H 2650 2200 50  0000 C CNN
 F 1 "MBR120" H 2650 2000 50  0000 C CNN
 F 2 "footprints:D_SOD-123F" H 2650 2100 50  0001 C CNN
@@
 MISO
 $Comp
-L R R7
+L R R3
 U 1 1 5B406515
 P 8550 4750
-F 0 "R7" V 8630 4750 50  0000 C CNN
-F 1 "330" V 8550 4750 50  0000 C CNN
+F 0 "R3" V 8630 4750 50  0000 C CNN
+F 1 "1K" V 8550 4750 50  0000 C CNN
 F 2 "footprints:R_0603" V 8480 4750 50  0001 C CNN
 F 3 "" H 8550 4750 50  0001 C CNN
@@
 $EndComp
 $Comp
-L LED D13
+L LED D3
 U 1 1 5B40657A
 P 8550 5150
-F 0 "D13" H 8550 5250 50  0000 C CNN
+F 0 "D3" H 8550 5250 50  0000 C CNN
 F 1 "D13" H 8550 5050 50  0000 C CNN
 F 2 "footprints:LED_0603" H 8550 5150 50  0001 C CNN
@@
 P 9150 5150
 F 0 "R2" V 9230 5150 50  0000 C CNN
-F 1 "330" V 9150 5150 50  0000 C CNN
+F 1 "1K" V 9150 5150 50  0000 C CNN
 F 2 "footprints:R_0603" V 9080 5150 50  0001 C CNN
 F 3 "" H 9150 5150 50  0001 C CNN
@@
 $EndComp
 $Comp
-L LED D5
+L LED D2
 U 1 1 5B44E5CF
 P 9150 4800
-F 0 "D5" H 9150 4900 50  0000 C CNN
+F 0 "D2" H 9150 4900 50  0000 C CNN
 F 1 "RX" H 9150 4700 50  0000 C CNN
 F 2 "footprints:LED_0603" H 9150 4800 50  0001 C CNN
@@
 P 8850 5150
 F 0 "R1" V 8930 5150 50  0000 C CNN
-F 1 "330" V 8850 5150 50  0000 C CNN
+F 1 "1K" V 8850 5150 50  0000 C CNN
 F 2 "footprints:R_0603" V 8780 5150 50  0001 C CNN
 F 3 "" H 8850 5150 50  0001 C CNN
@@
 $EndComp
 $Comp
-L LED D3
+L LED D1
 U 1 1 5B44E63D
 P 8850 4800
-F 0 "D3" H 8850 4900 50  0000 C CNN
+F 0 "D1" H 8850 4900 50  0000 C CNN
 F 1 "TX" H 8850 4700 50  0000 C CNN
 F 2 "footprints:LED_0603" H 8850 4800 50  0001 C CNN
@@
 $EndComp
 $Comp
-L R R3
+L R R4
 U 1 1 5B988358
 P 8100 3500
-F 0 "R3" V 8180 3500 50  0000 C CNN
+F 0 "R4" V 8180 3500 50  0000 C CNN
 F 1 "4K7" V 8100 3500 50  0000 C CNN
 F 2 "footprints:R_0603" V 8030 3500 50  0001 C CNN
@@
 $EndComp
 $Comp
-L R R6
+L R R5
 U 1 1 5B988442
 P 8300 3500
-F 0 "R6" V 8380 3500 50  0000 C CNN
+F 0 "R5" V 8380 3500 50  0000 C CNN
 F 1 "4K7" V 8300 3500 50  0000 C CNN
 F 2 "footprints:R_0603" V 8230 3500 50  0001 C CNN
@@
 	7250 5700 7550 5700
 Wire Wire Line
-	5750 5950 6000 5950
-Wire Wire Line
-	6000 5950 6050 5950
-Wire Wire Line
-	6050 5950 6100 5950
-Wire Wire Line
-	6100 5950 6200 5950
-Wire Wire Line
-	6200 5950 6300 5950
+	5750 5950 6300 5950
 Connection ~ 6200 5950
 Connection ~ 6100 5950
@@
 Connection ~ 6050 5950
 Wire Wire Line
-	5950 2550 6050 2550
-Wire Wire Line
-	6050 2550 6150 2550
-Wire Wire Line
-	6150 2550 6300 2550
-Wire Wire Line
-	6300 2550 6400 2550
+	5950 2550 6400 2550
 Connection ~ 6300 2550
 Connection ~ 6050 2550
@@
 	5000 4250 4700 4250
 Wire Wire Line
-	2300 2900 3050 2900
-Wire Wire Line
-	3050 2900 3450 2900
-Wire Wire Line
-	3450 2900 3750 2900
+	2300 2900 3750 2900
 Wire Wire Line
 	3050 2900 3050 2700
@@
 Connection ~ 3450 2900
 Wire Wire Line
-	3350 2300 3450 2300
-Wire Wire Line
-	3450 2300 3750 2300
+	3350 2300 3750 2300
 Wire Wire Line
 	3750 2300 3750 2600
 Wire Wire Line
-	3450 1950 3450 2300
-Wire Wire Line
-	3450 2300 3450 2600
+	3450 1950 3450 2600
 Connection ~ 3450 2300
 Connection ~ 3750 2300
@@
 	2750 2400 2700 2400
 Wire Wire Line
-	2050 2400 2300 2400
-Wire Wire Line
-	2300 2400 2400 2400
-Wire Wire Line
-	2300 2250 2300 2400
-Wire Wire Line
-	2300 2400 2300 2600
+	2050 2400 2400 2400
+Wire Wire Line
+	2300 2250 2300 2600
 Connection ~ 2300 2400
 Wire Wire Line
-	2400 2300 2650 2300
-Wire Wire Line
-	2650 2300 2750 2300
+	2400 2300 2750 2300
 Wire Wire Line
 	2400 2400 2400 2300
@@
 	8550 4900 8550 5000
 Wire Wire Line
-	8550 5300 8550 5350
-Wire Wire Line
-	8550 5350 8550 5450
+	8550 5300 8550 5450
 Wire Wire Line
 	5000 3400 4950 3400
@@
 	9150 5000 9150 4950
 Wire Wire Line
-	8850 4650 9000 4650
-Wire Wire Line
-	9000 4650 9150 4650
+	8850 4650 9150 4650
 Wire Wire Line
 	9000 4650 9000 4600
@@
 	8100 3350 8100 3250
 Wire Wire Line
-	8100 3250 8200 3250
-Wire Wire Line
-	8200 3250 8300 3250
+	8100 3250 8300 3250
 Wire Wire Line
 	8300 3250 8300 3350

Commit message: Updates
Parts:
- C1, C2, C3: footprint footprints:C_0805 -> beetje_footprints:C_0805
- C4: footprint footprints:C_0603 -> beetje_footprints:C_0603
- CON1: footprint footprints:Pin_Header_Straight_2x03_Pitch2.54mm -> beetje_footprints:Pin_Header_Straight_2x03_Pitch2.54mm
- D1, D2, D3: footprint footprints:LED_0603 -> beetje_footprints:LED_0603
- D4, D5: footprint footprints:D_SOD-123F -> beetje_footprints:D_SOD-123F
- F1: footprint footprints:R_1206 -> beetje_footprints:R_1206
- J2: footprint footprints:Beetje_Bottom -> beetje_footprints:Beetje_Bottom
- J4: footprint footprints:Beetje_Top -> beetje_footprints:Beetje_Top
- JMP1: footprint footprints:Jumper -> beetje_footprints:Jumper
- R1, R2, R3, R4, R5, R6, R7, R8: footprint footprints:R_0603 -> beetje_footprints:R_0603
- SW1, SW2: footprint footprints:EVQ-P7A -> beetje_footprints:EVQ-P7A
- U1: footprint footprints:TQFP-44_10x10mm_Pitch0.8mm -> beetje_footprints:TQFP-44_10x10mm_Pitch0.8mm
- U2: footprint footprints:SOT-23-5 -> beetje_footprints:SOT-23-5
- X1: footprint footprints:USB_Micro-B_Molex-105017-0001 -> beetje_footprints:USB_Micro-B_Molex-105017-0001
- Y1: footprint footprints:Resonator_SMD_CTSC_1.3mmx3.2mm -> beetje_footprints:Resonator_SMD_CTSC_1.3mmx3.2mm
Changed lines of the file:
@@
 F 0 "U1" H 5200 6050 50  0000 C CNN
 F 1 "ATMEGA32U4-AU" H 6850 2850 50  0000 C CNN
-F 2 "footprints:TQFP-44_10x10mm_Pitch0.8mm" H 6150 4350 50  0001 C CIN
+F 2 "beetje_footprints:TQFP-44_10x10mm_Pitch0.8mm" H 6150 4350 50  0001 C CIN
 F 3 "" H 7250 5450 50  0001 C CNN
 	1    6150 4350
@@
 F 0 "C3" H 4875 4750 50  0000 L CNN
 F 1 "10uF" H 4875 4550 50  0000 L CNN
-F 2 "footprints:C_0805" H 4888 4500 50  0001 C CNN
+F 2 "beetje_footprints:C_0805" H 4888 4500 50  0001 C CNN
 F 3 "" H 4850 4650 50  0001 C CNN
 	1    4850 4650
@@
 F 0 "X1" H 3750 4600 50  0000 L CNN
 F 1 "USB_OTG" H 3750 4500 50  0000 L CNN
-F 2 "footprints:USB_Micro-B_Molex-105017-0001" H 4100 4100 50  0001 C CNN
+F 2 "beetje_footprints:USB_Micro-B_Molex-105017-0001" H 4100 4100 50  0001 C CNN
 F 3 "" H 4100 4100 50  0001 C CNN
 	1    3950 4150
@@
 F 0 "R6" V 4500 4000 50  0000 C CNN
 F 1 "22" V 4550 4150 50  0000 C CNN
-F 2 "footprints:R_0603" V 4480 4150 50  0001 C CNN
+F 2 "beetje_footprints:R_0603" V 4480 4150 50  0001 C CNN
 F 3 "" H 4550 4150 50  0001 C CNN
 	1    4550 4150
@@
 F 0 "R7" V 4600 4100 50  0000 C CNN
 F 1 "22" V 4550 4250 50  0000 C CNN
-F 2 "footprints:R_0603" V 4480 4250 50  0001 C CNN
+F 2 "beetje_footprints:R_0603" V 4480 4250 50  0001 C CNN
 F 3 "" H 4550 4250 50  0001 C CNN
 	1    4550 4250
@@
 F 0 "U2" H 2900 2625 50  0000 C CNN
 F 1 "MIC5225-3.3" H 2700 2050 50  0000 L CNN
-F 2 "footprints:SOT-23-5" H 3050 2725 50  0001 C CNN
+F 2 "beetje_footprints:SOT-23-5" H 3050 2725 50  0001 C CNN
 F 3 "" H 3050 2400 50  0001 C CNN
 	1    3050 2400
@@
 F 0 "R8" V 2630 2400 50  0000 C CNN
 F 1 "100K" V 2550 2400 50  0000 C CNN
-F 2 "footprints:R_0603" V 2480 2400 50  0001 C CNN
+F 2 "beetje_footprints:R_0603" V 2480 2400 50  0001 C CNN
 F 3 "" H 2550 2400 50  0001 C CNN
 	1    2550 2400
@@
 F 0 "C1" H 2325 2850 50  0000 L CNN
 F 1 "10uF" H 2325 2650 50  0000 L CNN
-F 2 "footprints:C_0805" H 2338 2600 50  0001 C CNN
+F 2 "beetje_footprints:C_0805" H 2338 2600 50  0001 C CNN
 F 3 "" H 2300 2750 50  0001 C CNN
 	1    2300 2750
@@
 F 0 "C2" H 3475 2850 50  0000 L CNN
 F 1 "10uF" H 3475 2650 50  0000 L CNN
-F 2 "footprints:C_0805" H 3488 2600 50  0001 C CNN
+F 2 "beetje_footprints:C_0805" H 3488 2600 50  0001 C CNN
 F 3 "" H 3450 2750 50  0001 C CNN
 	1    3450 2750
@@
 F 0 "C4" H 3775 2850 50  0000 L CNN
 F 1 "1uF" H 3775 2650 50  0000 L CNN
-F 2 "footprints:C_0603" H 3788 2600 50  0001 C CNN
+F 2 "beetje_footprints:C_0603" H 3788 2600 50  0001 C CNN
 F 3 "" H 3750 2750 50  0001 C CNN
 	1    3750 2750
@@
 F 0 "D5" H 2650 2200 50  0000 C CNN
 F 1 "MBR120" H 2650 2000 50  0000 C CNN
-F 2 "footprints:D_SOD-123F" H 2650 2100 50  0001 C CNN
+F 2 "beetje_footprints:D_SOD-123F" H 2650 2100 50  0001 C CNN
 F 3 "" H 2650 2100 50  0001 C CNN
 	1    2650 2100
@@
 F 0 "D4" H 2300 2200 50  0000 C CNN
 F 1 "MBR120" H 2300 2000 50  0000 C CNN
-F 2 "footprints:D_SOD-123F" H 2300 2100 50  0001 C CNN
+F 2 "beetje_footprints:D_SOD-123F" H 2300 2100 50  0001 C CNN
 F 3 "" H 2300 2100 50  0001 C CNN
 	1    2300 2100
@@
 F 0 "SW1" H 4550 2900 50  0000 L CNN
 F 1 "RST" H 4500 2740 50  0000 C CNN
-F 2 "footprints:EVQ-P7A" H 4500 3000 50  0001 C CNN
+F 2 "beetje_footprints:EVQ-P7A" H 4500 3000 50  0001 C CNN
 F 3 "" H 4500 3000 50  0001 C CNN
 	1    4500 2800
@@
 F 0 "R3" V 8630 4750 50  0000 C CNN
 F 1 "1K" V 8550 4750 50  0000 C CNN
-F 2 "footprints:R_0603" V 8480 4750 50  0001 C CNN
+F 2 "beetje_footprints:R_0603" V 8480 4750 50  0001 C CNN
 F 3 "" H 8550 4750 50  0001 C CNN
 	1    8550 4750
@@
 F 0 "D3" H 8550 5250 50  0000 C CNN
 F 1 "D13" H 8550 5050 50  0000 C CNN
-F 2 "footprints:LED_0603" H 8550 5150 50  0001 C CNN
+F 2 "beetje_footprints:LED_0603" H 8550 5150 50  0001 C CNN
 F 3 "" H 8550 5150 50  0001 C CNN
 	1    8550 5150
@@
 F 0 "Y1" H 4700 3525 50  0000 C CNN
 F 1 "8 Mhz" H 4700 3450 50  0000 C CNN
-F 2 "footprints:Resonator_SMD_CTSC_1.3mmx3.2mm" H 4675 3300 50  0001 C CNN
+F 2 "beetje_footprints:Resonator_SMD_CTSC_1.3mmx3.2mm" H 4675 3300 50  0001 C CNN
 F 3 "" H 4675 3300 50  0001 C CNN
 	1    4700 3300
@@
 F 0 "R2" V 9230 5150 50  0000 C CNN
 F 1 "1K" V 9150 5150 50  0000 C CNN
-F 2 "footprints:R_0603" V 9080 5150 50  0001 C CNN
+F 2 "beetje_footprints:R_0603" V 9080 5150 50  0001 C CNN
 F 3 "" H 9150 5150 50  0001 C CNN
 	1    9150 5150
@@
 F 0 "D2" H 9150 4900 50  0000 C CNN
 F 1 "RX" H 9150 4700 50  0000 C CNN
-F 2 "footprints:LED_0603" H 9150 4800 50  0001 C CNN
+F 2 "beetje_footprints:LED_0603" H 9150 4800 50  0001 C CNN
 F 3 "" H 9150 4800 50  0001 C CNN
 	1    9150 4800
@@
 F 0 "R1" V 8930 5150 50  0000 C CNN
 F 1 "1K" V 8850 5150 50  0000 C CNN
-F 2 "footprints:R_0603" V 8780 5150 50  0001 C CNN
+F 2 "beetje_footprints:R_0603" V 8780 5150 50  0001 C CNN
 F 3 "" H 8850 5150 50  0001 C CNN
 	1    8850 5150
@@
 F 0 "D1" H 8850 4900 50  0000 C CNN
 F 1 "TX" H 8850 4700 50  0000 C CNN
-F 2 "footprints:LED_0603" H 8850 4800 50  0001 C CNN
+F 2 "beetje_footprints:LED_0603" H 8850 4800 50  0001 C CNN
 F 3 "" H 8850 4800 50  0001 C CNN
 	1    8850 4800
@@
 F 0 "J4" H 3000 5850 50  0000 C CNN
 F 1 "Beetje Top" H 2850 4950 50  0000 C CNN
-F 2 "footprints:Beetje_Top" H 3000 5450 50  0001 C CNN
+F 2 "beetje_footprints:Beetje_Top" H 3000 5450 50  0001 C CNN
 F 3 "" H 3000 5450 50  0001 C CNN
 	1    3000 5450
@@
 F 0 "J2" H 3650 5650 50  0000 C CNN
 F 1 "Beetje Bottom" H 3400 4950 50  0000 C CNN
-F 2 "footprints:Beetje_Bottom" H 3650 5350 50  0001 C CNN
+F 2 "beetje_footprints:Beetje_Bottom" H 3650 5350 50  0001 C CNN
 F 3 "" H 3650 5350 50  0001 C CNN
 	1    3650 5350
@@
 F 0 "JMP1" V 3130 1950 50  0000 C CNN
 F 1 "5V" V 3050 1950 50  0000 C CNN
-F 2 "footprints:Jumper" V 2980 1950 50  0001 C CNN
+F 2 "beetje_footprints:Jumper" V 2980 1950 50  0001 C CNN
 F 3 "" H 3050 1950 50  0001 C CNN
 	1    3050 1950
@@
 F 0 "F1" V 4400 3850 50  0000 C CNN
 F 1 "Polyfuse" V 4550 4100 50  0000 C CNN
-F 2 "footprints:R_1206" H 4550 3750 50  0001 L CNN
+F 2 "beetje_footprints:R_1206" H 4550 3750 50  0001 L CNN
 F 3 "" H 4500 3950 50  0001 C CNN
 	1    4500 3950
@@
 F 0 "SW2" H 8200 5000 50  0000 L CNN
 F 1 "D4" H 8150 4840 50  0000 C CNN
-F 2 "footprints:EVQ-P7A" H 8150 5100 50  0001 C CNN
+F 2 "beetje_footprints:EVQ-P7A" H 8150 5100 50  0001 C CNN
 F 3 "" H 8150 5100 50  0001 C CNN
 	1    8150 4900
@@
 F 0 "CON1" H 7845 1940 50  0000 C CNN
 F 1 "AVR-ISP-6" H 7685 1470 50  0000 L BNN
-F 2 "footprints:Pin_Header_Straight_2x03_Pitch2.54mm" V 7430 1740 50  0001 C CNN
+F 2 "beetje_footprints:Pin_Header_Straight_2x03_Pitch2.54mm" V 7430 1740 50  0001 C CNN
 F 3 "" H 7925 1700 50  0001 C CNN
 	1    7950 1700
@@
 F 0 "R4" V 8180 3500 50  0000 C CNN
 F 1 "4K7" V 8100 3500 50  0000 C CNN
-F 2 "footprints:R_0603" V 8030 3500 50  0001 C CNN
+F 2 "beetje_footprints:R_0603" V 8030 3500 50  0001 C CNN
 F 3 "" H 8100 3500 50  0001 C CNN
 	1    8100 3500
@@
 F 0 "R5" V 8380 3500 50  0000 C CNN
 F 1 "4K7" V 8300 3500 50  0000 C CNN
-F 2 "footprints:R_0603" V 8230 3500 50  0001 C CNN
+F 2 "beetje_footprints:R_0603" V 8230 3500 50  0001 C CNN
 F 3 "" H 8300 3500 50  0001 C CNN
 	1    8300 3500
