File: projects/Beetje/design_files_press_diff/project.kicad_pcb (KiCad board)
At the start: 2 copper layers, 25.4 x 25.4 mm, 11 parts, among them J2 Beetje_Bottom, J4 Beetje_Top, U1 MP3V5010, U2 MCP3021

Commit message: Updates
Parts:
- added REF**: TSSOP-28_4.4x9.7mm_Pitch0.65mm, Housings_SSOP:TSSOP-28_4.4x9.7mm_Pitch0.65mm, F.Cu at (173.9, 105.3)
- added REF**: SSOP-24_5.3x8.2mm_Pitch0.65mm, Housings_SSOP:SSOP-24_5.3x8.2mm_Pitch0.65mm, F.Cu at (173.2, 92.8)
Routing:
- net GND: track 64.7 -> 68.6 mm, vias 1 -> 2
- net VCC: track 60.1 -> 57.9 mm
Other:
- outline, holes or cut-outs redrawn
- board text added: "Rev 0.1 Sep 2018"
- board text removed: "Rev 0.0 Sep 2018"

Commit message: Updates
Parts:
- removed REF**: TSSOP-28_4.4x9.7mm_Pitch0.65mm, Housings_SSOP:TSSOP-28_4.4x9.7mm_Pitch0.65mm
- removed REF**: SSOP-24_5.3x8.2mm_Pitch0.65mm, Housings_SSOP:SSOP-24_5.3x8.2mm_Pitch0.65mm
- moved R1 19.5 mm to (127.6, 108.0), turned to 0 degrees
- moved R2 18.8 mm to (127.6, 105.4), turned to 0 degrees
- moved C3 18.8 mm to (127.0, 110.5), turned to 180 degrees
- moved U2 18.8 mm to (127.0, 101.6), turned to 270 degrees
- moved JP1 3.91 mm to (138.4, 109.2)
- moved JP2 3.91 mm to (138.4, 105.4), turned to 180 degrees
- moved C1 1.27 mm to (127.0, 113.0)
- moved C2 1.27 mm to (127.0, 97.8)
- moved U1 0.63 mm to (137.2, 105.4), turned to 270 degrees
Routing:
- net GND: track 68.6 -> 24.2 mm, vias 2 -> 0
- net VCC: track 57.9 -> 37.8 mm
- net /SDA: track 28.4 -> 17.5 mm, vias 1 -> 0
- net /AIN: track 5.95 -> 16.3 mm
- net /A0: track 28.3 -> 35.7 mm, vias 1 -> 2
- net /SCL: track 19.5 -> 17.9 mm, vias 1 -> 0
Other:
- outline, holes or cut-outs redrawn
- board text added: "Ain I2C 0 1 1 0"
- board text added: "I2C Addr:"
- board text added: "Rev 0.2 Sep 2018"
- board text removed: "Alog I2C 0 1 1 0"
- board text removed: "Rev 0.1 Sep 2018"
