File: projects/Beetje/design_files_CNTRL-ATL-DEL/project.sch (KiCad schematic (older format))
At the start: 6 parts, among them J2 Beetje_Bottom, J4 Beetje_Top, SW1 SW_Push

Commit message: Updates
Parts:
- removed C1: 0.1uF, footprints:C_0603, symbol C
- removed D1: LED, footprints:LED_0603, symbol LED
- removed R1: 1K, footprints:R_0603, symbol R
- removed SW1: SW_Push, footprints:SW_SPST_KMR2, symbol SW_Push
- added SW2: SWITCH_PUSH, footprints:CHERRY_PCB_100H, symbol SWITCH_PUSH
- J2: footprint footprints:Pin_Header_Straight_1x06_Pitch2.54mm -> footprints:Beetje_Bottom
- J4: footprint footprints:Pin_Header_Straight_1x08_Pitch2.54mm -> footprints:Beetje_Top
Connections:
- wire segments 21 -> 17
Other:
- note added: "https://github.com/BathroomEpiphanies/KiCAD-Keyboard-Tutorial"
Changed lines of the file:
@@
 LIBS:contrib
 LIBS:valves
+LIBS:components
 LIBS:project-cache
 EELAYER 25 0
@@
 $EndDescr
 $Comp
-L VBUS #PWR01
+L VBUS #PWR1
 U 1 1 5B3FDCD2
 P 1450 1350
-F 0 "#PWR01" H 1450 1200 50  0001 C CNN
+F 0 "#PWR1" H 1450 1200 50  0001 C CNN
 F 1 "VBUS" H 1450 1500 50  0000 C CNN
 F 2 "" H 1450 1350 50  0001 C CNN
@@
 $EndComp
 $Comp
-L GND #PWR02
+L GND #PWR10
 U 1 1 5B3FDCF5
 P 2700 1350
-F 0 "#PWR02" H 2700 1100 50  0001 C CNN
+F 0 "#PWR10" H 2700 1100 50  0001 C CNN
 F 1 "GND" H 2700 1200 50  0000 C CNN
 F 2 "" H 2700 1350 50  0001 C CNN
@@
 $EndComp
 $Comp
-L PWR_FLAG #FLG03
+L PWR_FLAG #FLG1
 U 1 1 5B3FDD3A
 P 1450 1350
-F 0 "#FLG03" H 1450 1425 50  0001 C CNN
+F 0 "#FLG1" H 1450 1425 50  0001 C CNN
 F 1 "PWR_FLAG" H 1450 1500 50  0000 C CNN
 F 2 "" H 1450 1350 50  0001 C CNN
@@
 $EndComp
 $Comp
-L PWR_FLAG #FLG04
+L PWR_FLAG #FLG3
 U 1 1 5B3FDD50
 P 2250 1350
-F 0 "#FLG04" H 2250 1425 50  0001 C CNN
+F 0 "#FLG3" H 2250 1425 50  0001 C CNN
 F 1 "PWR_FLAG" H 2250 1500 50  0000 C CNN
 F 2 "" H 2250 1350 50  0001 C CNN
@@
 $EndComp
 $Comp
-L PWR_FLAG #FLG05
+L PWR_FLAG #FLG4
 U 1 1 5B3FDD67
 P 2700 1350
-F 0 "#FLG05" H 2700 1425 50  0001 C CNN
+F 0 "#FLG4" H 2700 1425 50  0001 C CNN
 F 1 "PWR_FLAG" H 2700 1500 50  0000 C CNN
 F 2 "" H 2700 1350 50  0001 C CNN
@@
 	1    0    0    -1
 $EndComp
-Wire Wire Line
-	2400 6650 2200 6650
-Wire Wire Line
-	2200 6750 2400 6750
-Wire Wire Line
-	2400 6850 2200 6850
-Wire Wire Line
-	2400 6950 2200 6950
-Wire Wire Line
-	2400 7050 2200 7050
-Wire Wire Line
-	2400 7150 2200 7150
-Wire Wire Line
-	2400 7250 2350 7250
-Wire Wire Line
-	2400 7350 2350 7350
-$Comp
-L +BATT #PWR06
+$Comp
+L +BATT #PWR7
 U 1 1 5B402C38
 P 2350 7250
-F 0 "#PWR06" H 2350 7100 50  0001 C CNN
+F 0 "#PWR7" H 2350 7100 50  0001 C CNN
 F 1 "+BATT" V 2350 7500 50  0000 C CNN
 F 2 "" H 2350 7250 50  0001 C CNN
@@
 $EndComp
 $Comp
-L VBUS #PWR07
+L VBUS #PWR8
 U 1 1 5B402FA5
 P 2350 7350
-F 0 "#PWR07" H 2350 7200 50  0001 C CNN
+F 0 "#PWR8" H 2350 7200 50  0001 C CNN
 F 1 "VBUS" V 2350 7550 50  0000 C CNN
 F 2 "" H 2350 7350 50  0001 C CNN
@@
 MISO
 $Comp
-L GND #PWR08
+L GND #PWR12
 U 1 1 5B41D2F5
 P 3500 7150
-F 0 "#PWR08" H 3500 6900 50  0001 C CNN
+F 0 "#PWR12" H 3500 6900 50  0001 C CNN
 F 1 "GND" V 3500 6950 50  0000 C CNN
 F 2 "" H 3500 7150 50  0001 C CNN
@@
 F 0 "J4" H 2600 7350 50  0000 C CNN
 F 1 "Beetje_Top" H 2400 6450 50  0000 C CNN
-F 2 "footprints:Pin_Header_Straight_1x08_Pitch2.54mm" H 2600 6950 50  0001 C CNN
+F 2 "footprints:Beetje_Top" H 2600 6950 50  0001 C CNN
 F 3 "" H 2600 6950 50  0001 C CNN
 	1    2600 6950
@@
 F 0 "J2" H 3250 7150 50  0000 C CNN
 F 1 "Beetje_Bottom" H 3000 6450 50  0000 C CNN
-F 2 "footprints:Pin_Header_Straight_1x06_Pitch2.54mm" H 3250 6850 50  0001 C CNN
+F 2 "footprints:Beetje_Bottom" H 3250 6850 50  0001 C CNN
 F 3 "" H 3250 6850 50  0001 C CNN
 	1    3250 6850
 	-1   0    0    -1
 $EndComp
-Wire Wire Line
-	3450 6650 3750 6650
-Wire Wire Line
-	3450 6750 3750 6750
-Wire Wire Line
-	3450 6850 3750 6850
-Wire Wire Line
-	3450 6950 3750 6950
-Wire Wire Line
-	3450 7050 3500 7050
-Wire Wire Line
-	3450 7150 3500 7150
-$Comp
-L VCC #PWR09
+$Comp
+L VCC #PWR6
 U 1 1 5B6E5416
 P 2250 1350
-F 0 "#PWR09" H 2250 1200 50  0001 C CNN
+F 0 "#PWR6" H 2250 1200 50  0001 C CNN
 F 1 "VCC" H 2250 1500 50  0000 C CNN
 F 2 "" H 2250 1350 50  0001 C CNN
@@
 $EndComp
 $Comp
-L PWR_FLAG #FLG010
+L PWR_FLAG #FLG2
 U 1 1 5B3FFE6E
 P 1850 1350
-F 0 "#FLG010" H 1850 1425 50  0001 C CNN
+F 0 "#FLG2" H 1850 1425 50  0001 C CNN
 F 1 "PWR_FLAG" H 1850 1500 50  0000 C CNN
 F 2 "" H 1850 1350 50  0001 C CNN
@@
 $EndComp
 $Comp
-L +BATT #PWR011
+L +BATT #PWR4
 U 1 1 5B6E4208
 P 1850 1350
-F 0 "#PWR011" H 1850 1200 50  0001 C CNN
+F 0 "#PWR4" H 1850 1200 50  0001 C CNN
 F 1 "+BATT" V 1850 1600 50  0000 C CNN
 F 2 "" H 1850 1350 50  0001 C CNN
@@
 	-1   0    0    1
 $EndComp
-$Comp
-L LED D1
-U 1 1 5B773B85
-P 2450 1900
-F 0 "D1" H 2450 2000 50  0000 C CNN
-F 1 "LED" H 2450 1800 50  0000 C CNN
-F 2 "footprints:LED_0603" H 2450 1900 50  0001 C CNN
-F 3 "" H 2450 1900 50  0001 C CNN
-	1    2450 1900
-	0    -1   -1   0
-$EndComp
-$Comp
-L R R1
-U 1 1 5B773C20
-P 2450 2250
-F 0 "R1" V 2530 2250 50  0000 C CNN
-F 1 "1K" V 2450 2250 50  0000 C CNN
-F 2 "footprints:R_0603" V 2380 2250 50  0001 C CNN
-F 3 "" H 2450 2250 50  0001 C CNN
-	1    2450 2250
-	-1   0    0    1
-$EndComp
-$Comp
-L VCC #PWR012
-U 1 1 5B77413E
-P 1450 2050
-F 0 "#PWR012" H 1450 1900 50  0001 C CNN
-F 1 "VCC" H 1450 2200 50  0000 C CNN
-F 2 "" H 1450 2050 50  0001 C CNN
-F 3 "" H 1450 2050 50  0001 C CNN
-	1    1450 2050
-	1    0    0    -1
-$EndComp
-$Comp
-L GND #PWR013
-U 1 1 5B774158
-P 1450 2450
-F 0 "#PWR013" H 1450 2200 50  0001 C CNN
-F 1 "GND" H 1450 2300 50  0000 C CNN
-F 2 "" H 1450 2450 50  0001 C CNN
-F 3 "" H 1450 2450 50  0001 C CNN
-	1    1450 2450
-	1    0    0    -1
-$EndComp
-$Comp
-L C C1
-U 1 1 5B77416F
-P 1450 2250
-F 0 "C1" H 1475 2350 50  0000 L CNN
-F 1 "0.1uF" H 1475 2150 50  0000 L CNN
-F 2 "footprints:C_0603" H 1488 2100 50  0001 C CNN
-F 3 "" H 1450 2250 50  0001 C CNN
-	1    1450 2250
-	1    0    0    -1
-$EndComp
-Wire Wire Line
-	1450 2050 1450 2100
-Wire Wire Line
-	1450 2400 1450 2450
-Wire Notes Line
-	1750 7550 4400 7550
-Wire Notes Line
-	4400 6350 1750 6350
 Text Notes 1800 6500 0    60   ~ 0
 Beetje Footprint Rev 0.3
-Wire Notes Line
-	1750 6350 1750 7550
-Wire Notes Line
-	4400 7550 4400 6350
-$Comp
-L SW_Push SW1
-U 1 1 5B7EE011
-P 2000 2200
-F 0 "SW1" H 2050 2300 50  0000 L CNN
-F 1 "SW_Push" H 2000 2140 50  0000 C CNN
-F 2 "footprints:SW_SPST_KMR2" H 2000 2400 50  0001 C CNN
-F 3 "" H 2000 2400 50  0001 C CNN
-	1    2000 2200
-	0    1    1    0
-$EndComp
-$Comp
-L GND #PWR014
-U 1 1 5B7EE086
-P 2000 2450
-F 0 "#PWR014" H 2000 2200 50  0001 C CNN
-F 1 "GND" H 2000 2300 50  0000 C CNN
-F 2 "" H 2000 2450 50  0001 C CNN
-F 3 "" H 2000 2450 50  0001 C CNN
-	1    2000 2450
-	1    0    0    -1
-$EndComp
-Wire Wire Line
-	2000 2450 2000 2400
-Wire Wire Line
-	2000 2000 2000 1900
-$Comp
-L GND #PWR015
-U 1 1 5B7EE8E2
-P 2450 2450
-F 0 "#PWR015" H 2450 2200 50  0001 C CNN
-F 1 "GND" H 2450 2300 50  0000 C CNN
-F 2 "" H 2450 2450 50  0001 C CNN
-F 3 "" H 2450 2450 50  0001 C CNN
-	1    2450 2450
-	1    0    0    -1
-$EndComp
-Wire Wire Line
-	2450 1750 2450 1650
-Wire Wire Line
-	2450 2050 2450 2100
-Wire Wire Line
-	2450 2400 2450 2450
 Text Label 3650 6750 0    60   ~ 0
 D6
 $Comp
-L VCC #PWR016
+L VCC #PWR11
 U 1 1 5B996B2A
 P 3500 7050
-F 0 "#PWR016" H 3500 6900 50  0001 C CNN
+F 0 "#PWR11" H 3500 6900 50  0001 C CNN
 F 1 "VCC" V 3500 7250 50  0000 C CNN
 F 2 "" H 3500 7050 50  0001 C CNN
@@
 	0    1    1    0
 $EndComp
+Text Notes 1750 6100 0    60   ~ 0
+https://github.com/BathroomEpiphanies/KiCAD-Keyboard-Tutorial
+$Comp
+L SWITCH_PUSH SW2
+U 1 1 5B997630
+P 5000 3650
+F 0 "SW2" H 5150 3760 50  0000 C CNN
+F 1 "SWITCH_PUSH" H 5000 3570 50  0000 C CNN
+F 2 "footprints:CHERRY_PCB_100H" H 5000 3650 60  0001 C CNN
+F 3 "" H 5000 3650 60  0001 C CNN
+	1    5000 3650
+	1    0    0    -1
+$EndComp
+Wire Wire Line
+	2400 6650 2200 6650
+Wire Wire Line
+	2200 6750 2400 6750
+Wire Wire Line
+	2400 6850 2200 6850
+Wire Wire Line
+	2400 6950 2200 6950
+Wire Wire Line
+	2400 7050 2200 7050
+Wire Wire Line
+	2400 7150 2200 7150
+Wire Wire Line
+	2400 7250 2350 7250
+Wire Wire Line
+	2400 7350 2350 7350
+Wire Wire Line
+	3450 6650 3750 6650
+Wire Wire Line
+	3450 6750 3750 6750
+Wire Wire Line
+	3450 6850 3750 6850
+Wire Wire Line
+	3450 6950 3750 6950
+Wire Wire Line
+	3450 7050 3500 7050
+Wire Wire Line
+	3450 7150 3500 7150
+Wire Notes Line
+	1750 7550 4400 7550
+Wire Notes Line
+	4400 6350 1750 6350
+Wire Notes Line
+	1750 6350 1750 7550
+Wire Notes Line
+	4400 7550 4400 6350
+Wire Wire Line
+	4700 3650 4400 3650
+Wire Wire Line
+	5300 3650 5700 3650
+Wire Wire Line
+	5700 3650 5700 3950
+$Comp
+L GND #PWR13
+U 1 1 5B997746
+P 5700 3950
+F 0 "#PWR13" H 5700 3700 50  0001 C CNN
+F 1 "GND" H 5700 3800 50  0000 C CNN
+F 2 "" H 5700 3950 50  0001 C CNN
+F 3 "" H 5700 3950 50  0001 C CNN
+	1    5700 3950
+	1    0    0    -1
+$EndComp
+Text Label 4400 3650 0    60   ~ 0
+D9
 $EndSCHEMATC
