File: projects/Arduino/Arduino/Arduino.sch (KiCad schematic (older format))
At the start: 43 parts, among them CON1 ISP, J1 USB_B, J2 BARREL_JACK, J3 PWR_SEL, P1 Power, P2 Analog, P3 Digital, P4 Digital, P5 CONN_01X01, P6 CONN_01X01, P7 CONN_01X01, P8 CONN_01X01, SW1 Reset, U1 LM7805, U2 FT231XS, U3 74LS125, U4 MCP1700T, U5 ATMEGA328P-PU, Y1 Resonator

Commit message: Updates
Parts:
- removed U1: LM7805, symbol LM7805
- added U1: LM7805, TO_SOT_Packages_THT:TO-220_Vertical, symbol LM7805_TO220
- C1: footprint Capacitors_THT:CP_Radial_D10.0mm_P5.00mm -> Capacitors_THT:CP_Radial_D4.0mm_P1.50mm
- C2, C3: footprint (none) -> Capacitors_THT:C_Disc_D3.8mm_W2.6mm_P2.50mm
- C4: footprint Capacitors_THT:CP_Radial_D8.0mm_P3.50mm -> Capacitors_THT:C_Disc_D3.8mm_W2.6mm_P2.50mm
- C5: renamed from C8; footprint (none) -> Capacitors_THT:C_Disc_D3.8mm_W2.6mm_P2.50mm
- C6, C7: footprint (none) -> Capacitors_THT:C_Disc_D4.3mm_W1.9mm_P5.00mm
- C8: renamed from C5; footprint (none) -> Capacitors_THT:C_Disc_D4.3mm_W1.9mm_P5.00mm
- CON1: footprint AVR-ISP-6 -> Pin_Headers:Pin_Header_Straight_2x03_Pitch2.54mm
- D1: footprint (none) -> Diodes_THT:D_DO-41_SOD81_P10.16mm_Horizontal
- D13, D2, D3: footprint (none) -> LEDs:LED_D3.0mm
- D4: value TX -> RX; footprint (none) -> LEDs:LED_D3.0mm
- F1: footprint (none) -> Capacitors_THT:C_Disc_D7.5mm_W4.4mm_P5.00mm
- J3: footprint (none) -> Pin_Headers:Pin_Header_Straight_1x03_Pitch2.54mm
- SW1: footprint (none) -> Buttons_Switches_THT:SW_PUSH_6mm
- Y1: footprint (none) -> Crystals:Resonator-3pin_w7.0mm_h2.5mm
Connections:
- wire segments 182 -> 158

Commit message: Updates
Parts:
- C1: footprint Capacitors_THT:CP_Radial_D4.0mm_P1.50mm -> footprints:CP_Radial_D4.0mm_P1.50mm
- C2, C3, C4, C5: footprint Capacitors_THT:C_Disc_D3.8mm_W2.6mm_P2.50mm -> footprints:C_Disc_D3.8mm_W2.6mm_P2.50mm
- C6, C7, C8: footprint Capacitors_THT:C_Disc_D4.3mm_W1.9mm_P5.00mm -> footprints:C_Disc_D4.3mm_W1.9mm_P5.00mm
- CON1: footprint Pin_Headers:Pin_Header_Straight_2x03_Pitch2.54mm -> footprints:Pin_Header_Straight_2x03_Pitch2.54mm
- D1: value D -> Schottky; footprint Diodes_THT:D_DO-41_SOD81_P10.16mm_Horizontal -> footprints:D_DO-41_SOD81_P10.16mm_Horizontal
- D13, D2, D3, D4: footprint LEDs:LED_D3.0mm -> footprints:LED_D3.0mm
- F1: value Polyfuse -> PTC Fuse; footprint Capacitors_THT:C_Disc_D7.5mm_W4.4mm_P5.00mm -> footprints:C_Disc_D7.5mm_W4.4mm_P5.00mm
- J1: footprint Connectors:USB_B -> footprints:USB_B
- J2: footprint Connectors:BARREL_JACK -> footprints:BARREL_JACK
- J3: footprint Pin_Headers:Pin_Header_Straight_1x03_Pitch2.54mm -> footprints:Pin_Header_Straight_1x03_Pitch2.54mm
- P1, P4: footprint Socket_Arduino_Uno:Socket_Strip_Arduino_1x08 -> footprints:Socket_Strip_Arduino_1x08
- P2: footprint Socket_Arduino_Uno:Socket_Strip_Arduino_1x06 -> footprints:Socket_Strip_Arduino_1x06
- P3: footprint Socket_Arduino_Uno:Socket_Strip_Arduino_1x10 -> footprints:Socket_Strip_Arduino_1x10
- P5, P6, P7, P8: footprint Socket_Arduino_Uno:Arduino_1pin -> footprints:Arduino_1pin
- R1, R13, R2, R5, R6, R7, R8, R9: footprint Resistors_THT:R_Axial_DIN0204_L3.6mm_D1.6mm_P7.62mm_Horizontal -> footprints:R_Axial_DIN0204_L3.6mm_D1.6mm_P7.62mm_Horizontal
- R3, R4: value 470R -> 470; footprint Resistors_THT:R_Axial_DIN0204_L3.6mm_D1.6mm_P7.62mm_Horizontal -> footprints:R_Axial_DIN0204_L3.6mm_D1.6mm_P7.62mm_Horizontal
- SW1: footprint Buttons_Switches_THT:SW_PUSH_6mm -> footprints:SW_PUSH_6mm
- U1: footprint TO_SOT_Packages_THT:TO-220_Vertical -> footprints:TO-220-3_Horizontal
- U2: footprint Housings_SSOP:QSOP-20_3.9x8.7mm_Pitch0.635mm -> footprints:DIP-20_W7.62mm
- U3: footprint Housings_DIP:DIP-14_W7.62mm -> footprints:DIP-14_W7.62mm
- U4: footprint TO_SOT_Packages_THT:TO-92_Inline_Wide -> footprints:TO-92_Inline_Wide
- U5: footprint Housings_DIP:DIP-28_W7.62mm -> footprints:DIP-28_W7.62mm
- Y1: value Resonator -> 16Mhz; footprint Crystals:Resonator-3pin_w7.0mm_h2.5mm -> footprints:Resonator-3pin_w7.0mm_h2.5mm
Connections:
- net labels added: D+, D-
- net labels removed: 9, A5(SDA)
Other:
- moved on the sheet: C5, P1, P2, P3, P4, P5, P6, P7, P8, U5, Y1

Commit message: Updates
Connections:
- net labels added: 10(SS), 11(MOSI)
- net labels removed: 10(**/SS), 11(**/MOSI)
Changed lines of the file:
@@
 Text Label 9950 2000 0    60   ~ 0
 9(**)
-Text Label 9900 1900 0    60   ~ 0
-10(**/SS)
-Text Label 9900 1800 0    60   ~ 0
-11(**/MOSI)
-Text Label 9900 1700 0    60   ~ 0
-12(MISO)
-Text Label 9900 1600 0    60   ~ 0
-13(SCK)
 Text Label 9900 1400 0    60   ~ 0
 AREF
@@
 	1    0    0    -1
 $EndComp
-Text Label 8300 1800 0    60   ~ 0
-Reset
 $Comp
 L +3.3V #PWR01
@@
 Wire Wire Line
 	7250 4750 7500 4750
-Text Label 7250 3900 0    60   ~ 0
-Reset
 Text Label 7250 2450 0    60   ~ 0
 8
 Text Label 7250 2550 0    60   ~ 0
 9(**)
-Text Label 7250 2650 0    60   ~ 0
-10(**/SS)
-Text Label 7250 2750 0    60   ~ 0
-11(**/MOSI)
-Text Label 7250 2850 0    60   ~ 0
-12(MISO)
-Text Label 7250 2950 0    60   ~ 0
-13(SCK)
 Text Label 7250 3300 0    60   ~ 0
 A0
@@
 Wire Wire Line
 	6350 1400 5650 1400
-Text Label 5650 1400 0    60   ~ 0
-Reset
-Text Label 5650 1300 0    60   ~ 0
-13(SCK)
-Text Label 5650 1200 0    60   ~ 0
-12(MISO)
-Text Label 6900 1300 0    60   ~ 0
-11(**/MOSI)
 $Comp
 L VCC #PWR023
@@
 Wire Wire Line
 	4250 3700 4500 3700
-Text Label 4250 3700 0    60   ~ 0
-Reset
 $Comp
 L 74LS125 U3
@@
 Wire Notes Line
 	8250 3450 10500 3450
+Text Label 4300 3700 0    60   ~ 0
+Reset
+Text Label 7250 3900 0    60   ~ 0
+Reset
+Text Label 5650 1400 0    60   ~ 0
+Reset
+Text Label 8300 1800 0    60   ~ 0
+Reset
+Text Label 6950 1300 0    60   ~ 0
+11(MOSI)
+Text Label 7250 2750 0    60   ~ 0
+11(MOSI)
+Text Label 9950 1800 0    60   ~ 0
+11(MOSI)
+Text Label 9950 1700 0    60   ~ 0
+12(MISO)
+Text Label 5650 1200 0    60   ~ 0
+12(MISO)
+Text Label 7250 2850 0    60   ~ 0
+12(MISO)
+Text Label 9950 1600 0    60   ~ 0
+13(SCK)
+Text Label 5650 1300 0    60   ~ 0
+13(SCK)
+Text Label 7250 2950 0    60   ~ 0
+13(SCK)
+Text Label 7250 2650 0    60   ~ 0
+10(SS)
+Text Label 9950 1900 0    60   ~ 0
+10(SS)
+Connection ~ 3000 6350
 $EndSCHEMATC
