File: projects/Beetje/design_files_EEPROM/project.sch (KiCad schematic (older format))
At the start: 7 parts, among them J2 Beetje_Bottom, J4 Beetje_Top, U1 24LC1025

Commit message: updates
Parts:
- removed JP1: Jumper, footprints:Jumper, symbol Jumper_NO_Small
- added U2, U3, U4: 24LC1025, Housings_SOIC:SOIC-8_3.9x4.9mm_Pitch1.27mm, symbol 24LC1025
Connections:
- wire segments 30 -> 59
Other:
- moved on the sheet: R1, R2, U1

Commit message: Updates
Connections:
- net labels added: D6
- net labels removed: A1
Other:
- note added: "Beetje Rev. 3Footprint"
- note removed: "Beetje Footprint"
- note removed: "CS"
- note removed: "D2\nD3\nD15\nD14\nD16"
- note removed: "DO\nDI\nCLK"
Changed lines of the file:
@@
 	2400 7150 2200 7150
 Wire Wire Line
-	2400 7250 2200 7250
+	2400 7250 2350 7250
 Wire Wire Line
-	2400 7350 2200 7350
+	2400 7350 2350 7350
 $Comp
 L +BATT #PWR06
 U 1 1 5B402C38
-P 2200 7050
-F 0 "#PWR06" H 2200 6900 50  0001 C CNN
-F 1 "+BATT" V 2200 7300 50  0000 C CNN
-F 2 "" H 2200 7050 50  0001 C CNN
-F 3 "" H 2200 7050 50  0001 C CNN
-	1    2200 7050
+P 2350 7250
+F 0 "#PWR06" H 2350 7100 50  0001 C CNN
+F 1 "+BATT" V 2350 7500 50  0000 C CNN
+F 2 "" H 2350 7250 50  0001 C CNN
+F 3 "" H 2350 7250 50  0001 C CNN
+	1    2350 7250
 	0    -1   -1   0
 $EndComp
@@
 L VBUS #PWR07
 U 1 1 5B402FA5
-P 2200 7350
-F 0 "#PWR07" H 2200 7200 50  0001 C CNN
-F 1 "VBUS" V 2200 7550 50  0000 C CNN
-F 2 "" H 2200 7350 50  0001 C CNN
-F 3 "" H 2200 7350 50  0001 C CNN
-	1    2200 7350
+P 2350 7350
+F 0 "#PWR07" H 2350 7200 50  0001 C CNN
+F 1 "VBUS" V 2350 7550 50  0000 C CNN
+F 2 "" H 2350 7350 50  0001 C CNN
+F 3 "" H 2350 7350 50  0001 C CNN
+	1    2350 7350
 	0    -1   -1   0
 $EndComp
+Text Label 2200 6850 0    60   ~ 0
+D10
 Text Label 2200 6750 0    60   ~ 0
-D10
-Text Label 3650 6650 0    60   ~ 0
 D9
 Text Label 3600 6850 0    60   ~ 0
 SCL
-Text Label 3600 6750 0    60   ~ 0
+Text Label 3600 6950 0    60   ~ 0
 SDA
 Text Label 2200 6650 0    60   ~ 0
 ~RESET
-Text Label 2200 6850 0    60   ~ 0
+Text Label 3650 6650 0    60   ~ 0
 A0
+Text Label 3650 6750 0    60   ~ 0
+D6
+Text Label 2200 7150 0    60   ~ 0
+SCK
+Text Label 2200 7050 0    60   ~ 0
+MOSI
 Text Label 2200 6950 0    60   ~ 0
-A1
-Text Label 3600 7150 0    60   ~ 0
-SCK
-Text Label 3550 7050 0    60   ~ 0
-MOSI
-Text Label 3550 6950 0    60   ~ 0
 MISO
 $Comp
 L GND #PWR08
 U 1 1 5B41D2F5
-P 2200 7250
-F 0 "#PWR08" H 2200 7000 50  0001 C CNN
-F 1 "GND" V 2200 7050 50  0000 C CNN
-F 2 "" H 2200 7250 50  0001 C CNN
-F 3 "" H 2200 7250 50  0001 C CNN
-	1    2200 7250
-	0    1    1    0
+P 3450 7150
+F 0 "#PWR08" H 3450 6900 50  0001 C CNN
+F 1 "GND" V 3450 6950 50  0000 C CNN
+F 2 "" H 3450 7150 50  0001 C CNN
+F 3 "" H 3450 7150 50  0001 C CNN
+	1    3450 7150
+	0    -1   -1   0
 $EndComp
 $Comp
@@
 P 2600 6950
 F 0 "J4" H 2600 7350 50  0000 C CNN
-F 1 "Beetje_Top" H 2600 6450 50  0000 C CNN
+F 1 "Beetje_Top" H 2450 6450 50  0000 C CNN
 F 2 "footprints:Pin_Header_Straight_1x08_Pitch2.54mm" H 2600 6950 50  0001 C CNN
 F 3 "" H 2600 6950 50  0001 C CNN
@@
 P 3250 6850
 F 0 "J2" H 3250 7150 50  0000 C CNN
-F 1 "Beetje_Bottom" H 3250 6450 50  0000 C CNN
+F 1 "Beetje_Bottom" H 3050 6450 50  0000 C CNN
 F 2 "footprints:Pin_Header_Straight_1x06_Pitch2.54mm" H 3250 6850 50  0001 C CNN
 F 3 "" H 3250 6850 50  0001 C CNN
@@
 	3450 6950 3750 6950
 Wire Wire Line
-	3450 7050 3750 7050
+	3450 7050 3450 7050
 Wire Wire Line
-	3450 7150 3750 7150
+	3450 7150 3450 7150
 $Comp
 L VCC #PWR09
@@
 L VCC #PWR010
 U 1 1 5B6E81BF
-P 2200 7150
-F 0 "#PWR010" H 2200 7000 50  0001 C CNN
-F 1 "VCC" V 2200 7350 50  0000 C CNN
-F 2 "" H 2200 7150 50  0001 C CNN
-F 3 "" H 2200 7150 50  0001 C CNN
-	1    2200 7150
-	0    -1   -1   0
+P 3450 7050
+F 0 "#PWR010" H 3450 6900 50  0001 C CNN
+F 1 "VCC" V 3450 7250 50  0000 C CNN
+F 2 "" H 3450 7050 50  0001 C CNN
+F 3 "" H 3450 7050 50  0001 C CNN
+	1    3450 7050
+	0    1    1    0
 $EndComp
 $Comp
@@
 	-1   0    0    1
 $EndComp
-Text Notes 3800 7150 0    60   ~ 0
-D2\nD3\nD15\nD14\nD16
-Text Notes 4100 7150 0    60   ~ 0
-DO\nDI\nCLK
-Text Notes 2050 6750 0    60   ~ 0
-CS
 $Comp
 L VCC #PWR013
@@
 	4400 6350 1750 6350
 Text Notes 1800 6500 0    60   ~ 0
-Beetje Footprint
+Beetje Rev. 3Footprint
 Wire Notes Line
 	1750 6350 1750 7550

Commit message: Updates
Other:
- note added: "24LC1025: 0x50\n0x54"
- note added: "CAT24M01: 0x54\n0x55"
- note added: "CAT24M01: 0x56\n0x57"
Changed lines of the file:
@@
 Wire Wire Line
 	5800 4900 5900 4900
+Text Notes 3550 3850 2    60   ~ 0
+CAT24M01: 0x54\n0x55
+Text Notes 3600 5350 2    60   ~ 0
+CAT24M01: 0x56\n0x57
+Text Notes 3550 4150 2    60   ~ 0
+24LC1025: 0x50\n0x54
 $EndSCHEMATC
