File: projects/Beetje/design_files_HBridge/project.kicad_pcb (KiCad board)
At the start: 2 copper layers, 34.3 x 25.4 mm, 16 parts, among them J1 Conn_01x02, J2 Beetje_Bottom, J3 Conn_01x02, J4 Beetje_Top, U1 TB66212FNG

Commit message: Updates
Parts:
- removed C3: 0.1uF, Capacitors_SMD:C_0805_HandSoldering
- removed C4: 10uF, Capacitors_SMD:C_1206
- removed the R1 at (127.5, 109.2)
- removed R3, R4: 10K, Resistors_SMD:R_0805_HandSoldering
- added SW1: SW_Push, Buttons_Switches_SMD:SW_SPST_PTS645, F.Cu at (119.4, 113.3)
- added U2: MCP3021, TO_SOT_Packages_SMD:SOT-23-5, F.Cu at (130.8, 111.8)
- R1: renamed from R5; value 10K -> 30K
- U1: value TB66212FNG -> DRV8871DDA; footprint Housings_SSOP:SSOP-24_5.3x8.2mm_Pitch0.65mm -> footprints:PowerSOIC-8_W3.9mm
- moved R1 16.5 mm to (128.5, 104.1), turned to 270 degrees
- moved C1 6.51 mm to (133.6, 104.1)
- moved C2 6.51 mm to (131.1, 104.1)
- moved J3 5.12 mm to (118.1, 105.4)
- moved U1 4.10 mm to (138.7, 104.1), turned to 180 degrees
- moved J1 2.62 mm to (118.1, 97.8)
- moved VAL 1.52 mm to (138.0, 110.5)
- moved R2 1.05 mm to (146.1, 111.8), turned to 270 degrees
- turned D6 to 180 degrees
Connections:
- D6 pad 1: GND -> Net-(D6-Pad1)
- D6 pad 2: Net-(D6-Pad2) -> /D6
- R1 pad 1: /D6 -> Net-(R1-Pad1)
- R2 pad 1: Net-(D6-Pad2) -> GND
- R2 pad 2: /D6 -> Net-(D6-Pad1)
- U1 pad 1: /MTR_A -> GND
- U1 pad 2: /MTR_A -> /D9
- U1 pad 3: GND -> /D10
- U1 pad 4: GND -> Net-(R1-Pad1)
- U1 pad 5: /MTR_B -> /VMTR
- U1 pad 6: /MTR_B -> /MTR_A
- U1 pad 7: /MTR_B -> GND
Routing:
- net /A0: track 0.00 -> 34.7 mm, vias 0 -> 2
- net /D6: track 36.3 -> 8.13 mm
- net VCC: track 27.5 -> 8.86 mm
- net /VMTR: track 41.7 -> 24.6 mm, vias 1 -> 0
- net Net-(R1-Pad1): track 0.00 -> 15.3 mm, vias 0 -> 2
- net /D9: track 23.1 -> 8.49 mm
- net Net-(R1-Pad2): track 14.4 -> 0.00 mm, vias 2 -> 0
- net /D10: track 18.6 -> 7.97 mm
- net /MTR_A: track 29.3 -> 23.0 mm, vias 1 -> 0
- net /SCL: track 0.00 -> 5.16 mm
- net /SDA: track 0.00 -> 4.90 mm
- net Net-(D6-Pad2): track 4.44 -> 0.00 mm
- net Net-(D6-Pad1): track 0.00 -> 3.76 mm
- net /MTR_B: track 27.3 -> 25.6 mm, vias 1 -> 0
- net GND: track 107.4 -> 106.0 mm, vias 2 -> 0
Other:
- board text added: "6-45 VDC"
- board text added: "A0"
- board text added: "Beetje H-Bridge"
- board text added: "DRV8871"
- board text added: "MCP3021 I2C: 0X49"
- board text removed: "6-15 VDC"
- board text removed: "Beetje HBridge"

Commit message: Updates
Parts:
- removed SW1: SW_Push, Buttons_Switches_SMD:SW_SPST_PTS645
- C1: footprint Capacitors_SMD:C_0805_HandSoldering -> footprints:C_0805_HandSoldering
- C2: value 10uF -> 47uF; footprint Capacitors_SMD:C_1206 -> footprints:CP_Elec_8x10
- D6: footprint LEDs:LED_0805_HandSoldering -> footprints:LED_0805_HandSoldering
- R1: value 30K -> *; footprint Resistors_SMD:R_0805_HandSoldering -> footprints:R_0805_HandSoldering
- R2: footprint Resistors_SMD:R_0805_HandSoldering -> footprints:R_0805_HandSoldering
- U2: footprint TO_SOT_Packages_SMD:SOT-23-5 -> footprints:SOT-23-5
- moved VAL 19.7 mm to (118.9, 106.2)
- moved C2 13.1 mm to (118.1, 106.0), turned to 180 degrees
- moved J3 8.89 mm to (118.1, 114.3)
- moved R1 5.95 mm to (132.3, 99.6), turned to 180 degrees
- turned C1 to 90 degrees
Routing:
- net /A0: track 34.7 -> 0.00 mm, vias 2 -> 0
- net Net-(R1-Pad1): track 15.3 -> 4.57 mm, vias 2 -> 0
- net /VMTR: track 24.6 -> 32.3 mm
- net GND: track 106.0 -> 109.7 mm
- net /MTR_B: track 25.6 -> 27.9 mm
- net /MTR_A: track 23.0 -> 24.0 mm
Other:
- board size 34.3 x 25.4 mm -> 35.6 x 25.4 mm
- board text added: "* R1 Current Limiting 18K Ohm = 3.5A 22K Ohm = 3A 33K Ohm = 2A 62K Ohm = 1A"
- board text removed: "A0"
