File: projects/Nerf/NerfMuzzleFlash/design_files/project.kicad_pcb (KiCad board)
At the start: 2 copper layers, 40 x 40 mm, 13 parts, among them J1 CONN_01X03, Q1 TN0702

Commit message: updates
Parts:
- moved D2 4.09 mm to (181.6, 78.7), turned to 290 degrees
- moved D5 3.99 mm to (153.7, 78.7), turned to 250 degrees
- moved D1 1.78 mm to (166.4, 71.1), turned to 0 degrees
- moved D3 0.45 mm to (177.8, 100.3), turned to 40 degrees
- moved D4 0.33 mm to (157.5, 100.3), turned to 140 degrees
Routing:
- net GND: track 93.2 -> 104.6 mm
- net Net-(D5-Pad2): track 6.02 -> 8.79 mm
- net Net-(D1-Pad2): track 8.55 -> 6.11 mm
- net Net-(Q1-Pad1): track 63.8 -> 65.5 mm
- net Net-(D2-Pad2): track 6.02 -> 7.42 mm
- net Net-(D3-Pad2): track 9.55 -> 8.37 mm
- added copper zone on B.Cu, net GND
- added copper zone on F.Cu, net GND
Other:
- board text added: "@TheMakersBox"
