File: projects/Nerf/NerfSwitch/design_files/project.kicad_pcb (KiCad board)
At the start: 2 copper layers, 12.7 x 12.7 mm, 3 parts, among them J1 CONN_01X02, J2 CONN_01X02, SW1 SW_SPST

Commit message: Updates
Other:
- board size 12.7 x 12.7 mm -> 10.2 x 12.7 mm
Changed lines of the file:
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@@
-(kicad_pcb (version 4) (host pcbnew 4.0.7)
+(kicad_pcb (version 4) (host pcbnew 4.0.6)
   (general
     (links 3)
     (no_connects 0)
-    (area 130.274287 93.82 156.163334 113.105001)
+    (area 142.164999 100.254999 152.475001 113.105001)
     (thickness 1.6)
-    (drawings 20)
+    (drawings 25)
     (tracks 10)
     (zones 0)
@@
     )
   )
-  (gr_text ON (at 143.51 101.6) (layer B.SilkS)
-    (effects (font (size 1.5 1.5) (thickness 0.3)) (justify mirror))
-  )
-  (gr_text - (at 152.4 109.22) (layer B.SilkS)
-    (effects (font (size 1.5 1.5) (thickness 0.3)) (justify mirror))
-  )
-  (gr_text - (at 142.24 109.22) (layer B.SilkS)
-    (effects (font (size 1.5 1.5) (thickness 0.3)) (justify mirror))
-  )
-  (gr_text + (at 152.4 103.505) (layer B.SilkS)
-    (effects (font (size 1.5 1.5) (thickness 0.3)) (justify mirror))
-  )
-  (gr_text + (at 142.24 103.505) (layer B.SilkS)
-    (effects (font (size 1.5 1.5) (thickness 0.3)) (justify mirror))
-  )
-  (gr_text ON (at 151.13 101.6) (layer F.SilkS)
-    (effects (font (size 1.5 1.5) (thickness 0.3)))
-  )
-  (gr_text - (at 152.4 109.22) (layer F.SilkS)
-    (effects (font (size 1.5 1.5) (thickness 0.3)))
-  )
-  (gr_text - (at 142.24 109.22) (layer F.SilkS)
-    (effects (font (size 1.5 1.5) (thickness 0.3)))
-  )
-  (gr_text + (at 152.4 103.505) (layer F.SilkS)
-    (effects (font (size 1.5 1.5) (thickness 0.3)))
-  )
-  (gr_text + (at 142.24 103.505) (layer F.SilkS)
-    (effects (font (size 1.5 1.5) (thickness 0.3)))
-  )
-  (gr_line (start 151.13 113.03) (end 143.51 113.03) (angle 90) (layer Edge.Cuts) (width 0.15))
-  (gr_line (start 143.51 100.33) (end 151.13 100.33) (angle 90) (layer Edge.Cuts) (width 0.15))
+  (gr_line (start 148.59 102.87) (end 146.812 101.092) (angle 90) (layer B.SilkS) (width 0.4))
+  (gr_circle (center 144.78 102.87) (end 144.907 102.743) (layer B.SilkS) (width 0.2))
+  (gr_circle (center 149.86 102.87) (end 149.987 102.743) (layer B.SilkS) (width 0.2))
+  (gr_line (start 148.59 102.87) (end 149.86 102.87) (angle 90) (layer B.SilkS) (width 0.4))
+  (gr_line (start 144.78 102.87) (end 146.05 102.87) (angle 90) (layer B.SilkS) (width 0.4))
+  (gr_line (start 144.78 100.33) (end 149.86 100.33) (angle 90) (layer Edge.Cuts) (width 0.15))
+  (gr_line (start 144.78 113.03) (end 149.86 113.03) (angle 90) (layer Edge.Cuts) (width 0.15))
+  (gr_text ON (at 144.145 101.6) (layer B.SilkS)
+    (effects (font (size 1 1) (thickness 0.2)) (justify mirror))
+  )
+  (gr_text - (at 151.13 110.49) (layer B.SilkS)
+    (effects (font (size 1.5 1.5) (thickness 0.3)) (justify mirror))
+  )
+  (gr_text - (at 143.51 110.49) (layer B.SilkS)
+    (effects (font (size 1.5 1.5) (thickness 0.3)) (justify mirror))
+  )
+  (gr_text + (at 151.13 102.87) (layer B.SilkS)
+    (effects (font (size 1.5 1.5) (thickness 0.3)) (justify mirror))
+  )
+  (gr_text + (at 143.51 102.87) (layer B.SilkS)
+    (effects (font (size 1.5 1.5) (thickness 0.3)) (justify mirror))
+  )
+  (gr_text ON (at 150.495 101.6) (layer F.SilkS)
+    (effects (font (size 1 1) (thickness 0.2)))
+  )
+  (gr_text - (at 151.13 110.49) (layer F.SilkS)
+    (effects (font (size 1.5 1.5) (thickness 0.3)))
+  )
+  (gr_text - (at 143.51 110.49) (layer F.SilkS)
+    (effects (font (size 1.5 1.5) (thickness 0.3)))
+  )
+  (gr_text + (at 151.13 102.87) (layer F.SilkS)
+    (effects (font (size 1.5 1.5) (thickness 0.3)))
+  )
+  (gr_text + (at 143.51 102.87) (layer F.SilkS)
+    (effects (font (size 1.5 1.5) (thickness 0.3)))
+  )
   (dimension 12.7 (width 0.3) (layer Dwgs.User)
     (gr_text "0.5000 in" (at 147.32 95.17) (layer Dwgs.User)
@@
     (arrow2b (pts (xy 137.16 100.33) (xy 137.746421 101.456504)))
   )
-  (gr_line (start 140.97 110.49) (end 140.97 102.87) (angle 90) (layer Edge.Cuts) (width 0.15))
-  (gr_line (start 153.67 102.87) (end 153.67 110.49) (angle 90) (layer Edge.Cuts) (width 0.15))
-  (gr_arc (start 143.51 102.87) (end 140.97 102.87) (angle 90) (layer Edge.Cuts) (width 0.15))
-  (gr_arc (start 143.51 110.49) (end 143.51 113.03) (angle 90) (layer Edge.Cuts) (width 0.15))
-  (gr_arc (start 151.13 110.49) (end 153.67 110.49) (angle 90) (layer Edge.Cuts) (width 0.15))
-  (gr_arc (start 151.13 102.87) (end 151.13 100.33) (angle 90) (layer Edge.Cuts) (width 0.15))
+  (gr_line (start 142.24 110.49) (end 142.24 102.87) (angle 90) (layer Edge.Cuts) (width 0.15))
+  (gr_line (start 152.4 102.87) (end 152.4 110.49) (angle 90) (layer Edge.Cuts) (width 0.15))
+  (gr_arc (start 144.78 102.87) (end 142.24 102.87) (angle 90) (layer Edge.Cuts) (width 0.15))
+  (gr_arc (start 144.78 110.49) (end 144.78 113.03) (angle 90) (layer Edge.Cuts) (width 0.15))
+  (gr_arc (start 149.86 110.49) (end 152.4 110.49) (angle 90) (layer Edge.Cuts) (width 0.15))
+  (gr_arc (start 149.86 102.87) (end 149.86 100.33) (angle 90) (layer Edge.Cuts) (width 0.15))
   (segment (start 143.51 105.41) (end 144.78 104.14) (width 0.4064) (layer F.Cu) (net 1))
   (segment (start 144.78 104.14) (end 147.32 104.14) (width 0.4064) (layer F.Cu) (net 1))
