File: projects/Altimeter/KiCad_design_files/project.kicad_pcb (KiCad board)
At the start: 2 copper layers, 18 x 41 mm, 15 parts, among them CON1 AVR-ISP-6, J1 Display, SW1 SW_Reed, SW2 SW_SPDT, U1 ATMEGA328P-AU, U2 MPL3115A

Commit message: Updates
Other:
- board text added: "DESIGN"
- board text added: "Rev 1.0 May 2019"
- board text added: "SIGMA"
- board text added: "Vacuum Sensor"
- board text removed: "Altimeter V0"
Changed lines of the file:
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@@
     (area 128.104999 73.524999 146.255001 114.675001)
     (thickness 1.6)
-    (drawings 23)
+    (drawings 26)
     (tracks 207)
     (zones 0)
@@
   (page A4)
   (layers
-    (0 F.Cu signal)
-    (31 B.Cu signal hide)
+    (0 F.Cu signal hide)
+    (31 B.Cu signal)
     (32 B.Adhes user)
     (33 F.Adhes user)
@@
     (aux_axis_origin -2.54 3.81)
     (grid_origin 170.18 101.6)
-    (visible_elements 7FFF7FFF)
+    (visible_elements 7FFFFFFF)
     (pcbplotparams
-      (layerselection 0x00030_80000001)
-      (usegerberextensions false)
+      (layerselection 0x010f0_80000001)
+      (usegerberextensions true)
       (excludeedgelayer true)
       (linewidth 0.100000)
@@
       (outputformat 1)
       (mirror false)
-      (drillshape 1)
+      (drillshape 0)
       (scaleselection 1)
-      (outputdirectory ""))
+      (outputdirectory gerbers/))
   )
   (net 0 "")
@@
     )
   )
+  (gr_text DESIGN (at 131.318 86.106 90) (layer B.SilkS)
+    (effects (font (size 1.25 1.1) (thickness 0.2)) (justify mirror))
+  )
+  (gr_text "Rev 1.0\nMay 2019" (at 137.922 81.28 90) (layer B.SilkS)
+    (effects (font (size 0.8 0.8) (thickness 0.15)) (justify mirror))
+  )
+  (gr_text SIGMA (at 131.318 80.264 90) (layer B.SilkS)
+    (effects (font (size 1.25 1.25) (thickness 0.3)) (justify mirror))
+  )
   (gr_line (start 137.68 92.1) (end 137.68 91.85) (angle 90) (layer F.SilkS) (width 0.1))
   (gr_line (start 137.68 91.85) (end 137.43 92.1) (angle 90) (layer F.SilkS) (width 0.1))
@@
   (gr_circle (center 137.18 89.1) (end 137.18 88.85) (layer F.SilkS) (width 0.2))
   (gr_text + (at 136.652 84.963) (layer B.SilkS)
-    (effects (font (size 1.5 1.5) (thickness 0.3)) (justify mirror))
-  )
-  (gr_text "Altimeter V0" (at 129.794 83.693 90) (layer B.SilkS)
+    (effects (font (size 1 1) (thickness 0.15)) (justify mirror))
+  )
+  (gr_text "Vacuum Sensor" (at 129.286 83.82 90) (layer B.SilkS)
     (effects (font (size 1.5 1.5) (thickness 0.3) italic) (justify mirror))
   )
@@
   (gr_line (start 146.18 114.6) (end 128.18 114.6) (angle 90) (layer Dwgs.User) (width 0.2))
   (dimension 12 (width 0.3) (layer Dwgs.User)
-    (gr_text "12.000 mm" (at 135.18 70.25) (layer Dwgs.User)
+    (gr_text "12.0 mm" (at 135.18 70.25) (layer Dwgs.User)
       (effects (font (size 1.5 1.5) (thickness 0.3)))
     )
@@
   )
   (dimension 38 (width 0.3) (layer Dwgs.User)
-    (gr_text "38.000 mm" (at 117.83 94.6 90) (layer Dwgs.User)
+    (gr_text "38.0 mm" (at 117.83 94.6 90) (layer Dwgs.User)
       (effects (font (size 1.5 1.5) (thickness 0.3)))
     )
