File: projects/Nerf/Arduino/design_files MOSFET/Arduino.sch (KiCad schematic (older format))
At the start: 42 parts, among them J1 BATT_IN, J10 MTR_2, J11 BATT_OUT, J2 BATT_IN, J3 PUSHER, J4 JAM, J5 I2C, J6 TRIGGER, J7 FTDI, J8 INTERRUPTS, J9 MTR_1, Q1 IRLB8721, SW1 SW_Rotary8, U1 MCP1702, U2 L293D, U3 HALL SENSOR, U4 HALL SENSOR, U5 ATMEGA328P-PU, U6 HALL SENSOR, Y1 16Mhz

Commit message: Updates
Parts:
- removed J6: TRIGGER, Pin_Headers:Pin_Header_Straight_1x04_Pitch2.54mm, symbol Conn_01x04
- removed J8: INTERRUPTS, Pin_Headers:Pin_Header_Straight_1x04_Pitch2.54mm, symbol Conn_01x04
- added J12: CLIP, footprints:Molex_PicoBlade_53048-0210_02x1.25mm_Angled, symbol CONN_01X02
- added J13, J14, J16: NPTH, Wire_Pads:SolderWirePad_single_2-5mmDrill, symbol CONN_01X01
- added J6: TRIGGER, Connectors_Molex:Molex_PicoBlade_53048-0610_06x1.25mm_Angled, symbol Conn_01x06
- added J8: SENSORS, Connectors_Molex:Molex_PicoBlade_53048-0510_05x1.25mm_Angled, symbol Conn_01x05
- added R13: 100K, footprints:R__P7mm, symbol R
- added R14: 10K, footprints:R__P7mm, symbol R
- added R15: 1K, footprints:R__P7mm, symbol R
- added R16: 10K, footprints:R__P5.08mm, symbol R
- C1, C2, C4: footprint Capacitors_THT:C_Disc_D5.0mm_W2.5mm_P2.50mm -> footprints:C_Disc_D5.0mm_W2.5mm_P2.50mm
- C3, C6, C7, C8: footprint Capacitors_THT:C_Disc_D3.4mm_W2.1mm_P2.50mm -> footprints:C_Disc_D3.4mm_W2.1mm_P2.50mm
- C5: footprint footprints:C_Disc_D3.8mm_W2.6mm_P2.50mm -> footprints:C_Disc_D3.4mm_W2.1mm_P2.50mm
- D1: value D -> 1N4001; footprint Diodes_THT:D_DO-15_P12.70mm_Horizontal -> footprints:D_DO-15_P12.70mm_Horizontal
- D2: footprint LEDs:LED_D3.0mm_Horizontal_O1.27mm_Z10.0mm -> footprints:LED_D3.0mm_Horizontal_O1.27mm_Z10.0mm
- J1, J11: footprint Connectors_Phoenix:PhoenixContact_MCV-G_03x3.50mm_Vertical -> footprints:TerminalBlock_Phoenix_PT-1,5-3-3.5-H_1x03_P3.50mm_Horizontal
- J10, J9: footprint Connectors_Phoenix:PhoenixContact_GMSTBVA-G_02x7.50mm_Vertical -> footprints:PhoenixContact_MCV-G_02x3.50mm_Vertical
- J2: footprint Connectors_Phoenix:PhoenixContact_GMSTBVA-G_02x7.50mm_Vertical -> footprints:TerminalBlock_Phoenix_PT-1,5-2-5.0-H_1x02_P5.00mm_Horizontal
- J3, J4: footprint Connectors_Phoenix:PhoenixContact_MCV-G_02x3.50mm_Vertical -> footprints:TerminalBlock_Phoenix_PT-1,5-2-3.5-H_1x02_P3.50mm_Horizontal
- J5: footprint Pin_Headers:Pin_Header_Straight_1x04_Pitch2.54mm -> footprints:Molex_PicoBlade_53048-0410_04x1.25mm_Angled
- J7: footprint Pin_Headers:Pin_Header_Straight_1x06_Pitch2.54mm -> footprints:Pin_Header_Straight_1x06_Pitch2.54mm
- Q1: footprint TO_SOT_Packages_THT:TO-220-3_Horizontal -> footprints:TO-220-3_Horizontal
- R1, R10, R11, R3, R4, R5, R6, R7, R9: footprint footprints:R_Axial_DIN0204_L3.6mm_D1.6mm_P7.62mm_Horizontal -> footprints:R__P5.08mm
- R12: value 4.7K -> 10K
- R8: value 47K -> 100K
- SW1: footprint Pin_Headers:Pin_Header_Straight_1x08_Pitch2.54mm -> footprints:SW_Rotary8
- U1: footprint TO_SOT_Packages_THT:TO-92_Inline_Narrow_Oval -> footprints:TO-92_Inline_Narrow_Oval
- U2: footprint Housings_DIP:DIP-16_W7.62mm -> footprints:DIP-16_W7.62mm
- U3, U4, U6: footprint TO_SOT_Packages_THT:TO-92_Inline_Wide -> footprints:Hall_Sensor
Connections:
- wire segments 155 -> 159
- no-connect marks 3 -> 5
Other:
- note added: "A0 -\nA1 CLIP\nA2 FIRE SEL\nA3 Voltage\n\n"
- note added: "D2 INT pin 1\nD3 INT pin 2\nD4 Pusher SW\nD5 Pusher A\nD6 Pusher B\nD7 Rev SW\nD8 Trig SW\nD9 Flywheel\nD10 Clip U3\nD11 Clip U4\nD12 Clip U6\nD13 LED"
- note removed: "A0 SEL 3\nA1 SEL 2\nA2 SEL 1\nA3 Voltage\n\n"
- note removed: "D2 INT pin 1\nD3 INT pin 2\nD4 Pusher SW\nD5 Pusher A\nD6 Pusher B\nD7 Accel SW\nD8 Trig SW\nD9 Flywheel\nD10 Clip U3\nD11 Clip U4\nD12 Clip U6\nD13 LED"
- moved on the sheet: C5, D2, J5, J7, R12, R2, R8, SW1, U3, U4, U5, U6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
