File: projects/Nerf/Ardu RapidStrike/design_files V02 debounce/Arduino.kicad_pcb (KiCad board)
At the start: 2 copper layers, 80 x 40 mm, 54 parts, among them J1 BATT_IN, J11 BATT_OUT, J12 CLIP, J13 NPTH, J14 NPTH, J16 NPTH, J2 BATT_IN, J3 PUSHER, J4 JAM, J5 I2C, J6 TRIGGER, J7 FTDI, J8 SENSORS, J9 MTR_1, Q1 IRLB8721, SW1 SW_Rotary8, SW2 SW_Push, U1 MCP1702, U2 L293D, U3 HALL SENSOR, U4 HALL SENSOR, U5 ATMEGA328P-PU, U6 HALL SENSOR, Y1 16Mhz

Commit message: Updates
Parts:
- added C9: 0.1uF, footprints:C_Disc_D3.4mm_W2.1mm_P2.50mm, F.Cu at (184.2, 146.7)
- added J10: MTR_2, footprints:PhoenixContact_MCV-G_02x3.50mm_Vertical, F.Cu at (166.6, 148.1)
- added J15: BATT, Connectors_Terminal_Blocks:TerminalBlock_bornier-2_P5.08mm, F.Cu at (265.9, 95.9)
- added J17: PSH_IN, footprints:Molex_PicoBlade_53048-0410_04x1.25mm_Angled, F.Cu at (227.8, 78.1)
- added J18: PSH_OUT, footprints:Molex_PicoBlade_53048-0410_04x1.25mm_Angled, F.Cu at (174.5, 134.0)
- added R17: 10K, footprints:R__P5.08mm, F.Cu at (194.8, 145.2)
- added U7: 74LS14, Housings_DIP:DIP-14_W7.62mm, F.Cu at (237.7, 92.1)
- J3: footprint footprints:TerminalBlock_Phoenix_PT-1,5-2-3.5-H_1x02_P3.50mm_Horizontal -> Connectors_Terminal_Blocks:TerminalBlock_bornier-2_P5.08mm
- moved J3 119.7 mm to (254.5, 95.9)
- moved R3 117.7 mm to (263.4, 60.3)
- moved R1 115.2 mm to (253.2, 60.3)
- moved U2 114.1 mm to (248.2, 75.6)
- moved J16 16.8 mm to (137.7, 90.8)
- moved SW1 16.8 mm to (137.7, 90.8)
Connections:
- C2 pad 1: /BATT -> Net-(C2-Pad1)
- C3 pad 1: VCC -> Net-(C3-Pad1)
- C6 pad 1: /8 -> Net-(C6-Pad1)
- C7 pad 1: /7 -> Net-(C7-Pad1)
- C8 pad 1: /4 -> Net-(C8-Pad1)
- J7 pad 6: Net-(J7-Pad6) -> /#RTS
- R1 pad 2: /6(**) -> Net-(J17-Pad2)
- R10 pad 1: /4 -> Net-(C8-Pad1)
- R11 pad 1: /4 -> /PUSH
- R11 pad 2: /PUSH -> Net-(C8-Pad1)
- R3 pad 2: /5(**) -> Net-(J17-Pad3)
- R4 pad 1: /8 -> Net-(C6-Pad1)
- R5 pad 1: /8 -> /TRIG
- R5 pad 2: /TRIG -> Net-(C6-Pad1)
- R6 pad 1: /7 -> Net-(C7-Pad1)
- R7 pad 1: /7 -> /ACCEL
- R7 pad 2: /ACCEL -> Net-(C7-Pad1)
- U2 pad 1: VCC -> Net-(C3-Pad1)
- U2 pad 10: /5(**) -> Net-(J17-Pad3)
- U2 pad 15: /6(**) -> Net-(J17-Pad2)
- U2 pad 16: VCC -> Net-(C3-Pad1)
- U2 pad 2: /6(**) -> Net-(J17-Pad2)
- U2 pad 7: /5(**) -> Net-(J17-Pad3)
- U2 pad 8: /BATT -> Net-(C2-Pad1)
- U2 pad 9: VCC -> Net-(C3-Pad1)
Routing:
- net GND: track 453.3 -> 0.00 mm
- net VCC: track 197.5 -> 0.00 mm
- net /BATT: track 118.6 -> 0.00 mm
- net /A2: track 107.2 -> 0.00 mm
- net /9(**): track 92.5 -> 0.00 mm
- net /12(MISO): track 66.5 -> 0.00 mm
- net /6(**): track 50.4 -> 0.00 mm
- net /A0: track 41.5 -> 0.00 mm
- net Net-(J10-Pad1): track 34.8 -> 0.00 mm
- net /5(**): track 33.4 -> 0.00 mm
- net Net-(D1-Pad1): track 30.4 -> 0.00 mm
- net /8: track 30.3 -> 0.00 mm
- net /10(SS): track 29.5 -> 0.00 mm
- net /PUSH: track 27.3 -> 0.00 mm
- net /13(SCK): track 26.7 -> 0.00 mm
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Other:
- outline, holes or cut-outs redrawn
- board text removed: "A"
- board text removed: "B"
- board text removed: "C"
- board text removed: "D"
