File: projects/Nerf/Ardu RapidStrike/design_files V03/a_MOSFET.kicad_pcb (KiCad board)
At the start: 2 copper layers, 128 x 78 mm, 81 parts, among them J1 BATT_OUT, J10 PWM_IN, J11 PWM_OUT, J12 CLIP, J13 BUTTON, J14 NPTH, J15 BATT, J16 NPTH, J17 PSH_IN, J18 PSH_OUT, J19 TRIG, J2 BATT_IN, J20 PUSH, J21 BUTTON, J22 TRIG_OUT, J23 TRIG_IN, J24 TO_IR, J25 PHOTO, J26 IR_LED, J27 BUTTON, J3 PUSHER, J4 JAM, J5 I2C, J6 REV, J7 FTDI, J8 PHOTO, J9 FLYWHEELS, Q1 IRLB8721, Q2 Photo_NPN, SW1 SW_Rotary8, SW2 SW_Push, U1 MCP1702, U2 L293D, U3 HALL SENSOR, U4 HALL SENSOR, U5 ATMEGA328P-PU, U6 HALL SENSOR, U7 74LS14, Y1 16Mhz

Commit message: Updates
Parts:
- added F1: Polyfuse, Fuse_Holders_and_Fuses:Fuse_Littelfuse-LVR125, F.Cu at (149.5, 66.9)
- J1: footprint Connectors_Terminal_Blocks:TerminalBlock_bornier-2_P5.08mm -> footprints:TerminalBlock_Phoenix_PT-1,5-2-3.5-H_1x02_P3.50mm_Horizontal
- J2: footprint footprints:XT30PW_M -> footprints:TerminalBlock_Phoenix_PT-1,5-2-3.5-H_1x02_P3.50mm_Horizontal
- J9: footprint footprints:XT30PW_F -> footprints:TerminalBlock_Phoenix_PT-1,5-2-3.5-H_1x02_P3.50mm_Horizontal
- R13: value 100K -> 30K
- R15: value 1K -> 3K3
- moved J2 29.3 mm to (133.5, 73.4), turned to 0 degrees
- moved J9 9.86 mm to (152.0, 73.4), turned to 0 degrees
- moved J1 8.84 mm to (143.0, 73.4)
- moved Q1 6.82 mm to (138.0, 52.4)
- moved G*** 5.47 mm to (149.5, 58.9)
- moved R9 5.28 mm to (132.2, 53.9), turned to 270 degrees
- moved J10 4.12 mm to (132.5, 66.9)
- moved J14 3.72 mm to (144.5, 62.9)
- moved D1 2.19 mm to (135.0, 51.4)
Connections:
- J1 pad 1: GND -> /BATT
- J1 pad 2: Net-(J1-Pad2) -> GND
- J2 pad 1: Net-(J1-Pad2) -> /BATT
- J9 pad 1: Net-(J1-Pad2) -> Net-(F1-Pad2)
Routing:
- net Net-(J1-Pad2): track 39.3 -> 0.00 mm
- net /BATT: track 0.00 -> 23.1 mm
- net Net-(D1-Pad1): track 24.4 -> 36.6 mm
- net /9(**): track 45.0 -> 38.1 mm
- net Net-(F1-Pad2): track 0.00 -> 6.67 mm
- net GND: track 345.6 -> 340.9 mm
Other:
- outline, holes or cut-outs redrawn
- board text added: "MOSFET BOARD"
- board text added: "MOSFET Board"
- board text added: "Rev 0.3 Jun 2019"
- board text removed: "FLYWHEELS BOARD"
- board text removed: "Flywheel Board"
