File: projects/Nerf/Ardu RapidStrike/design_files V06 SMD/project.sch (KiCad schematic (older format))
At the start: 67 parts, among them CON1 ISP, J1 BATT_OUT, J10 PWM, J11 A2, J12 CLIP, J14 NPTH, J15 BATT, J17 PSH_IN, J18 PSH_OUT, J19 TRIG, J2 BATT_IN, J20 PUSH, J21 BUTTON, J24 TO_IR, J25 PHOTO, J26 IR_LED, J27 BUTTON, J3 PUSHER, J4 JAM, J5 I2C, J6 REV, J7 FTDI, J8 FRONT, J9 MTRS, Q1 IRLB8721, Q2 Photo_NPN, SW2 SW_Push, U1 MCP1702, U2 L293D, U3 HALL SENSOR, U4 HALL SENSOR, U5 ATMEGA328P-AU, U6 HALL SENSOR, Y1 16Mhz

Commit message: Updates
Parts:
- removed D2: D13, footprints:LED_D3.0mm_Horizontal_O1.27mm_Z10.0mm, symbol LED
- removed J1: BATT_OUT, footprints:TerminalBlock_bornier-2_P5.08mm, symbol Conn_01x02
- removed J10: PWM, footprints:Pin_Header_Straight_1x01_Pitch2.00mm, symbol CONN_01X01
- removed J12: CLIP, Connectors_Molex:Molex_PicoBlade_53261-0271_02x1.25mm_Angled, symbol CONN_01X02
- removed J19: TRIG, footprints:Pin_Header_Straight_2x01_Pitch2.00mm, symbol Conn_01x02
- removed J20: PUSH, Connectors_Molex:Molex_PicoBlade_53261-0271_02x1.25mm_Angled, symbol Conn_01x02
- removed J21: BUTTON, Connectors_Molex:Molex_PicoBlade_53261-0271_02x1.25mm_Angled, symbol Conn_01x02
- removed J6: REV, footprints:Pin_Header_Straight_2x01_Pitch2.00mm, symbol Conn_01x02
- removed J8: FRONT, Connectors_Molex:Molex_PicoBlade_53261-0471_04x1.25mm_Angled, symbol Conn_01x04
- removed U2: L293D, footprints:DIP-16_W7.62mm, symbol L293D
- added J13: LED, footprints:Pin_Header_Straight_2x01_Pitch2.00mm, symbol Conn_01x02
- added J6: INPUTS, Connectors_Molex:Molex_PicoBlade_53261-1071_10x1.25mm_Angled, symbol CONN_01X10
- added J8: PHOTO, Connectors_Molex:Molex_PicoBlade_53261-0371_03x1.25mm_Angled, symbol Conn_01x03
- added U2: TC78H611FNG, Housings_SSOP:TSSOP-16-1EP_4.4x5mm_Pitch0.65mm, symbol TC78H611FNG
- C2: value 1uF -> 10uF
- J4: footprint footprints:TerminalBlock_Phoenix_PT-1,5-2-3.5-H_1x02_P3.50mm_Horizontal -> Connectors_Molex:Molex_PicoBlade_53261-0271_02x1.25mm_Angled
- J7: footprint footprints:Pin_Header_Angled_1x06_Pitch2.54mm -> Pin_Headers:Pin_Header_Straight_1x06_Pitch2.54mm_SMD_Pin1Right
- LS1: footprint footprints:SPEAKER -> footprints:PS1240_piezo
Connections:
- wire segments 199 -> 212
Other:
- note added: "BUTTON"
- note added: "CLIP"
- note added: "PUSHER SW"
- note added: "REV"
- note added: "TRIG"
- note removed: "TRIGGER BOARD"
- moved on the sheet: C10, C6, C7, C8, D1, F1, R10, R11, R18, R19, R4, R5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

Commit message: Updates
Parts:
- removed J13: LED, footprints:Pin_Header_Straight_2x01_Pitch2.00mm, symbol Conn_01x02
- removed J15: BATT, footprints:TerminalBlock_bornier-2_P5.08mm, symbol Conn_01x02
- removed J17: PSH_IN, footprints:Molex_PicoBlade_53047-0510_05x1.25mm_Straight, symbol Conn_01x05
- removed J18: PSH_OUT, Connectors_Molex:Molex_PicoBlade_53261-0571_05x1.25mm_Angled, symbol Conn_01x05
- added D13: LED, footprints:LED_D3.0mm_Horizontal_O1.27mm_Z10.0mm, symbol LED
- added J1: TEST, Pin_Headers:Pin_Header_Straight_1x03_Pitch2.00mm, symbol CONN_01X03
- added JP1: 2S, footprints:JMPR, symbol Jumper_NO_Small
- added JP2: NiMH, footprints:JMPR, symbol Jumper_NO_Small
- F1: footprint Fuse_Holders_and_Fuses:Fuse_SMD2920 -> Resistors_SMD:R_1812_HandSoldering
- F2: footprint footprints:Fuse_Littelfuse-LVR125 -> Fuse_Holders_and_Fuses:Fuse_SMD1206_HandSoldering
- U5: value ATMEGA328P-AU -> ATMEGA328P
Connections:
- wire segments 212 -> 205
Other:
- note added: "A0 SPKR\nA1 DART IR\nA2 \nA3 Voltage\nD2 Pusher SW\nD3 Rev SW\nD4 BUTTON\nD5 Pusher A\nD6 Pusher B\nD7 Trig SW\nD8 CLIP\nD9 Flywheel\nD10 Clip U3\nD11 Clip U4\nD12 Clip U6\nD13 LED"
- note added: "TEST\nPOINTS"
- note removed: "A0 BUTTON\nA1 DART IR\nA2 \nA3 Voltage\nD2 Pusher SW\nD3 Rev SW\nD4 SPKR\nD5 Pusher A\nD6 Pusher B\nD7 CLIP\nD8 Trig SW\nD9 Flywheel\nD10 Clip U3\nD11 Clip U4\nD12 Clip U6\nD13 LED"
- moved on the sheet: C2, C3, J3, J4, R1, R3, U2
