File: projects/Nerf/Ardu RapidStrike/design_files Stryfe V04/project.sch (KiCad schematic (older format))
At the start: 42 parts, among them CON1 ISP, J1 JAM, J12 CLIP, J14 NPTH, J2 BATT_IN, J21 DEBUG, J3 LED, J5 I2C, J6 REV, J7 FTDI, J8 PHOTO, J9 FW_MTRS, Q1 IRLR8729, U1 MCP1702, U3 HALL SENSOR, U4 HALL SENSOR, U5 ATMEGA328P-PU, U6 HALL SENSOR, Y1 16Mhz

Commit message: Updates
Parts:
- R12: value 4K9K 1% -> 4K99 1%
Changed lines of the file:
@@
 P 3700 5650
 F 0 "R12" V 3700 5650 50  0000 C CNN
-F 1 "4K9K 1%" H 3950 5650 50  0000 C CNN
+F 1 "4K99 1%" H 3950 5650 50  0000 C CNN
 F 2 "footprints:R_7.5mm" V 3630 5650 50  0001 C CNN
 F 3 "" H 3700 5650 50  0001 C CNN
