File: projects/OSTR/design_files_MicroBit V9/base.kicad_pcb (KiCad board)
At the start: 2 copper layers, 38.1 x 58.4 mm, 29 parts, among them J1 microbit_edge_connector, J2 BATT1, J3 BATT2, J4 LEFT_STEPPER, J5 RIGHT_STEPPER, J6 SERVO, J7 TEST, J8 Sensors, J9 Sensors, P9 CONN_01X01, Q3 PNP, Q4 NPN, SW1 PWR, U1 ULN2803, U2 MCP1702

Commit message: Updates
Parts:
- removed D1: D, Diodes_THT:D_A-405_P7.62mm_Horizontal
- removed Q3: PNP, TO_SOT_Packages_THT:TO-126_Vertical
- J4: value LEFT_STEPPER -> RIGHT_STEPPER
- J5: value RIGHT_STEPPER -> LEFT_STEPPER; footprint JST_B5B-XH-A -> library:JST_B5B-XH-A
- R3: value 1K -> 10K
- SW1: footprint SW_Micro_SPST -> library:SW_Micro_SPST
- U1: value ULN2803 -> TLC59213; footprint Housings_DIP:DIP-18_W7.62mm_Socket_LongPads -> Housings_DIP:DIP-20_W7.62mm_LongPads
- moved R2 31.0 mm to (132.7, 76.8)
- moved R3 17.8 mm to (135.9, 76.8)
- moved R1 0.90 mm to (139.1, 76.8), turned to 90 degrees
Connections:
- C1 pad 1: Net-(C1-Pad1) -> /BAT
- C2 pad 1: Net-(C1-Pad1) -> /BAT
- J4 pad 5: Net-(C1-Pad1) -> /BAT
- J5 pad 5: Net-(C1-Pad1) -> /BAT
- J6 pad 2: Net-(C1-Pad1) -> /BAT
- R1 pad 1: Net-(Q3-Pad3) -> Net-(R1-Pad1)
- R1 pad 2: +3V3 -> /BAT
- R2 pad 2: /P14 -> /P15
- R3 pad 1: Net-(Q3-Pad3) -> GND
- R3 pad 2: /P15 -> /P14
- U1 pad 1: /P0 -> Net-(R1-Pad1)
- U1 pad 10: Net-(C1-Pad1) -> /P14
- U1 pad 11: Net-(J5-Pad4) -> GND
- U1 pad 12: Net-(J5-Pad3) -> Net-(J5-Pad4)
- U1 pad 13: Net-(J5-Pad2) -> Net-(J5-Pad3)
- U1 pad 14: Net-(J5-Pad1) -> Net-(J5-Pad2)
- U1 pad 15: Net-(J4-Pad4) -> Net-(J5-Pad1)
- U1 pad 16: Net-(J4-Pad3) -> Net-(J4-Pad4)
- U1 pad 17: Net-(J4-Pad2) -> Net-(J4-Pad3)
- U1 pad 18: Net-(J4-Pad1) -> Net-(J4-Pad2)
- U1 pad 2: /P6 -> /P0
- U1 pad 3: /P7 -> /P6
- U1 pad 4: /P1 -> /P7
- U1 pad 5: /P8 -> /P1
- U1 pad 6: /P9 -> /P8
- U1 pad 7: /P10 -> /P9
- U1 pad 8: /P13 -> /P10
- U1 pad 9: GND -> /P13
Routing:
- net Net-(C1-Pad1): track 79.0 -> 0.00 mm
- net /BAT: track 52.7 -> 114.2 mm
- net Net-(Q4-Pad2): track 5.87 -> 38.0 mm
- net Net-(R1-Pad1): track 0.00 -> 30.6 mm
- net Net-(Q3-Pad3): track 21.0 -> 0.00 mm
- net +3V3: track 82.9 -> 68.4 mm
- net /P15: track 7.99 -> 20.2 mm
- net /P16: track 29.5 -> 23.3 mm
- net /P14: track 19.2 -> 13.5 mm
- net /P0: track 27.4 -> 24.5 mm
- net /P3: track 45.9 -> 43.3 mm
- net Net-(J8-Pad4): track 20.7 -> 23.3 mm
- net Net-(J5-Pad1): track 9.42 -> 6.88 mm
- net Net-(J3-Pad2): track 42.4 -> 44.5 mm
- net /P1: track 20.5 -> 22.4 mm
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- added copper zone on F.Cu, net GND
Other:
- board text added: "Ver 0.9 Oct 2019"
- board text removed: "Ver 0.8 Sep 2019"
