File: projects/Attiny/Attin85_HBridge R2/design_files/project.sch (KiCad schematic (older format))
At the start: 23 parts, among them CON1 AVR-ISP-6, J1 BATT_IN, J2 SIG1_IN, J3 MTR_1_OUT, J4 VCC, J5 MTR_2_OUT, J6 SIG2_IN, U1 TC78H651FNG, U2 ATTINY84-20SSU

Commit message: Updates
Parts:
- removed J6: SIG2_IN, footprints:Pin_Header_Straight_1x02_Pitch2.54mm, symbol Conn_01x02
- removed R1: JMP, footprints:Jumper, symbol R
- removed R11, R9: 10K, Resistors_SMD:R_0603_HandSoldering, symbol R
- added D1: Diode, footprints:D_SOD-323_HandSoldering, symbol D_ALT
- added J6: SR04, footprints:Pin_Header_Straight_1x04_Pitch2.54mm, symbol CONN_01X04
- added JP1: JMP, footprints:Jumper, symbol Jumper_NO_Small
- C1, C3: footprint Capacitors_SMD:C_0603_HandSoldering -> footprints:C_0603_HandSoldering
- C2: value 10uF -> 47uF; footprint footprints:CP_Elec_5x5.3 -> footprints:CP_Elec_6.3x5.3
- J1: value BATT_IN -> BATT
- J2: value SIG1_IN -> SIG_1
- J3: value MTR_1_OUT -> MTR_1
- J5: value MTR_2_OUT -> MTR_2
- R10, R3, R4, R5, R6, R8: footprint Resistors_SMD:R_0603_HandSoldering -> footprints:R_0603_HandSoldering
- U1: footprint Housings_SSOP:TSSOP-16_4.4x5mm_Pitch0.65mm -> footprints:TSSOP-16_4.4x5mm_Pitch0.65mm
- U2: value ATTINY84-20SSU -> ATTINY84; footprint Housings_SOIC:SOIC-14_3.9x8.7mm_Pitch1.27mm -> footprints:SOIC-14_3.9x8.7mm_Pitch1.27mm
Connections:
- net labels added: ECHO, TRIG
- wire segments 78 -> 86
Changed lines of the file:
@@
 EESchema Schematic File Version 2
 LIBS:project
+LIBS:TC78H651FNG
 LIBS:power
 LIBS:device
@@
 LIBS:contrib
 LIBS:valves
-LIBS:TC78H651FNG
 LIBS:project-cache
 EELAYER 25 0
@@
 P 5550 3000
 F 0 "J3" H 5700 2950 50  0000 C CNN
-F 1 "MTR_1_OUT" H 5550 3150 50  0000 C CNN
+F 1 "MTR_1" H 5550 3150 50  0000 C CNN
 F 2 "footprints:Pin_Header_Straight_1x02_Pitch2.54mm" H 5550 3000 50  0001 C CNN
 F 3 "" H 5550 3000 50  0001 C CNN
@@
 P 2500 2400
 F 0 "J1" H 2500 2500 50  0000 C CNN
-F 1 "BATT_IN" H 2500 2200 50  0000 C CNN
+F 1 "BATT" H 2500 2200 50  0000 C CNN
 F 2 "footprints:Pin_Header_Straight_1x02_Pitch2.54mm" H 2500 2400 50  0001 C CNN
 F 3 "" H 2500 2400 50  0001 C CNN
@@
 F 0 "C1" H 3325 5150 50  0000 L CNN
 F 1 "0.1uF" H 3325 4950 50  0000 L CNN
-F 2 "Capacitors_SMD:C_0603_HandSoldering" H 3338 4900 50  0001 C CNN
+F 2 "footprints:C_0603_HandSoldering" H 3338 4900 50  0001 C CNN
 F 3 "" H 3300 5050 50  0001 C CNN
 	1    3300 5050
@@
 P 3250 2800
 F 0 "C2" H 3275 2900 50  0000 L CNN
-F 1 "10uF" H 3275 2700 50  0000 L CNN
-F 2 "footprints:CP_Elec_5x5.3" H 3250 2800 50  0001 C CNN
+F 1 "47uF" H 3275 2700 50  0000 L CNN
+F 2 "footprints:CP_Elec_6.3x5.3" H 3250 2800 50  0001 C CNN
 F 3 "" H 3250 2800 50  0001 C CNN
 	1    3250 2800
@@
 P 6750 4550
 F 0 "J2" H 6750 4650 50  0000 C CNN
-F 1 "SIG1_IN" H 6750 4350 50  0000 C CNN
+F 1 "SIG_1" H 6750 4350 50  0000 C CNN
 F 2 "footprints:Pin_Header_Straight_1x02_Pitch2.54mm" H 6750 4550 50  0001 C CNN
 F 3 "" H 6750 4550 50  0001 C CNN
@@
 VM
 $Comp
-L R R1
-U 1 1 5E56B20C
-P 3500 1700
-F 0 "R1" V 3580 1700 50  0000 C CNN
-F 1 "JMP" V 3500 1700 50  0000 C CNN
-F 2 "footprints:Jumper" V 3430 1700 50  0001 C CNN
-F 3 "" H 3500 1700 50  0001 C CNN
-	1    3500 1700
-	0    1    1    0
-$EndComp
-$Comp
 L TC78H651FNG U1
 U 1 1 5E6AB4B9
@@
 F 0 "U1" H 4450 3600 60  0000 C CNN
 F 1 "TC78H651FNG" H 4800 2700 60  0000 L CNN
-F 2 "Housings_SSOP:TSSOP-16_4.4x5mm_Pitch0.65mm" H 5000 2450 60  0001 L CNN
+F 2 "footprints:TSSOP-16_4.4x5mm_Pitch0.65mm" H 5000 2450 60  0001 L CNN
 F 3 "https://toshiba.semicon-storage.com/info/docget.jsp?did=61125&prodName=TC78H651FNG" H 5000 2350 60  0001 L CNN
 	1    4700 3150
@@
 P 5550 3200
 F 0 "J5" H 5700 3150 50  0000 C CNN
-F 1 "MTR_2_OUT" H 5550 3000 50  0000 C CNN
+F 1 "MTR_2" H 5550 3000 50  0000 C CNN
 F 2 "footprints:Pin_Header_Straight_1x02_Pitch2.54mm" H 5550 3200 50  0001 C CNN
 F 3 "" H 5550 3200 50  0001 C CNN
@@
 P 4700 5050
 F 0 "U2" H 3850 5800 50  0000 C CNN
-F 1 "ATTINY84-20SSU" H 5400 4300 50  0000 C CNN
-F 2 "Housings_SOIC:SOIC-14_3.9x8.7mm_Pitch1.27mm" H 4700 4850 50  0001 C CIN
+F 1 "ATTINY84" H 5400 4300 50  0000 C CNN
+F 2 "footprints:SOIC-14_3.9x8.7mm_Pitch1.27mm" H 4700 4850 50  0001 C CIN
 F 3 "" H 4700 5050 50  0001 C CNN
 	1    4700 5050
@@
 F 0 "C3" H 2975 2900 50  0000 L CNN
 F 1 "1uF" H 2975 2700 50  0000 L CNN
-F 2 "Capacitors_SMD:C_0603_HandSoldering" H 2988 2650 50  0001 C CNN
+F 2 "footprints:C_0603_HandSoldering" H 2988 2650 50  0001 C CNN
 F 3 "" H 2950 2800 50  0001 C CNN
 	1    2950 2800
@@
 	8850 3950 8550 3950
 Wire Wire Line
-	3100 1700 3350 1700
+	3100 1700 3600 1700
 Wire Wire Line
 	3200 1700 3200 1650
@@
 	3200 1800 3200 1850
 Wire Wire Line
-	3650 1700 4700 1700
+	3900 1700 4700 1700
 Connection ~ 3200 1700
 Wire Wire Line
@@
 	5750 5350 6150 5350
 Wire Wire Line
-	5750 5450 6550 5450
-Wire Wire Line
-	5750 5550 6550 5550
+	5750 5450 7500 5450
+Wire Wire Line
+	5750 5550 6900 5550
 Wire Wire Line
 	5750 5650 6150 5650
@@
 F 0 "R4" V 4150 3500 50  0000 C CNN
 F 1 "10K" V 4100 3650 50  0000 C CNN
-F 2 "Resistors_SMD:R_0603_HandSoldering" V 4030 3650 50  0001 C CNN
+F 2 "footprints:R_0603_HandSoldering" V 4030 3650 50  0001 C CNN
 F 3 "" H 4100 3650 50  0001 C CNN
 	1    4100 3650
@@
 F 0 "R5" V 4250 3500 50  0000 C CNN
 F 1 "10K" V 4200 3650 50  0000 C CNN
-F 2 "Resistors_SMD:R_0603_HandSoldering" V 4130 3650 50  0001 C CNN
+F 2 "footprints:R_0603_HandSoldering" V 4130 3650 50  0001 C CNN
 F 3 "" H 4200 3650 50  0001 C CNN
 	1    4200 3650
@@
 F 0 "R6" V 4350 3500 50  0000 C CNN
 F 1 "10K" V 4300 3650 50  0000 C CNN
-F 2 "Resistors_SMD:R_0603_HandSoldering" V 4230 3650 50  0001 C CNN
+F 2 "footprints:R_0603_HandSoldering" V 4230 3650 50  0001 C CNN
 F 3 "" H 4300 3650 50  0001 C CNN
 	1    4300 3650
@@
 F 0 "R3" V 4050 3500 50  0000 C CNN
 F 1 "10K" V 4000 3650 50  0000 C CNN
-F 2 "Resistors_SMD:R_0603_HandSoldering" V 3930 3650 50  0001 C CNN
+F 2 "footprints:R_0603_HandSoldering" V 3930 3650 50  0001 C CNN
 F 3 "" H 4000 3650 50  0001 C CNN
 	1    4000 3650
@@
 MISO
 $Comp
-L Conn_01x02 J6
-U 1 1 5E6B180B
-P 6750 5550
-F 0 "J6" H 6750 5650 50  0000 C CNN
-F 1 "SIG2_IN" H 6750 5350 50  0000 C CNN
-F 2 "footprints:Pin_Header_Straight_1x02_Pitch2.54mm" H 6750 5550 50  0001 C CNN
-F 3 "" H 6750 5550 50  0001 C CNN
-	1    6750 5550
-	1    0    0    1
-$EndComp
-$Comp
-L R R9
-U 1 1 5E6B2747
-P 6350 5950
-F 0 "R9" V 6400 5800 50  0000 C CNN
-F 1 "10K" V 6350 5950 50  0000 C CNN
-F 2 "Resistors_SMD:R_0603_HandSoldering" V 6280 5950 50  0001 C CNN
-F 3 "" H 6350 5950 50  0001 C CNN
-	1    6350 5950
-	1    0    0    -1
-$EndComp
-$Comp
-L R R11
-U 1 1 5E6B289B
-P 6500 5950
-F 0 "R11" V 6550 5800 50  0000 C CNN
-F 1 "10K" V 6500 5950 50  0000 C CNN
-F 2 "Resistors_SMD:R_0603_HandSoldering" V 6430 5950 50  0001 C CNN
-F 3 "" H 6500 5950 50  0001 C CNN
-	1    6500 5950
-	1    0    0    -1
-$EndComp
-$Comp
-L GND #PWR017
-U 1 1 5E6B2993
-P 6500 6250
-F 0 "#PWR017" H 6500 6000 50  0001 C CNN
-F 1 "GND" H 6650 6200 50  0000 C CNN
-F 2 "" H 6500 6250 50  0001 C CNN
-F 3 "" H 6500 6250 50  0001 C CNN
-	1    6500 6250
-	1    0    0    -1
-$EndComp
-Wire Wire Line
-	6500 5550 6500 5800
-Wire Wire Line
-	6350 5800 6350 5450
-Connection ~ 6350 5450
-Wire Wire Line
-	6350 6100 6350 6200
-Wire Wire Line
-	6350 6200 6500 6200
-Wire Wire Line
-	6500 6100 6500 6250
-Connection ~ 6500 6200
-Connection ~ 6500 5550
-$Comp
 L R R8
 U 1 1 5E6B31E5
@@
 F 0 "R8" V 6400 4650 50  0000 C CNN
 F 1 "10K" V 6350 4800 50  0000 C CNN
-F 2 "Resistors_SMD:R_0603_HandSoldering" V 6280 4800 50  0001 C CNN
+F 2 "footprints:R_0603_HandSoldering" V 6280 4800 50  0001 C CNN
 F 3 "" H 6350 4800 50  0001 C CNN
 	1    6350 4800
@@
 F 0 "R10" V 6550 4650 50  0000 C CNN
 F 1 "10K" V 6500 4800 50  0000 C CNN
-F 2 "Resistors_SMD:R_0603_HandSoldering" V 6430 4800 50  0001 C CNN
+F 2 "footprints:R_0603_HandSoldering" V 6430 4800 50  0001 C CNN
 F 3 "" H 6500 4800 50  0001 C CNN
 	1    6500 4800
@@
 	6500 4950 6500 5100
 $Comp
-L GND #PWR018
+L GND #PWR017
 U 1 1 5E6B3491
 P 6500 5100
-F 0 "#PWR018" H 6500 4850 50  0001 C CNN
+F 0 "#PWR017" H 6500 4850 50  0001 C CNN
 F 1 "GND" H 6650 5050 50  0000 C CNN
 F 2 "" H 6500 5100 50  0001 C CNN
@@
 Wire Wire Line
 	4200 3800 4200 3900
+$Comp
+L D_ALT D1
+U 1 1 5E6FD3A8
+P 3750 1700
+F 0 "D1" H 3750 1800 50  0000 C CNN
+F 1 "Diode" H 3750 1600 50  0000 C CNN
+F 2 "footprints:D_SOD-323_HandSoldering" H 3750 1700 50  0001 C CNN
+F 3 "" H 3750 1700 50  0001 C CNN
+	1    3750 1700
+	1    0    0    -1
+$EndComp
+$Comp
+L Jumper_NO_Small JP1
+U 1 1 5E6FDF07
+P 3750 2000
+F 0 "JP1" H 3750 2080 50  0000 C CNN
+F 1 "JMP" H 3760 1940 50  0000 C CNN
+F 2 "footprints:Jumper" H 3750 2000 50  0001 C CNN
+F 3 "" H 3750 2000 50  0001 C CNN
+	1    3750 2000
+	1    0    0    -1
+$EndComp
+Wire Wire Line
+	4050 1700 4050 2000
+Wire Wire Line
+	4050 2000 3850 2000
+Connection ~ 4050 1700
+Wire Wire Line
+	3650 2000 3500 2000
+Wire Wire Line
+	3500 2000 3500 1700
+Connection ~ 3500 1700
+$Comp
+L CONN_01X04 J6
+U 1 1 5E6FF7BD
+P 7550 5850
+F 0 "J6" H 7550 6100 50  0000 C CNN
+F 1 "SR04" V 7650 5850 50  0000 C CNN
+F 2 "footprints:Pin_Header_Straight_1x04_Pitch2.54mm" H 7550 5850 50  0001 C CNN
+F 3 "" H 7550 5850 50  0001 C CNN
+	1    7550 5850
+	0    1    1    0
+$EndComp
+$Comp
+L GND #PWR018
+U 1 1 5E6FF8FB
+P 7950 5800
+F 0 "#PWR018" H 7950 5550 50  0001 C CNN
+F 1 "GND" H 8100 5750 50  0000 C CNN
+F 2 "" H 7950 5800 50  0001 C CNN
+F 3 "" H 7950 5800 50  0001 C CNN
+	1    7950 5800
+	1    0    0    -1
+$EndComp
+$Comp
+L VCC #PWR019
+U 1 1 5E6FFB2C
+P 7250 5550
+F 0 "#PWR019" H 7250 5400 50  0001 C CNN
+F 1 "VCC" H 7250 5700 50  0000 C CNN
+F 2 "" H 7250 5550 50  0001 C CNN
+F 3 "" H 7250 5550 50  0001 C CNN
+	1    7250 5550
+	0    -1   -1   0
+$EndComp
+Wire Wire Line
+	7700 5650 7700 5550
+Wire Wire Line
+	7700 5550 7950 5550
+Wire Wire Line
+	7950 5550 7950 5800
+Wire Wire Line
+	7400 5650 7400 5550
+Wire Wire Line
+	7400 5550 7250 5550
+Wire Wire Line
+	7500 5450 7500 5650
+Wire Wire Line
+	7600 5300 7600 5650
+Wire Wire Line
+	6900 5300 7600 5300
+Text Label 7100 5300 0    60   ~ 0
+ECHO
+Text Label 7100 5450 0    60   ~ 0
+TRIG
+Wire Wire Line
+	6900 5550 6900 5300
 $EndSCHEMATC
