File: projects/Beetje/design_files_PCF8532_RTC/project.sch (KiCad schematic (older format))
At the start: 12 parts, among them J2 Conn_01x06, J4 Conn_01x08, U1 PCF8523, Y1 32.768Hz, Y2 Alternate

Commit message: Updates
Parts:
- removed Y1: 32.768Hz, footprints:Crystal_SMD_SeikoEpson_MC306-4pin_8.0x3.2mm, symbol Crystal_GND23
- C1, C2: footprint footprints:C_0603 -> footprints:C_0805_HandSoldering
- J2: value Conn_01x06 -> Beetje_Bottom; footprint footprints:Pin_Header_Straight_1x06_Pitch2.54mm -> footprints:Beetje_Bottom
- J4: value Conn_01x08 -> Beetje_Top; footprint footprints:Pin_Header_Straight_1x08_Pitch2.54mm -> footprints:Beetje_Top
- R1, R2, R3: footprint footprints:R_0603 -> footprints:R_0805_HandSoldering
- Y1: renamed from Y2; value Alternate -> 32.768Hz
Connections:
- net labels added: D6
- net labels removed: A1
- wire segments 44 -> 35
- no-connect marks 2 -> 8
Other:
- note added: "Beetje Footprint"
- note removed: "D2\nD3\nD15\nD14\nD16"
- moved on the sheet: J2, J4
Changed lines of the file:
@@
 encoding utf-8
 Sheet 1 1
-Title "Beetje Blok PCF8532 RTC"
-Date "2018-08-17"
-Rev "0.0"
+Title "Beetje Blok RTC"
+Date "2018-09-28"
+Rev "0.1"
 Comp "www.MakersBox.us"
 Comment1 "648.ken@gmail.com"
@@
 $EndComp
 Wire Wire Line
-	4350 4650 4150 4650
-Wire Wire Line
-	4150 4750 4350 4750
-Wire Wire Line
-	4350 4850 4150 4850
-Wire Wire Line
-	4350 4950 4150 4950
-Wire Wire Line
-	4350 5050 4150 5050
-Wire Wire Line
-	4350 5150 4150 5150
-Wire Wire Line
-	4350 5250 4150 5250
-Wire Wire Line
-	4350 5350 4150 5350
+	4350 4900 4150 4900
+Wire Wire Line
+	4150 5000 4350 5000
+Wire Wire Line
+	4350 5100 4150 5100
+Wire Wire Line
+	4350 5200 4150 5200
+Wire Wire Line
+	4350 5300 4150 5300
+Wire Wire Line
+	4350 5400 4150 5400
+Wire Wire Line
+	4350 5500 4300 5500
+Wire Wire Line
+	4350 5600 4250 5600
 $Comp
 L +BATT #PWR06
 U 1 1 5B402C38
-P 4150 5050
-F 0 "#PWR06" H 4150 4900 50  0001 C CNN
-F 1 "+BATT" V 4150 5300 50  0000 C CNN
-F 2 "" H 4150 5050 50  0001 C CNN
-F 3 "" H 4150 5050 50  0001 C CNN
-	1    4150 5050
+P 4300 5500
+F 0 "#PWR06" H 4300 5350 50  0001 C CNN
+F 1 "+BATT" V 4300 5750 50  0000 C CNN
+F 2 "" H 4300 5500 50  0001 C CNN
+F 3 "" H 4300 5500 50  0001 C CNN
+	1    4300 5500
 	0    -1   -1   0
 $EndComp
@@
 L VBUS #PWR07
 U 1 1 5B402FA5
-P 4150 5350
-F 0 "#PWR07" H 4150 5200 50  0001 C CNN
-F 1 "VBUS" V 4150 5550 50  0000 C CNN
-F 2 "" H 4150 5350 50  0001 C CNN
-F 3 "" H 4150 5350 50  0001 C CNN
-	1    4150 5350
+P 4250 5600
+F 0 "#PWR07" H 4250 5450 50  0001 C CNN
+F 1 "VBUS" V 4250 5800 50  0000 C CNN
+F 2 "" H 4250 5600 50  0001 C CNN
+F 3 "" H 4250 5600 50  0001 C CNN
+	1    4250 5600
 	0    -1   -1   0
 $EndComp
-Text Label 4150 4750 0    60   ~ 0
+Text Label 4150 5100 0    60   ~ 0
 D10
-Text Label 5600 4650 0    60   ~ 0
+Text Label 4150 5000 0    60   ~ 0
 D9
-Text Label 5550 4850 0    60   ~ 0
+Text Label 5550 5200 0    60   ~ 0
 SCL
-Text Label 5550 4750 0    60   ~ 0
+Text Label 5550 5100 0    60   ~ 0
 SDA
-Text Label 4150 4650 0    60   ~ 0
+Text Label 4150 4900 0    60   ~ 0
 ~RESET
-Text Label 4150 4850 0    60   ~ 0
+Text Label 5600 4900 0    60   ~ 0
 A0
-Text Label 4150 4950 0    60   ~ 0
-A1
-Text Label 5550 5150 0    60   ~ 0
+Text Label 4150 5400 0    60   ~ 0
 SCK
-Text Label 5500 5050 0    60   ~ 0
+Text Label 4150 5300 0    60   ~ 0
 MOSI
-Text Label 5500 4950 0    60   ~ 0
+Text Label 4150 5200 0    60   ~ 0
 MISO
 $Comp
 L GND #PWR08
 U 1 1 5B41D2F5
-P 4150 5250
-F 0 "#PWR08" H 4150 5000 50  0001 C CNN
-F 1 "GND" V 4150 5050 50  0000 C CNN
-F 2 "" H 4150 5250 50  0001 C CNN
-F 3 "" H 4150 5250 50  0001 C CNN
-	1    4150 5250
-	0    1    1    0
+P 5450 5400
+F 0 "#PWR08" H 5450 5150 50  0001 C CNN
+F 1 "GND" V 5450 5200 50  0000 C CNN
+F 2 "" H 5450 5400 50  0001 C CNN
+F 3 "" H 5450 5400 50  0001 C CNN
+	1    5450 5400
+	0    -1   -1   0
 $EndComp
 $Comp
 L Conn_01x08 J4
 U 1 1 5B6D51CD
-P 4550 4950
-F 0 "J4" H 4550 5350 50  0000 C CNN
-F 1 "Conn_01x08" H 4550 4450 50  0000 C CNN
-F 2 "footprints:Pin_Header_Straight_1x08_Pitch2.54mm" H 4550 4950 50  0001 C CNN
-F 3 "" H 4550 4950 50  0001 C CNN
-	1    4550 4950
+P 4550 5200
+F 0 "J4" H 4550 5600 50  0000 C CNN
+F 1 "Beetje_Top" H 4350 4700 50  0000 C CNN
+F 2 "footprints:Beetje_Top" H 4550 5200 50  0001 C CNN
+F 3 "" H 4550 5200 50  0001 C CNN
+	1    4550 5200
 	1    0    0    -1
 $EndComp
@@
 L Conn_01x06 J2
 U 1 1 5B6D5224
-P 5200 4850
-F 0 "J2" H 5200 5150 50  0000 C CNN
-F 1 "Conn_01x06" H 5200 4450 50  0000 C CNN
-F 2 "footprints:Pin_Header_Straight_1x06_Pitch2.54mm" H 5200 4850 50  0001 C CNN
-F 3 "" H 5200 4850 50  0001 C CNN
-	1    5200 4850
+P 5200 5100
+F 0 "J2" H 5200 5400 50  0000 C CNN
+F 1 "Beetje_Bottom" H 5050 4700 50  0000 C CNN
+F 2 "footprints:Beetje_Bottom" H 5200 5100 50  0001 C CNN
+F 3 "" H 5200 5100 50  0001 C CNN
+	1    5200 5100
 	-1   0    0    -1
 $EndComp
 Wire Wire Line
-	5400 4650 5700 4650
-Wire Wire Line
-	5400 4750 5700 4750
-Wire Wire Line
-	5400 4850 5700 4850
-Wire Wire Line
-	5400 4950 5700 4950
-Wire Wire Line
-	5400 5050 5700 5050
-Wire Wire Line
-	5400 5150 5700 5150
+	5400 4900 5700 4900
+Wire Wire Line
+	5400 5000 5700 5000
+Wire Wire Line
+	5400 5100 5700 5100
+Wire Wire Line
+	5400 5200 5700 5200
+Wire Wire Line
+	5400 5300 5450 5300
+Wire Wire Line
+	5400 5400 5450 5400
 $Comp
 L VCC #PWR09
@@
 L VCC #PWR010
 U 1 1 5B6E81BF
-P 4150 5150
-F 0 "#PWR010" H 4150 5000 50  0001 C CNN
-F 1 "VCC" V 4150 5350 50  0000 C CNN
-F 2 "" H 4150 5150 50  0001 C CNN
-F 3 "" H 4150 5150 50  0001 C CNN
-	1    4150 5150
-	0    -1   -1   0
+P 5450 5300
+F 0 "#PWR010" H 5450 5150 50  0001 C CNN
+F 1 "VCC" V 5450 5500 50  0000 C CNN
+F 2 "" H 5450 5300 50  0001 C CNN
+F 3 "" H 5450 5300 50  0001 C CNN
+	1    5450 5300
+	0    1    1    0
 $EndComp
 $Comp
@@
 	-1   0    0    1
 $EndComp
-Text Notes 5750 5150 0    60   ~ 0
-D2\nD3\nD15\nD14\nD16
 $Comp
 L VCC #PWR013
@@
 F 0 "C1" H 3625 3800 50  0000 L CNN
 F 1 "1uF" H 3625 3600 50  0000 L CNN
-F 2 "footprints:C_0603" H 3638 3550 50  0001 C CNN
+F 2 "footprints:C_0805_HandSoldering" H 3638 3550 50  0001 C CNN
 F 3 "" H 3600 3700 50  0001 C CNN
 	1    3600 3700
@@
 $EndComp
 $Comp
-L Crystal_GND23 Y1
-U 1 1 5B774C9D
-P 4050 3650
-F 0 "Y1" V 3900 3500 50  0000 L CNN
-F 1 "32.768Hz" V 4300 3400 50  0000 L CNN
-F 2 "footprints:Crystal_SMD_SeikoEpson_MC306-4pin_8.0x3.2mm" H 4050 3650 50  0001 C CNN
-F 3 "" H 4050 3650 50  0001 C CNN
-	1    4050 3650
-	0    1    1    0
-$EndComp
-NoConn ~ 3850 3650
-NoConn ~ 4250 3650
-Wire Wire Line
-	4550 3450 4500 3450
-Wire Wire Line
-	4500 3450 4150 3450
-Wire Wire Line
-	4150 3450 4050 3500
-Wire Wire Line
-	4050 3800 4150 3850
-Wire Wire Line
-	4150 3850 4500 3850
-Wire Wire Line
-	4500 3850 4550 3850
-$Comp
 L VCC #PWR015
 U 1 1 5B7754D8
@@
 	5350 3700 5550 3700
 Wire Wire Line
-	5350 3850 5700 3850
-Wire Wire Line
-	5700 3850 5850 3850
-Wire Wire Line
-	4950 3050 4950 3150
-Wire Wire Line
-	4950 3150 4950 3250
-Wire Wire Line
-	4950 4050 4950 4150
-Wire Wire Line
-	4950 4150 4950 4200
+	5350 3850 5850 3850
+Wire Wire Line
+	4950 3050 4950 3250
+Wire Wire Line
+	4950 4050 4950 4200
 Text Label 5400 3450 0    60   ~ 0
 SCL
@@
 F 0 "R2" V 5850 3600 50  0000 C CNN
 F 1 "4K7" V 5800 3450 50  0000 C CNN
-F 2 "footprints:R_0603" V 5730 3450 50  0001 C CNN
+F 2 "footprints:R_0805_HandSoldering" V 5730 3450 50  0001 C CNN
 F 3 "" H 5800 3450 50  0001 C CNN
 	1    5800 3450
@@
 F 0 "R3" V 5850 3700 50  0000 C CNN
 F 1 "4K7" V 5800 3550 50  0000 C CNN
-F 2 "footprints:R_0603" V 5730 3550 50  0001 C CNN
+F 2 "footprints:R_0805_HandSoldering" V 5730 3550 50  0001 C CNN
 F 3 "" H 5800 3550 50  0001 C CNN
 	1    5800 3550
@@
 	6100 3550 5950 3550
 Wire Wire Line
-	6100 3100 6100 3450
-Wire Wire Line
-	6100 3450 6100 3550
-Wire Wire Line
-	6100 3550 6100 3850
+	6100 3100 6100 3850
 $Comp
 L VCC #PWR017
@@
 F 0 "R1" V 5030 2900 50  0000 C CNN
 F 1 "1K" V 4950 2900 50  0000 C CNN
-F 2 "footprints:R_0603" V 4880 2900 50  0001 C CNN
+F 2 "footprints:R_0805_HandSoldering" V 4880 2900 50  0001 C CNN
 F 3 "" H 4950 2900 50  0001 C CNN
 	1    4950 2900
@@
 F 0 "C2" V 4450 3000 50  0000 L CNN
 F 1 "3.3uF" V 4550 3200 50  0000 L CNN
-F 2 "footprints:C_0603" H 4538 3000 50  0001 C CNN
+F 2 "footprints:C_0805_HandSoldering" H 4538 3000 50  0001 C CNN
 F 3 "" H 4500 3150 50  0001 C CNN
 	1    4500 3150
@@
 Text Notes 6150 3900 0    60   ~ 0
 Close jumper\nto omit BT1.
-$Comp
-L Crystal Y2
+Text Label 5600 5000 0    60   ~ 0
+D6
+Text Notes 3950 4750 0    60   ~ 0
+Beetje Footprint
+Wire Notes Line
+	3850 4600 5850 4600
+Wire Notes Line
+	5850 4600 5850 5800
+Wire Notes Line
+	5850 5800 3850 5800
+Wire Notes Line
+	3850 5800 3850 4600
+$Comp
+L Crystal Y1
 U 1 1 5B778058
 P 4350 3650
-F 0 "Y2" V 4200 3550 50  0000 C CNN
-F 1 "Alternate" H 4350 3800 50  0000 C CNN
+F 0 "Y1" V 4200 3550 50  0000 C CNN
+F 1 "32.768Hz" V 4600 3650 50  0000 C CNN
 F 2 "Crystals:Crystal_SMD_G8-2pin_3.2x1.5mm_HandSoldering" H 4350 3650 50  0001 C CNN
 F 3 "" H 4350 3650 50  0001 C CNN
@@
 $EndComp
 Wire Wire Line
-	4350 3500 4500 3450
-Connection ~ 4500 3450
-Wire Wire Line
-	4350 3800 4500 3850
-Connection ~ 4500 3850
+	4550 3850 4350 3850
+Wire Wire Line
+	4350 3850 4350 3800
+Wire Wire Line
+	4550 3450 4350 3450
+Wire Wire Line
+	4350 3450 4350 3500
+NoConn ~ 4150 4900
+NoConn ~ 4150 5000
+NoConn ~ 4150 5100
+NoConn ~ 4150 5200
+NoConn ~ 4150 5300
+NoConn ~ 4150 5400
+NoConn ~ 5700 5000
+NoConn ~ 5700 4900
 $EndSCHEMATC

Commit message: Updates
Connections:
- no-connect marks 8 -> 7
Changed lines of the file:
@@
 Text Label 4150 5000 0    60   ~ 0
 D9
+Text Label 5550 5100 0    60   ~ 0
+SCL
 Text Label 5550 5200 0    60   ~ 0
-SCL
-Text Label 5550 5100 0    60   ~ 0
 SDA
 Text Label 4150 4900 0    60   ~ 0
@@
 NoConn ~ 4150 4900
 NoConn ~ 4150 5000
-NoConn ~ 4150 5100
 NoConn ~ 4150 5200
 NoConn ~ 4150 5300

Commit message: Updates
Parts:
- removed JP1: (no value), footprints:Jumper, symbol Jumper_NO_Small
- added Y2: ALT, footprints:Crystal_SMD_SeikoEpson_MC306-4pin_8.0x3.2mm, symbol Crystal
Connections:
- wire segments 35 -> 36
Other:
- note removed: "Close jumper\nto omit BT1."
