File: projects/Beetje/design_files_Temp_Press_Humid/project.kicad_pcb (KiCad board)
At the start: 2 copper layers, 25.4 x 25.4 mm, 12 parts, among them J2 Beetje_Bottom, J4 Beetje_Top, U1 Si7021, U2 MPL3115A

Commit message: Updates
Parts:
- J2: footprint footprints:Beetje_Bottom -> beetje_footprints:Beetje_Bottom
- J4: footprint footprints:Beetje_Top -> beetje_footprints:Beetje_Top
Other:
- board text added: "Rev 0.1 Mar 2020"
- board text removed: "Rev 0.0 Mar 2020"
