File: projects/HotWheels LiPo/design_files Charger/project.sch (KiCad schematic (older format))
At the start: 32 parts, among them J1 LED, J2 USB_B, J3 BAT, J4 CONN, J44 CONN, J5 CONN, J55 CONN, J6 LED, J7 LED, J8 LED, J9 LED, SW1 SW_SPDT, U1 MCP73833

Commit message: Updates
Parts:
- added J10: JST_PH, footprints:JST_PH_S2B-PH-K_02x2.00mm_Angled, symbol CONN_01X02
- J3: footprint footprints:JST_PH_S2B-PH-K_02x2.00mm_Angled -> Connectors_Molex:Molex_PicoBlade_53048-0210_02x1.25mm_Angled
Connections:
- net GND: now also J10.2 (P2)
- net at C2.1, J3.1 (P1), J4.1 (P1)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: now also J10.1 (P1)
Changed lines of the file:
@@
 encoding utf-8
 Sheet 1 1
-Title "Beetje LiPo Blok "
+Title "LiPo LED Board "
 Date "2018-09-11"
 Rev "0.2"
@@
 F 0 "J3" H 3150 3900 50  0000 C CNN
 F 1 "BAT" V 3250 3750 50  0000 C CNN
-F 2 "footprints:JST_PH_S2B-PH-K_02x2.00mm_Angled" H 3150 3750 50  0001 C CNN
+F 2 "Connectors_Molex:Molex_PicoBlade_53048-0210_02x1.25mm_Angled" H 3150 3750 50  0001 C CNN
 F 3 "" H 3150 3750 50  0001 C CNN
 	1    3150 3750
@@
 Connection ~ 3350 3400
 Connection ~ 2600 3400
+$Comp
+L CONN_01X02 J10
+U 1 1 5EAB43D0
+P 3150 4050
+F 0 "J10" H 3150 4200 50  0000 C CNN
+F 1 "JST_PH" V 3250 4050 50  0000 C CNN
+F 2 "footprints:JST_PH_S2B-PH-K_02x2.00mm_Angled" H 3150 4050 50  0001 C CNN
+F 3 "" H 3150 4050 50  0001 C CNN
+	1    3150 4050
+	-1   0    0    -1
+$EndComp
+Wire Wire Line
+	3350 4000 3400 4000
+Wire Wire Line
+	3400 4000 3400 3700
+Connection ~ 3400 3700
+Wire Wire Line
+	3350 4100 3450 4100
+Wire Wire Line
+	3450 4100 3450 3800
+Connection ~ 3450 3800
 $EndSCHEMATC
