File: projects/HotWheels/328 Accel/design_files V0.3/project.sch (KiCad schematic (older format))
At the start: 42 parts, among them CON1 AVR-ISP-6, J1 HL, J2 CHG, J3 BAT, J44 Conn, J45 Conn, J46 Conn, J47 Conn, J48 Conn, J49 Conn, J54 Conn, J55 Conn, J56 Conn, J57 Conn, J58 Conn, J59 Conn, J6 HL, J7 TL, J8 TL, SW1 SW_SPDT, U1 MIC5225-3.3, U2 LIS3DH, U3 ATMEGA328-MU

Commit message: Updates
Parts:
- added D1, D2, D3, D6: LED, footprints:LED_0805_HandSoldering, symbol LED
- added J10, J4, J5, J9: LED, footprints:LED_PADS, symbol CONN_01X02
- added J22: CHG, footprints:JST_SH_SM02B-SRSS-TB_02x1.00mm_Angled, symbol CONN_01X02
- added JP2: A2, footprints:Jumper, symbol Jumper_NO_Small
- added JP3: A1, footprints:Jumper, symbol Jumper_NO_Small
- J1, J6, J7, J8: footprint Pin_Headers:Pin_Header_Straight_1x02_Pitch2.00mm -> footprints:PIN_HEADER_LED
- J2, J3: footprint Connectors_JST:JST_SH_SM02B-SRSS-TB_02x1.00mm_Angled -> footprints:JST_SH_SM02B-SRSS-TB_02x1.00mm_Angled
- J44, J45, J46, J47, J48, J49, J54, J55, J56, J57, J58, J59: footprint Wire_Pads:SolderWirePad_single_0-8mmDrill -> footprints:SolderWirePad_single_0-8mmDrill
- R1, R2, R3, R4: footprint footprints:R_0805_HandSoldering -> footprints:R_0603
- U1: footprint TO_SOT_Packages_SMD:SOT-23-5 -> footprints:SOT-23-5
- U3: footprint Housings_DFN_QFN:QFN-32-1EP_5x5mm_Pitch0.5mm -> footprints:QFN-32-1EP_5x5mm_Pitch0.5mm
Connections:
- wire segments 114 -> 136
- no-connect marks 24 -> 21
Other:
- note added: "328 PWM Pins:\n3, 5, 6, 9, 10, 11"
- note added: "JST-PH"
- note added: "JST-SH"
- moved on the sheet: J2, R10, R5
