File: projects/HotWheels/328 Accel/design_files/_saved_project.sch (KiCad schematic (older format))
At the start: 53 parts, among them CON1 AVR-ISP-6, J1 HL, J10 LED, J11 UL, J2 CHG, J22 CHG, J3 BAT, J4 LED, J44 Conn, J45 Conn, J46 Conn, J47 Conn, J48 Conn, J49 Conn, J5 LED, J54 Conn, J55 Conn, J56 Conn, J57 Conn, J58 Conn, J59 Conn, J6 HL, J7 TL, J8 TL, J9 LED, SW1 SW_SPDT, U1 MIC5225-3.3, U2 ADXL343, U3 ATMEGA328-MU

Commit message: Updates
Parts:
- added J12: 3V3, Wire_Pads:SolderWirePad_single_SMD_5x10mm, symbol Conn_01x01
Changed lines of the file:
@@
 	5600 2000 5050 2000
 $Comp
-L GND #PWR011
+L GND #PWR010
 U 1 1 5ED1A3C3
 P 6150 2450
-F 0 "#PWR011" H 6150 2200 50  0001 C CNN
+F 0 "#PWR010" H 6150 2200 50  0001 C CNN
 F 1 "GND" H 6150 2300 50  0000 C CNN
 F 2 "" H 6150 2450 50  0001 C CNN
@@
 	3650 3850 3350 3850
 $Comp
-L +BATT #PWR012
+L +BATT #PWR011
 U 1 1 5ED1DC07
 P 3650 3050
-F 0 "#PWR012" H 3650 2900 50  0001 C CNN
+F 0 "#PWR011" H 3650 2900 50  0001 C CNN
 F 1 "+BATT" V 3650 3300 50  0000 C CNN
 F 2 "" H 3650 3050 50  0001 C CNN
@@
 $EndComp
 $Comp
-L GND #PWR013
+L GND #PWR012
 U 1 1 5ED1E058
 P 3800 4050
-F 0 "#PWR013" H 3800 3800 50  0001 C CNN
+F 0 "#PWR012" H 3800 3800 50  0001 C CNN
 F 1 "GND" H 3800 3900 50  0000 C CNN
 F 2 "" H 3800 4050 50  0001 C CNN
@@
 $EndComp
 $Comp
-L GND #PWR014
+L GND #PWR013
 U 1 1 5ED28276
 P 1850 2500
-F 0 "#PWR014" H 1850 2250 50  0001 C CNN
+F 0 "#PWR013" H 1850 2250 50  0001 C CNN
 F 1 "GND" H 1850 2350 50  0000 C CNN
 F 2 "" H 1850 2500 50  0001 C CNN
@@
 Connection ~ 1850 2450
 $Comp
-L GND #PWR016
+L GND #PWR014
 U 1 1 5ED2945E
 P 1700 7250
-F 0 "#PWR016" H 1700 7000 50  0001 C CNN
+F 0 "#PWR014" H 1700 7000 50  0001 C CNN
 F 1 "GND" H 1700 7100 50  0000 C CNN
 F 2 "" H 1700 7250 50  0001 C CNN
@@
 	8900 5900 9650 5900
 $Comp
-L GND #PWR017
+L GND #PWR015
 U 1 1 5ED343AE
 P 7650 4050
-F 0 "#PWR017" H 7650 3800 50  0001 C CNN
+F 0 "#PWR015" H 7650 3800 50  0001 C CNN
 F 1 "GND" H 7650 3900 50  0000 C CNN
 F 2 "" H 7650 4050 50  0001 C CNN
@@
 Connection ~ 3650 3050
 $Comp
-L +3V3 #PWR019
+L +3V3 #PWR016
 U 1 1 5EE9927E
 P 2450 1750
-F 0 "#PWR019" H 2450 1600 50  0001 C CNN
+F 0 "#PWR016" H 2450 1600 50  0001 C CNN
 F 1 "+3V3" H 2450 1890 50  0000 C CNN
 F 2 "" H 2450 1750 50  0001 C CNN
@@
 $EndComp
 $Comp
-L +3V3 #PWR020
+L +3V3 #PWR017
 U 1 1 5EE99B8A
 P 4250 2800
-F 0 "#PWR020" H 4250 2650 50  0001 C CNN
+F 0 "#PWR017" H 4250 2650 50  0001 C CNN
 F 1 "+3V3" H 4250 2940 50  0000 C CNN
 F 2 "" H 4250 2800 50  0001 C CNN
@@
 $EndComp
 $Comp
-L +3V3 #PWR021
+L +3V3 #PWR018
 U 1 1 5EE9A3D0
 P 4200 6100
-F 0 "#PWR021" H 4200 5950 50  0001 C CNN
+F 0 "#PWR018" H 4200 5950 50  0001 C CNN
 F 1 "+3V3" H 4200 6240 50  0000 C CNN
 F 2 "" H 4200 6100 50  0001 C CNN
@@
 $EndComp
 $Comp
-L +3V3 #PWR022
+L +3V3 #PWR019
 U 1 1 5EE9AF34
 P 1000 950
-F 0 "#PWR022" H 1000 800 50  0001 C CNN
+F 0 "#PWR019" H 1000 800 50  0001 C CNN
 F 1 "+3V3" H 1000 1090 50  0000 C CNN
 F 2 "" H 1000 950 50  0001 C CNN
@@
 Vin
 $Comp
-L +3V3 #PWR023
+L +3V3 #PWR020
 U 1 1 5EE9C4CC
 P 1700 5600
-F 0 "#PWR023" H 1700 5450 50  0001 C CNN
+F 0 "#PWR020" H 1700 5450 50  0001 C CNN
 F 1 "+3V3" H 1700 5740 50  0000 C CNN
 F 2 "" H 1700 5600 50  0001 C CNN
@@
 Text Label 6250 1850 0    60   ~ 0
 Vin
+$Comp
+L Conn_01x01 J12
+U 1 1 5EE9FDD3
+P 2650 1950
+F 0 "J12" H 2800 1950 50  0000 C CNN
+F 1 "3V3" H 2600 1950 50  0000 C CNN
+F 2 "Wire_Pads:SolderWirePad_single_SMD_5x10mm" H 2650 1950 50  0001 C CNN
+F 3 "" H 2650 1950 50  0001 C CNN
+	1    2650 1950
+	1    0    0    -1
+$EndComp
+Connection ~ 2450 1950
 $EndSCHEMATC
