File: projects/HotWheels/328 Accel/design_files/project.sch (KiCad schematic (older format))
At the start: 44 parts, among them CON1 AVR-ISP-6, J1 HL, J2 CHG, J3 BAT, J44 Conn, J45 Conn, J46 Conn, J47 Conn, J48 Conn, J49 Conn, J54 Conn, J55 Conn, J56 Conn, J57 Conn, J58 Conn, J59 Conn, J6 HL, J7 TL, J8 TL, SW1 SW_SPDT, U1 MIC5225-3.3, U2 LIS3DH, U3 ATMEGA328-MU

Commit message: Updates
Parts:
- removed J? (x2): BL, footprints:PIN_HEADER_LED, symbol CONN_01X02
- added D1, D2, D3, D6: LED, footprints:LED_0805_HandSoldering, symbol LED
- added J10, J4, J5, J9: LED, footprints:LED_PADS, symbol CONN_01X02
- added J11: UL, footprints:PIN_HEADER_LED, symbol CONN_01X02
- added J22: CHG, footprints:JST_SH_SM02B-SRSS-TB_02x1.00mm_Angled, symbol CONN_01X02
- added JP2: A2, footprints:Jumper, symbol Jumper_NO_Small
- added JP3: A1, footprints:Jumper, symbol Jumper_NO_Small
Connections:
- wire segments 114 -> 140
- no-connect marks 24 -> 21
Other:
- note added: "328 PWM Pins:\n3, 5, 6, 9, 10, 11"
- note added: "JST-PH"
- note added: "JST-SH"
- moved on the sheet: J2

Commit message: Updates
Parts:
- removed C3: 10uF, footprints:C_0805, symbol C
- removed JP1: JMP, footprints:Jumper, symbol Jumper_NC_Small
- removed U2: LIS3DH, footprints:LIS3DH_EP, symbol LIS3DH
- added J12: TP, Wire_Pads:SolderWirePad_single_SMD_5x10mm, symbol Conn_01x01
- added R13: 10K, footprints:R_0603, symbol R
- added U2: ADXL343, footprints:lga-14, symbol ADXL343
Connections:
- net labels added: +3V3, Vin
- net labels removed: VBUS
- wire segments 140 -> 139
- no-connect marks 21 -> 18
Other:
- note removed: "Cut JP1 if used \nwith LiPo Charge Brd"
- moved on the sheet: C4, J44, R2, R3, R4

Commit message: Updates
Parts:
- J12: value TP -> 3V3
Changed lines of the file:
@@
 P 2650 1950
 F 0 "J12" H 2800 1950 50  0000 C CNN
-F 1 "TP" H 2600 1950 50  0000 C CNN
+F 1 "3V3" H 2600 1950 50  0000 C CNN
 F 2 "Wire_Pads:SolderWirePad_single_SMD_5x10mm" H 2650 1950 50  0001 C CNN
 F 3 "" H 2650 1950 50  0001 C CNN
