File: projects/HotWheels/IR/design_files_32U4/project.sch (KiCad schematic (older format))
At the start: 40 parts, among them CON1 AVR-ISP-6, J1 I2C, J2 RJ45, Q1 Q_Photo_NPN, Q2 Q_Photo_NPN, SW1 RST, SW2 D4, U1 ATMEGA32U4-AU, U2 MIC5225-3.3, X1 USB_OTG, Y1 8 Mhz

Commit message: Updates
Parts:
- removed C1: 10uF, beetje_footprints:C_0805, symbol C
- removed D1: TX, beetje_footprints:LED_0603, symbol LED
- removed D2: RX, beetje_footprints:LED_0603, symbol LED
- removed D3: D13, beetje_footprints:LED_0603, symbol LED
- removed D4, D5: MBR120, beetje_footprints:D_SOD-123F, symbol D_Schottky
- removed JMP1: 5V, beetje_footprints:Jumper, symbol R
- removed SW1: RST, beetje_footprints:EVQ-P7A, symbol SW_Push
- removed U2: MIC5225-3.3, beetje_footprints:SOT-23-5, symbol MIC5219-2.5
- added J3: SERVO_1, Pin_Headers:Pin_Header_Angled_1x03_Pitch2.54mm, symbol CONN_01X03
- added J4: SERVO, Pin_Headers:Pin_Header_Angled_1x03_Pitch2.54mm, symbol CONN_01X03
- C1: renamed from C2; value 10uF -> 0.1uF
- CON1: value AVR-ISP-6 -> ISP
- R1, R2, R3: value 1K -> JMP; footprint beetje_footprints:R_0603 -> footprints:Jumper
- R13, R14: value 100 -> 330
- R8: value 100K -> JMP; footprint beetje_footprints:R_0603 -> footprints:Jumper
- SW1: renamed from SW2; footprint beetje_footprints:EVQ-P7A -> Buttons_Switches_THT:SW_PUSH_6mm
- X1: value USB_OTG -> USB
- renumbered C4 to C2, D8 to D5, D9 to D6, D6 to D8
Connections:
- net labels removed: +BATT, RXLED, TXLED, VBUS, VHI
- wire segments 128 -> 120
- no-connect marks 15 -> 11
Other:
- note removed: "3.3V:\nU2 = MIC5225-3.3\nY1 = 8 Mhz\nJMP1 = Open"
- note removed: "5V:\nU2 = MIC5225-5\nY1 = 16 Mhz\nJMP1 = Short"
- moved on the sheet: D5, D6, Q1, Q2, R12, R13, R14, R9, SW1
