File: projects/HotWheels/Attiny/design_files Attiny85 V0/project.sch (KiCad schematic (older format))
At the start: 18 parts, among them CON1 ISP, IC1 ATTINY25, J1 CHG, J2 HL, J3 BAT, J4 TL, J6 UL, J8 FL, SW1 SW_SPDT

Commit message: Updates
Other:
- note added: "D2/A1"
- note added: "D3/A3"
- note added: "D4/A2"
- note added: "Swith UL & TL\nfor analog read"
Changed lines of the file:
@@
 	3100 3600 3250 3600
 Connection ~ 3250 3950
+Text Notes 9300 3900 0    60   ~ 0
+Swith UL & TL\nfor analog read
+Text Notes 9150 2900 0    60   ~ 0
+D2/A1
+Text Notes 9150 3450 0    60   ~ 0
+D4/A2
+Text Notes 9100 4750 0    60   ~ 0
+D3/A3
 $EndSCHEMATC

Commit message: Updates
Other:
- note added: "D0"
- note added: "Swith UL & TL for analog read?\nPilot hole.\nExtend J1 pads.\nVias under switch pads?\nISP Reset hole?\ncover ISP pads on top\n+/- HL/TL top and bottom\noptional battery connector footprint\nflip orientation?"
- note removed: "Swith UL & TL\nfor analog read"
Changed lines of the file:
@@
 F 0 "IC1" H 4550 4400 50  0000 C CNN
 F 1 "ATTINY25" H 6700 3600 50  0000 C CNN
-F 2 "Housings_SOIC:SOIJ-8_5.3x5.3mm_Pitch1.27mm" H 6650 4000 50  0000 C CIN
+F 2 "Housings_SOIC:SOIJ-8_5.3x5.3mm_Pitch1.27mm" H 5500 3600 50  0000 C CIN
 F 3 "" H 5700 4000 50  0000 C CNN
 	1    5700 4000
@@
 	3100 3600 3250 3600
 Connection ~ 3250 3950
-Text Notes 9300 3900 0    60   ~ 0
-Swith UL & TL\nfor analog read
+Text Notes 7950 2150 0    60   ~ 0
+Swith UL & TL for analog read?\nPilot hole.\nExtend J1 pads.\nVias under switch pads?\nISP Reset hole?\ncover ISP pads on top\n+/- HL/TL top and bottom\noptional battery connector footprint\nflip orientation?
 Text Notes 9150 2900 0    60   ~ 0
 D2/A1
@@
 Text Notes 9100 4750 0    60   ~ 0
 D3/A3
+Text Notes 9150 4050 0    60   ~ 0
+D0
 $EndSCHEMATC
