File: projects/LEGO/design_files_attiny826_LiPo V1/project.kicad_pcb (KiCad board)
At the start: 2 copper layers, 64 x 10 mm, 33 parts, among them J1 USB-MICRO, J2 BAT, J3 UDPI, SW1 SW_SPST, U1 ATtiny826, U2 MCP73833

Commit message: Updates
Parts:
- D1, D2: footprint LED_SMD:LED_0805_2012Metric -> footprints:LED_0805_2012Metric
- D3: value D0 -> PA4; footprint LED_SMD:LED_1206_3216Metric -> footprints:LED_1206_3216Metric
- D4: value D1 -> PA5; footprint LED_SMD:LED_1206_3216Metric -> footprints:LED_1206_3216Metric
- D5: value D8 -> PB1; footprint LED_SMD:LED_1206_3216Metric -> footprints:LED_1206_3216Metric
- D6: value D7 -> PB2; footprint LED_SMD:LED_1206_3216Metric -> footprints:LED_1206_3216Metric
- D7: value D9 -> PB0; footprint LED_SMD:LED_1206_3216Metric -> footprints:LED_1206_3216Metric
- D8: value D16 -> PA3; footprint LED_SMD:LED_1206_3216Metric -> footprints:LED_1206_3216Metric
- D9: value D15 -> PA2; footprint LED_SMD:LED_1206_3216Metric -> footprints:LED_1206_3216Metric
- J2: footprint Connector_Molex:Molex_PicoBlade_53048-0210_1x02_P1.25mm_Horizontal -> footprints:JST_SH_SM02B-SRSS-TB_02x1.00mm_Angled
- R1: value 1 -> 39K
- R2: value 2 -> 10K
- U1: footprint Package_DFN_QFN:VQFN-20-1EP_3x3mm_P0.4mm_EP1.7x1.7mm -> footprints:VQFN-20-1EP_3x3mm_P0.4mm_EP1.7x1.7mm
- moved J2 2.00 mm to (106.8, 83.2)
Connections:
- net /A5 renamed /PIN_PB4
- net /D0 renamed /PIN_PA4
- net /D1 renamed /PIN_PA5
- net /D15 renamed /PIN_PA2
- net /D16 renamed /PIN_PA3
- net /D7 renamed /PIN_PB2
- net /D8 renamed /PIN_PB1
- net /D9 renamed /PIN_PB0
- R1 pad 1: (no net) -> /PIN_PC0
- U1 pad 15: (no net) -> /PIN_PC0
Routing:
- net +BATT: track 62.4 -> 90.5 mm, vias 2 -> 3
- net /PIN_PC0: track 0.00 -> 6.88 mm
- net VBUS: track 17.9 -> 21.0 mm
- net GND: track 126.0 -> 127.3 mm, vias 3 -> 4
- net Net-(R4-Pad1): track 10.0 -> 10.8 mm
Other:
- board text added: "Brick Blinky"
- board text added: "CHG DONE"
- board text added: "Rev 0.1 May 2022"
- board text added: "attiny836_LiPo V1"
- board text added: "bit.ly/MakersBox"
- board text removed: "Rev 0.0"

Commit message: Updates
Parts:
- D3, D4, D5, D6, D7, D8, D9: footprint footprints:LED_1206_3216Metric -> footprints:LED_0805_2012Metric
Routing:
- net Net-(D6-Pad2): track 24.5 -> 27.0 mm, vias 1 -> 3
- net GND: track 127.3 -> 124.9 mm
- net /PIN_PB4: track 10.4 -> 11.1 mm
- net Net-(D4-Pad2): track 33.3 -> 32.7 mm
