File: projects/LEGO/design_files_attiny826_LiPo V1/project.sch (KiCad schematic (older format))
At the start: 33 parts, among them J1 USB-MICRO, J2 BAT, J3 UDPI, SW1 SW_SPST, U1 ATtiny826, U2 MCP73833

Commit message: Updates
Parts:
- C1, C2, C3, C4: symbol project:C -> project-rescue:C-project
- D1, D2: footprint LED_SMD:LED_0805_2012Metric -> footprints:LED_0805_2012Metric; symbol project:LED -> project-rescue:LED-project
- D3: value D0 -> PA4; footprint LED_SMD:LED_1206_3216Metric -> footprints:LED_1206_3216Metric; symbol project:LED -> project-rescue:LED-project
- D4: value D1 -> PA5; footprint LED_SMD:LED_1206_3216Metric -> footprints:LED_1206_3216Metric; symbol project:LED -> project-rescue:LED-project
- D5: value D8 -> PB1; footprint LED_SMD:LED_1206_3216Metric -> footprints:LED_1206_3216Metric; symbol project:LED -> project-rescue:LED-project
- D6: value D7 -> PB2; footprint LED_SMD:LED_1206_3216Metric -> footprints:LED_1206_3216Metric; symbol project:LED -> project-rescue:LED-project
- D7: value D9 -> PB0; footprint LED_SMD:LED_1206_3216Metric -> footprints:LED_1206_3216Metric; symbol project:LED -> project-rescue:LED-project
- D8: value D16 -> PA3; footprint LED_SMD:LED_1206_3216Metric -> footprints:LED_1206_3216Metric; symbol project:LED -> project-rescue:LED-project
- D9: value D15 -> PA2; footprint LED_SMD:LED_1206_3216Metric -> footprints:LED_1206_3216Metric; symbol project:LED -> project-rescue:LED-project
- J1: symbol project:USB_OTG -> project-rescue:USB_OTG-project
- J2: footprint Connector_Molex:Molex_PicoBlade_53048-0210_1x02_P1.25mm_Horizontal -> footprints:JST_SH_SM02B-SRSS-TB_02x1.00mm_Angled
- R1: value 1 -> 39K; symbol project:R -> project-rescue:R-project
- R10, R11, R12, R13, R14, R3, R4, R5, R6, R7, R8, R9: symbol project:R -> project-rescue:R-project
- R2: value 2 -> 10K; symbol project:R -> project-rescue:R-project
- U1: footprint Package_DFN_QFN:VQFN-20-1EP_3x3mm_P0.4mm_EP1.7x1.7mm -> footprints:VQFN-20-1EP_3x3mm_P0.4mm_EP1.7x1.7mm
- U2: symbol project-rescue:MCP73833-AMI_UN-ND-MCP73833 -> project:project-rescue_MCP73833-AMI_UN-ND-MCP73833
Connections:
- net labels added: PIN_PA6, PIN_PA7, PIN_PB3, PIN_PB5
- net labels removed: D2, D3, D4, D6
- wire segments 113 -> 112
Other:
- note added: "VCC"
- note added: "Vcc = Vm * ( R2 / (R1 + R2) ) \nhttps://gist.github.com/dwhacks/7208805"
- note added: "Vm"
- note removed: "39K / 10K ?"
- note removed: "A5 = Vcc * ( R2 / (R1 + R2) ) \nhttps://gist.github.com/dwhacks/7208805"
- moved on the sheet: D5, D6, D7, R10, R8, R9

Commit message: Updates
Parts:
- D3, D4, D5, D6, D7, D8, D9: footprint footprints:LED_1206_3216Metric -> footprints:LED_0805_2012Metric
Changed lines of the file:
@@
 F 0 "D3" H 6800 2100 50  0000 C CNN
 F 1 "PA4" H 6800 1900 50  0000 C CNN
-F 2 "footprints:LED_1206_3216Metric" H 6800 2000 50  0001 C CNN
+F 2 "footprints:LED_0805_2012Metric" H 6800 2000 50  0001 C CNN
 F 3 "" H 6800 2000 50  0001 C CNN
 	1    6800 2000
@@
 F 0 "D4" H 6800 2400 50  0000 C CNN
 F 1 "PA5" H 6800 2200 50  0000 C CNN
-F 2 "footprints:LED_1206_3216Metric" H 6800 2300 50  0001 C CNN
+F 2 "footprints:LED_0805_2012Metric" H 6800 2300 50  0001 C CNN
 F 3 "" H 6800 2300 50  0001 C CNN
 	1    6800 2300
@@
 F 0 "D5" H 6800 3300 50  0000 C CNN
 F 1 "PB1" H 6800 3100 50  0000 C CNN
-F 2 "footprints:LED_1206_3216Metric" H 6800 3200 50  0001 C CNN
+F 2 "footprints:LED_0805_2012Metric" H 6800 3200 50  0001 C CNN
 F 3 "" H 6800 3200 50  0001 C CNN
 	1    6800 3200
@@
 F 0 "D6" H 6800 2700 50  0000 C CNN
 F 1 "PB2" H 6800 2500 50  0000 C CNN
-F 2 "footprints:LED_1206_3216Metric" H 6800 2600 50  0001 C CNN
+F 2 "footprints:LED_0805_2012Metric" H 6800 2600 50  0001 C CNN
 F 3 "" H 6800 2600 50  0001 C CNN
 	1    6800 2600
@@
 F 0 "D8" H 6800 3900 50  0000 C CNN
 F 1 "PA3" H 6800 3700 50  0000 C CNN
-F 2 "footprints:LED_1206_3216Metric" H 6800 3800 50  0001 C CNN
+F 2 "footprints:LED_0805_2012Metric" H 6800 3800 50  0001 C CNN
 F 3 "" H 6800 3800 50  0001 C CNN
 	1    6800 3800
@@
 F 0 "D9" H 6800 3600 50  0000 C CNN
 F 1 "PA2" H 6800 3400 50  0000 C CNN
-F 2 "footprints:LED_1206_3216Metric" H 6800 3500 50  0001 C CNN
+F 2 "footprints:LED_0805_2012Metric" H 6800 3500 50  0001 C CNN
 F 3 "" H 6800 3500 50  0001 C CNN
 	1    6800 3500
@@
 F 0 "D7" H 6800 3000 50  0000 C CNN
 F 1 "PB0" H 6800 2800 50  0000 C CNN
-F 2 "footprints:LED_1206_3216Metric" H 6800 2900 50  0001 C CNN
+F 2 "footprints:LED_0805_2012Metric" H 6800 2900 50  0001 C CNN
 F 3 "" H 6800 2900 50  0001 C CNN
 	1    6800 2900
