File: projects/tester/UCT3/design_files/project.kicad_pcb (KiCad board)
At the start: 2 copper layers, 64.8 x 50.8 mm, 75 parts, among them J1 USB_OTG, J2 ISP, P1 M3, P2 M3, P3 M3, P4 M3, P5 Standoff, P6 Standoff, SW1 RESET, U1 ATMEGA32U4-AU, X1 MEC8-110-02, X2 MEC8-110-02, Y1 16 Mhz

Commit message: Updates
Parts:
- added J1: Conn_02x13_Top_Bottom, footprints:MEC8-113-CARD, F.Cu at (119.5, 98.8)
- added REF**: SAMTEC_MEC8-113-02-X-D-RA1, footprints:SAMTEC_MEC8-113-02-X-D-RA1, F.Cu at (122.0, 88.7)
- moved OSHW1 0.39 mm to (156.2, 118.5)
Other:
- board text added: "Rapid Prototyping Board"
- board text removed: "@TheMakerBox"
- board text removed: "Universal Harness Tester"
