File: projects/LEGO/design_files_attiny826_LEDs/project.kicad_pcb (KiCad board)
At the start: 2 copper layers, 39.8 x 31.5 mm, 37 parts, among them J1 USB-MICRO, J10 PA4*, J11 PA5*, J12 PB2*, J13 PB0*, J14 PA1, J15 PB1*, J16 PA3*, J17 PB5, J18 PB5, J2 PA4*, J3 UDPI, J4 PA5*, J5 PB2*, J6 PB0*, J7 PB1*, J8 PA3*, J9 PA2, SW1 SW_SPST, U1 ATtiny826

Commit message: Updates
Parts:
- removed PA6: PA6, footprints:TestPoint
- added R9: 10K, footprints:R_0805_2012Metric, F.Cu at (125.2, 131.2)
- added TP2: VCC, footprints:TestPoint, F.Cu at (122.3, 130.7)
- moved TP3 7.50 mm to (114.8, 130.7)
- moved TP4 5.50 mm to (119.8, 130.7)
- moved TP1 1.00 mm to (117.3, 130.7)
- renumbered PA7 to TP3, PB4 to TP4
Connections:
- U1 pad 7: /PIN_PA6 -> (no net)
Routing:
- net /PIN_PA6: track 15.1 -> 0.00 mm
- net /PIN_PB4: track 15.3 -> 21.2 mm
- net VCC: track 66.0 -> 71.1 mm
- net GND: track 148.5 -> 152.2 mm
